Commit message: Fixed the friction parameters for the wheels and the caster wheels for the simulation, before this the robot was not rotating well

File: ari_description/urdf/wheels/caster.gazebo.xacro (robot description, xacro)
@@ -10,5 +10,5 @@
   <xacro:macro name="caster_gazebo" params="side">
     <!-- Contact model for the caster wheel surface -->
-    <gazebo reference="caster_${side}_1_link">
+    <!--gazebo reference="caster_${side}_1_link">
       <kp>1000000.0</kp>
       <kd>1000.0</kd>
@@ -20,10 +20,10 @@
       <implicitSpringDamper>0</implicitSpringDamper>
       <material>Gazebo/DarkGrey</material>
-    </gazebo>
-    <gazebo reference="caster_${side}_2_link">
+    </gazebo-->
+    <gazebo reference="caster_${side}_link">
       <kp>1000000.0</kp>
       <kd>1000.0</kd>
-      <mu1>0.4</mu1>
-      <mu2>0.4</mu2>
+      <mu1>1.0</mu1>
+      <mu2>0.1</mu2>
       <fdir1>1 0 0</fdir1>
       <maxVel>1.0</maxVel>

File: ari_description/urdf/wheels/caster.urdf.xacro (robot description, xacro)
@@ -37,5 +37,4 @@
       <origin xyz="${-separation_x / 2} ${-offset_y * reflect} ${offset_z}" rpy="${90.0 * deg_to_rad} 0 0"/>
       <axis xyz="0 0 -1"/>
-      <dynamics damping="0.005" friction="0.0"/>
     </joint>
     <!-- Gazebo extensions -->

File: ari_description/urdf/wheels/wheel.gazebo.xacro (robot description, xacro)
@@ -14,5 +14,5 @@
       <kd>1000.0</kd>
       <mu1>1.0</mu1>
-      <mu2>0.0</mu2> <!-- Frictionless wheels 0.0-->
+      <mu2>0.1</mu2> <!-- Frictionless wheels 0.0-->
       <fdir1>1 0 0</fdir1>
       <maxVel>1.0</maxVel>
