Commit message: Update inertia of caster v2 in urdf

File: ari_description/urdf/wheels/caster_v2.urdf.xacro (robot description, xacro)
@@ -12,8 +12,8 @@
     <link name="caster_${side}_link">
       <inertial>
-        <origin xyz="${-0.016512 * reflect} 0.17601 ${-0.029897 * reflect}" rpy="0 0 0"/>
+        <origin xyz="-0.016512 0 -0.029897" rpy="0 0 0"/>
         <mass value="0.046595"/>
-        <inertia  ixx="7.5074E-06" ixy="${-5.6754E-07 * reflect}" ixz="-2.3436E-07"
-                  iyy="1.6751E-05" iyz="${-1.435E-08 * reflect}"
+        <inertia  ixx="7.5074E-06" ixy="-5.6754E-07" ixz="-2.3436E-07"
+                  iyy="1.6751E-05" iyz="1.435E-08"
                   izz="1.1856E-05"/>
       </inertial>

Commit message: fix warning collision

File: ari_description/urdf/wheels/caster_v2.urdf.xacro (robot description, xacro)
@@ -25,4 +25,10 @@
         <material name="Grey"/>
       </visual>
+      <collision>
+        <origin xyz="0.0 0.0 0.0" rpy="0 0 0"/>
+        <geometry>
+           <sphere radius="${radius}" />
+         </geometry>
+       </collision>
     </link>
     <link name="caster_${side}_2_link">
