Commit message: Add collision meshes

File: ari_description/urdf/arm/arm.urdf.xacro (robot description, xacro)
@@ -49,5 +49,5 @@
         <origin xyz="0 0 0" rpy="0 0 0" />
         <geometry>
-          <mesh filename="package://ari_description/meshes/arm/${name}_base.stl" scale="1 ${reflect} 1"/>
+          <mesh filename="package://ari_description/meshes/arm/${name}_base_collision.stl" scale="1 ${reflect} 1"/>
         </geometry>
       </collision>
@@ -84,5 +84,5 @@
         <origin xyz="0 0 0" rpy="0 0 0" />
         <geometry>
-          <mesh filename="package://ari_description/meshes/arm/${name}_1.stl" scale="1 ${reflect} 1"/>
+          <mesh filename="package://ari_description/meshes/arm/${name}_1_collision.stl" scale="1 ${reflect} 1"/>
         </geometry>
       </collision>
@@ -118,5 +118,5 @@
         <origin xyz="0 0 0" rpy="0 0 0" />
         <geometry>
-          <mesh filename="package://ari_description/meshes/arm/${name}_2.stl" scale="1 ${reflect} 1"/>
+          <mesh filename="package://ari_description/meshes/arm/${name}_2_collision.stl" scale="1 ${reflect} 1"/>
         </geometry>
       </collision>
@@ -153,5 +153,5 @@
         <origin xyz="0 0 0" rpy="0 0 0" />
         <geometry>
-          <mesh filename="package://ari_description/meshes/arm/${name}_3.stl" scale="1 ${reflect} 1"/>
+          <mesh filename="package://ari_description/meshes/arm/${name}_3_collision.stl" scale="1 ${reflect} 1"/>
         </geometry>
       </collision>
@@ -222,8 +222,8 @@
         <geometry>
           <xacro:if value="${end_effector}">
-            <mesh filename="package://ari_description/meshes/arm/${name}_4.stl" scale="1 ${reflect} 1"/>
+            <mesh filename="package://ari_description/meshes/arm/${name}_4_collision.stl" scale="1 ${reflect} 1"/>
           </xacro:if>
           <xacro:unless value="${end_effector}">
-            <mesh filename="package://ari_description/meshes/arm/${name}_${side}_4.stl" scale="1 1 1"/>
+            <mesh filename="package://ari_description/meshes/arm/${name}_${side}_4_collision.stl" scale="1 1 1"/>
           </xacro:unless>
         </geometry>
@@ -312,5 +312,5 @@
         <geometry>
           <mesh
-            filename="package://ari_description/meshes/arm/hand_1.stl" scale="1 ${reflect} 1"/>
+            filename="package://ari_description/meshes/arm/hand_1_collision.stl" scale="1 ${reflect} 1"/>
         </geometry>
       </collision>
@@ -377,5 +377,5 @@
         <geometry>
           <mesh
-            filename="package://ari_description/meshes/arm/hand_2.stl" scale="1 ${reflect} 1"/>
+            filename="package://ari_description/meshes/arm/hand_2_collision.stl" scale="1 ${reflect} 1"/>
         </geometry>
       </collision>

File: ari_description/urdf/base/base.urdf.xacro (robot description, xacro)
@@ -44,5 +44,5 @@
       <origin xyz="0 0 0" rpy="0 0 0" />
       <geometry>
-        <mesh filename="package://ari_description/meshes/base/base.stl" />
+        <mesh filename="package://ari_description/meshes/base/base_collision.stl" />
       </geometry>
       <material name="Grey" />

File: ari_description/urdf/head/head.urdf.xacro (robot description, xacro)
@@ -45,5 +45,5 @@
         <origin xyz="0.0 0 0" rpy="0 0 0.0" />
         <geometry>
-          <mesh filename="package://ari_description/meshes/head/head_1.stl" scale="1 1 1"/>
+          <mesh filename="package://ari_description/meshes/head/head_1_collision.stl" scale="1 1 1"/>
         </geometry>
         <material name="White" />
@@ -95,5 +95,5 @@
         <origin xyz="0 0 0" rpy="0 0 0" />
         <geometry>
-          <mesh filename="package://ari_description/meshes/head/head_2.stl" scale="1 1 1"/>
+          <mesh filename="package://ari_description/meshes/head/head_2_collision.stl" scale="1 1 1"/>
         </geometry>
         <material name="White" />
