Commit message: Fix color fingers in Gazebo visualization

File: ari_description/urdf/arm/actuators.urdf.xacro (robot description, xacro)
@@ -49,5 +49,5 @@
           <sphere radius="0.001"/>
         </geometry>
-        <material name="Hey5DarkGrey" />
+        <material name="White" />
       </visual>
       <collision>

File: ari_description/urdf/arm/arm.urdf.xacro (robot description, xacro)
@@ -239,5 +239,5 @@
     <link name="${name}_${side}_grasping_frame"/>
     <joint name="${name}_${side}_grasping_fixed_joint" type="fixed">
-      <parent link="${name}_${side}_4_link" />/>
+      <parent link="${name}_${side}_4_link" />
       <child link="${name}_${side}_grasping_frame"/>
       <axis xyz="0 0 1" />
@@ -395,5 +395,5 @@
      <material>Gazebo/DarkGrey</material>
    </gazebo>
-   <gazebo reference="$hand_${side}_1_link">
+   <gazebo reference="hand_${side}_1_link">
      <mu1>0.9</mu1>
      <mu2>0.9</mu2>

Commit message: reduce the hand limits from 90deg to 75deg

File: ari_description/urdf/arm/actuators.urdf.xacro (robot description, xacro)
@@ -12,9 +12,9 @@
     <xacro:actuator_impl parent="${parent}" name="${name}">
       <xacro:insert_block name="origin" />
-      <limit lower="${0 * deg_to_rad}" upper="${90 * deg_to_rad}" effort="4.0" velocity="2.5" /> <!-- TODO: Tune effort -->
+      <limit lower="${0 * deg_to_rad}" upper="${75 * deg_to_rad}" effort="4.0" velocity="2.5" /> <!-- TODO: Tune effort -->
       <safety_controller k_position="20"
                          k_velocity="20"
                          soft_lower_limit="${0.0 * deg_to_rad}"
-                         soft_upper_limit="${90.0 * deg_to_rad}" />
+                         soft_upper_limit="${75.0 * deg_to_rad}" />
     </xacro:actuator_impl>
   </xacro:macro>

Commit message: fix robot state publisher launch file

File: ari_description/urdf/arm/actuators.urdf.xacro (robot description, xacro)
@@ -12,5 +12,5 @@
     <xacro:actuator_impl parent="${parent}" name="${name}">
       <xacro:insert_block name="origin" />
-      <limit lower="${0 * deg_to_rad}" upper="${75 * deg_to_rad}" effort="4.0" velocity="2.5" /> <!-- TODO: Tune effort -->
+      <limit lower="${0 * deg_to_rad}" upper="${75 * deg_to_rad}" effort="4.0" velocity="2.5" /> <!-- TODO; Tune effort -->
       <safety_controller k_position="20"
                          k_velocity="20"
@@ -22,9 +22,9 @@
     Common actuator implementation. Create a joint/link pair representing an actuator.
     Parameters:
-    - name: Actuator name. The created link and joint are prepended with 'name_'
-    - parent: Parent link
-    - origin: XML block containing the pose of the actuator joint with respect to its parent
-    - limit: XML block containing the joint limit specification
-    - safety_controller: XML block containing the soft joint limits specification
+    - name; Actuator name. The created link and joint are prepended with 'name_'
+    - parent; Parent link
+    - origin; XML block containing the pose of the actuator joint with respect to its parent
+    - limit; XML block containing the joint limit specification
+    - safety_controller; XML block containing the soft joint limits specification
   -->
   <xacro:macro name="actuator_impl" params="name parent *origin *limit *safety_controller">
@@ -35,5 +35,5 @@
       <axis xyz="0 0 1" />
       <xacro:insert_block name="limit" />
-      <dynamics friction="0.0" damping="0.5"/> <!-- TODO: Tune -->
+      <dynamics friction="0.0" damping="0.5"/> <!-- TODO; Tune -->
       <xacro:insert_block name="safety_controller" />
     </joint>

File: ari_description/urdf/head/head.urdf.xacro (robot description, xacro)
@@ -11,5 +11,5 @@
   <xacro:include filename="$(find ari_description)/urdf/deg_to_rad.xacro" />
   <xacro:include filename="$(find ari_description)/urdf/sensors/rpi_camera.gazebo.xacro" />
-<!-- TODO ROS2: disabled until realsense camera available
+<!-- TODO ROS2; disabled until realsense camera available
     <xacro:include filename="$(find realsense2_description)/urdf/_d435.urdf.xacro" />
 -->

File: ari_description/urdf/torso/torso_sensors.urdf.xacro (robot description, xacro)
@@ -10,5 +10,5 @@
   <!--File includes-->
   <xacro:include filename="$(find ari_description)/urdf/deg_to_rad.xacro" />
-<!-- TODO ROS2: disabled until realsense camera available
+<!-- TODO ROS2; disabled until realsense camera available
   <xacro:include filename="$(find realsense2_description)/urdf/_d435.urdf.xacro" />
   <xacro:include filename="$(find realsense2_description)/urdf/_t265.urdf.xacro" />
@@ -67,5 +67,5 @@
   <!-- Torso sensors -->
   <!-- Torso front camera -->
-<!-- TODO ROS2: disabled until realsense camera available
+<!-- TODO ROS2; disabled until realsense camera available
   <xacro:sensor_d435 parent="${parent}" name="${name}_front_camera" topics_ns="${name}_front_camera" use_nominal_extrinsics="${use_nominal_extrinsics}">
     <origin xyz="${torso_front_camera_position_x} ${torso_front_camera_position_y} ${torso_front_camera_position_z}"
@@ -74,5 +74,5 @@
 -->
   <!-- Torso back camera -->
-<!-- TODO ROS2: disabled until realsense camera available
+<!-- TODO ROS2; disabled until realsense camera available
   <xacro:sensor_t265 parent="${parent}" name="${name}_back_camera" topics_ns="${name}_back_camera">
     <origin xyz="${torso_back_camera_position_x} ${torso_back_camera_position_y} ${torso_back_camera_position_z}"
