Commit message: Set joint rotation direction correctly for both arms

File: ari_description/urdf/arm/arm_v2.urdf.xacro (robot description, xacro)
@@ -161,5 +161,5 @@
       <origin xyz="-0.023833 ${0.1003 * reflect} -0.008"
               rpy="${(90 - 5.00192155 * reflect) * deg_to_rad} ${90 * deg_to_rad} 0" />
-      <axis xyz="0 0 ${1*reflect}" />
+      <axis xyz="0 0 1" />
       <limit lower="-2.09" upper="2.09" effort="${arm_3_max_effort}" velocity="${arm_3_max_vel}" />
       <dynamics friction="${arm_friction}" damping="${arm_damping}"/>
@@ -221,8 +221,8 @@
         <geometry>
           <xacro:if value="${end_effector}">
-            <mesh filename="package://ari_left_arm/meshes/arm_left_4_link.STL" scale="1 ${reflect} 1"/>
+            <mesh filename="package://ari_left_arm/meshes/arm_left_4_link.STL" scale="${reflect} 1 1"/>
           </xacro:if>
           <xacro:unless value="${end_effector}">
-            <mesh filename="package://ari_left_arm/meshes/arm_left_4_link.STL" scale="1 ${reflect} 1"/>
+            <mesh filename="package://ari_left_arm/meshes/arm_left_4_link.STL" scale="${reflect} 1 1"/>
           </xacro:unless>
         </geometry>

Commit message: fix bug in test

File: ari_description/urdf/arm/arm_v2.urdf.xacro (robot description, xacro)
@@ -127,10 +127,10 @@
               rpy="0 ${1.5708 * 1} 0" />
       <axis xyz="0 0 1" />
-      <limit lower="${-24 * deg_to_rad}" upper="${70 * deg_to_rad}" effort="${arm_2_max_effort}" velocity="${arm_2_max_vel}" />
-      <dynamics friction="${arm_friction}" damping="${arm_damping}"/>
-      <safety_controller k_position="20"
-                         k_velocity="20"
-                         soft_lower_limit="${-24 * deg_to_rad  + arm_eps}"
-                         soft_upper_limit="${70 * deg_to_rad - arm_eps}" />
+      <limit lower="${0 * deg_to_rad}" upper="${100 * deg_to_rad}" effort="${arm_2_max_effort}" velocity="${arm_2_max_vel}" />
+      <dynamics friction="${arm_friction}" damping="${arm_damping}"/>
+      <safety_controller k_position="20"
+                         k_velocity="20"
+                         soft_lower_limit="${0 * deg_to_rad  + arm_eps}"
+                         soft_upper_limit="${100 * deg_to_rad - arm_eps}" />
     </joint>
     <link name="${name}_${side}_3_link">
@@ -162,10 +162,10 @@
               rpy="${(90 - 5.0) * deg_to_rad} ${90 * deg_to_rad} 0" />
       <axis xyz="0 0 ${reflect}" />
-      <limit lower="${-45 * deg_to_rad}" upper="${195.0 * deg_to_rad}" effort="${arm_3_max_effort}" velocity="${arm_3_max_vel}" />
-      <dynamics friction="${arm_friction}" damping="${arm_damping}"/>
-      <safety_controller k_position="20"
-                         k_velocity="20"
-                         soft_lower_limit="${-45 * deg_to_rad + arm_eps}"
-                         soft_upper_limit="${195 * deg_to_rad - arm_eps}" />
+      <limit lower="${-120 * deg_to_rad}" upper="${120.0 * deg_to_rad}" effort="${arm_3_max_effort}" velocity="${arm_3_max_vel}" />
+      <dynamics friction="${arm_friction}" damping="${arm_damping}"/>
+      <safety_controller k_position="20"
+                         k_velocity="20"
+                         soft_lower_limit="${-120 * deg_to_rad + arm_eps}"
+                         soft_upper_limit="${120 * deg_to_rad - arm_eps}" />
     </joint>
     <!--************************-->
@@ -185,45 +185,14 @@
       </inertial>
       <visual>
-        <xacro:if value="${end_effector}">
-          <origin xyz="0 0 0" rpy="0 0 0" />
-        </xacro:if>
-        <xacro:unless value="${end_effector}">
-          <xacro:if value="${side == 'left'}">
-            <origin xyz="0 0 0" rpy="0 0 0" />
-          </xacro:if>
-          <xacro:if value="${side == 'right'}">
-            <origin xyz="0 0 0" rpy="0 0 ${-90 * deg_to_rad}" />
-          </xacro:if>
-        </xacro:unless>
-        <geometry>
-          <xacro:if value="${end_effector}">
-            <mesh filename="package://ari_description/meshes/arm/arm_4_v2.stl" scale="1 ${reflect} 1"/>
-          </xacro:if>
-          <xacro:unless value="${end_effector}">
-            <mesh filename="package://ari_description/meshes/arm/arm_4_v2.stl" scale="1 ${reflect} 1"/>
-          </xacro:unless>
+        <origin xyz="0 0 0" rpy="0 0 0" />
+        <geometry>
+          <mesh filename="package://ari_description/meshes/arm/arm_4_v2.stl" scale="1 ${reflect} 1"/>
         </geometry>
         <material name="White" />
       </visual>
       <collision>
-        <xacro:if value="${end_effector}">
-          <origin xyz="0 0 0" rpy="0 0 0" />
-        </xacro:if>
-        <xacro:unless value="${end_effector}">
-          <xacro:if value="${side == 'left'}">
-            <origin xyz="0 0 0" rpy="0 0 0" />
-          </xacro:if>
-          <xacro:if value="${side == 'right'}">
-            <origin xyz="0 0 0" rpy="0 0 ${-90 * deg_to_rad}" />
-          </xacro:if>
-        </xacro:unless>
-        <origin xyz="0 0 0" rpy="0 0 0" />
-        <geometry>
-          <xacro:if value="${end_effector}">
-            <mesh filename="package://ari_description/meshes/arm/arm_4_v2.stl" scale="1 ${reflect} 1"/>
-          </xacro:if>
-          <xacro:unless value="${end_effector}">
-            <mesh filename="package://ari_description/meshes/arm/arm_4_v2.stl" scale="1 ${reflect} 1"/>
-          </xacro:unless>
+        <origin xyz="0 0 0" rpy="0 0 0" />
+        <geometry>
+          <mesh filename="package://ari_description/meshes/arm/arm_4_v2.stl" scale="1 ${reflect} 1"/>
         </geometry>
       </collision>
@@ -234,13 +203,13 @@
       <origin xyz="0 0.00049107 -0.1001"
               rpy="${90 * deg_to_rad} ${-90 * deg_to_rad} 0" />
-      <axis xyz="0 0 ${-1*reflect}" />
+      <axis xyz="0 0 ${1*reflect}" />
       <xacro:property name="arm_4_upper_limit"       value="135.0"/>
       <xacro:property name="arm_4_lower_limit"       value="-5.0"/>
-      <limit lower="${0 * deg_to_rad}" upper="${100 * deg_to_rad}" effort="${arm_4_max_effort}" velocity="${arm_4_max_vel}" />
-      <dynamics friction="${arm_friction}" damping="${arm_damping}"/>
-      <safety_controller k_position="20"
-                         k_velocity="20"
-                         soft_lower_limit="${0 * deg_to_rad + arm_eps}"
-                         soft_upper_limit="${100 * deg_to_rad - arm_eps}" />
+      <limit lower="${-100 * deg_to_rad}" upper="${0 * deg_to_rad}" effort="${arm_4_max_effort}" velocity="${arm_4_max_vel}" />
+      <dynamics friction="${arm_friction}" damping="${arm_damping}"/>
+      <safety_controller k_position="20"
+                         k_velocity="20"
+                         soft_lower_limit="${-100 * deg_to_rad + arm_eps}"
+                         soft_upper_limit="${0 * deg_to_rad - arm_eps}" />
     </joint>
     <link name="${name}_${side}_5_link">
@@ -253,48 +222,31 @@
         </inertial>
       <visual>
-        <origin
-          xyz="0 0 0"
-          rpy="0 0 0" />
-        <geometry>
-          <mesh
-            filename="package://ari_description/meshes/arm/arm_5_v2.stl" scale="${reflect} 1 1"/>
-        </geometry>
-        <material
-          name="White" />
-      </visual>
-      <collision>
-        <origin
-          xyz="0 0 0"
-          rpy="0 0 0" />
-        <geometry>
-          <mesh
-            filename="package://ari_description/meshes/arm/arm_5_v2.stl" scale="${reflect} 1 1"/>
-        </geometry>
-      </collision>
-    </link>
-    <joint
-      name="${name}_${side}_5_joint"
-      type="revolute">
-      <origin
-        xyz="-0.106 0 0.0010076"
-        rpy="${-90 * deg_to_rad} 0 ${-90 * deg_to_rad}" />
-      <parent
-        link="${name}_${side}_4_link" />
-      <child
-        link="${name}_${side}_5_link" />
-      <axis
-        xyz="0 0 ${reflect}" />
+        <origin xyz="0 0 0" rpy="0 0 0" />
+        <geometry>
+          <mesh filename="package://ari_description/meshes/arm/arm_5_v2.stl" scale="${reflect} 1 1"/>
+        </geometry>
+        <material name="White" />
+      </visual>
+      <collision>
+        <origin xyz="0 0 0" rpy="0 0 0" />
+        <geometry>
+          <mesh filename="package://ari_description/meshes/arm/arm_5_v2.stl" scale="${reflect} 1 1"/>
+        </geometry>
+      </collision>
+    </link>
+    <joint name="${name}_${side}_5_joint" type="revolute">
+      <origin xyz="-0.106 0 0.0010076" rpy="${-90 * deg_to_rad} 0 ${-90 * deg_to_rad}" />
+      <parent link="${name}_${side}_4_link" />
+      <child link="${name}_${side}_5_link" />
+      <axis xyz="0 0 ${reflect}" />
       <xacro:property name="arm_5_upper_limit"       value="135.0"/>
       <xacro:property name="arm_5_lower_limit"       value="-5.0"/>
-      <limit
-        lower="-2.09"
-        upper="2.09"
-        effort="${arm_4_max_effort}"
-        velocity="${arm_4_max_vel}" />
-      <dynamics friction="${arm_friction}" damping="${arm_damping}"/>
-      <safety_controller k_position="20"
-                         k_velocity="20"
-                         soft_lower_limit="${-135.0 * deg_to_rad + arm_eps}"
-                         soft_upper_limit="${135.0 * deg_to_rad - arm_eps}" />
+      <limit lower="${-120 * deg_to_rad}" upper="${120 * deg_to_rad}"
+        effort="${arm_4_max_effort}" velocity="${arm_4_max_vel}" />
+      <dynamics friction="${arm_friction}" damping="${arm_damping}"/>
+      <safety_controller k_position="20"
+                         k_velocity="20"
+                         soft_lower_limit="${-120.0 * deg_to_rad + arm_eps}"
+                         soft_upper_limit="${120.0 * deg_to_rad - arm_eps}" />
     </joint>
    <gazebo reference="${name}_${side}_1_link">

Commit message: Add frame for hand

File: ari_description/urdf/arm/arm_v2.urdf.xacro (robot description, xacro)
@@ -252,4 +252,17 @@
                          soft_upper_limit="${120.0 * deg_to_rad - arm_eps}" />
     </joint>
+  <!-- hand Link -->
+  <joint name="${name}_${side}_hand_joint" type="fixed">
+      <parent link="${name}_${side}_5_link"/>
+      <child link="${name}_${side}_hand_link"/>
+      <origin xyz="0.0 0.01262 -0.24674" rpy="0 0 0" />
+  </joint>
+  <link name="${name}_${side}_hand_link">
+      <inertial>
+          <origin xyz="0 0 0" rpy="0 0 0"/>
+          <mass value="0.0001" />
+          <inertia ixx="0.0001"  ixy="0"  ixz="0" iyy="0.0001" iyz="0" izz="0.0001" />
+      </inertial>
+  </link>
    <gazebo reference="${name}_${side}_1_link">
      <mu1>0.9</mu1>

Commit message: set correct joint limits

File: ari_description/urdf/arm/arm_v2.urdf.xacro (robot description, xacro)
@@ -94,10 +94,10 @@
       <origin xyz="0.0 0.0047319 -0.00041399" rpy="${(-90 - 5.0) * deg_to_rad} 0.0 0.0"/>
       <axis xyz="0 0 ${-1 * reflect}" />
-      <limit lower="${-120.0 * deg_to_rad}" upper="${120.0 * deg_to_rad}" effort="${arm_1_max_effort}" velocity="${arm_1_max_vel}" />
-      <dynamics friction="${arm_friction}" damping="${arm_damping}"/>
-      <safety_controller k_position="20"
-                         k_velocity="20"
-                         soft_lower_limit="${-120.0 * deg_to_rad + arm_eps}"
-                         soft_upper_limit="${120.0 * deg_to_rad - arm_eps}" />
+      <limit lower="${-110.0 * deg_to_rad}" upper="${110.0 * deg_to_rad}" effort="${arm_1_max_effort}" velocity="${arm_1_max_vel}" />
+      <dynamics friction="${arm_friction}" damping="${arm_damping}"/>
+      <safety_controller k_position="20"
+                         k_velocity="20"
+                         soft_lower_limit="${-110.0 * deg_to_rad + arm_eps}"
+                         soft_upper_limit="${110.0 * deg_to_rad - arm_eps}" />
     </joint>
    <link name="${name}_${side}_2_link">
@@ -129,10 +129,10 @@
               rpy="0 ${1.5708 * 1} 0" />
       <axis xyz="0 0 1" />
-      <limit lower="${0 * deg_to_rad}" upper="${100 * deg_to_rad}" effort="${arm_2_max_effort}" velocity="${arm_2_max_vel}" />
-      <dynamics friction="${arm_friction}" damping="${arm_damping}"/>
-      <safety_controller k_position="20"
-                         k_velocity="20"
-                         soft_lower_limit="${0 * deg_to_rad  + arm_eps}"
-                         soft_upper_limit="${100 * deg_to_rad - arm_eps}" />
+      <limit lower="${2 * deg_to_rad}" upper="${95 * deg_to_rad}" effort="${arm_2_max_effort}" velocity="${arm_2_max_vel}" />
+      <dynamics friction="${arm_friction}" damping="${arm_damping}"/>
+      <safety_controller k_position="20"
+                         k_velocity="20"
+                         soft_lower_limit="${2 * deg_to_rad  + arm_eps}"
+                         soft_upper_limit="${95 * deg_to_rad - arm_eps}" />
     </joint>
     <link name="${name}_${side}_3_link">
@@ -164,10 +164,10 @@
               rpy="${(90 - 5.0) * deg_to_rad} ${90 * deg_to_rad} 0" />
       <axis xyz="0 0 ${reflect}" />
-      <limit lower="${-120 * deg_to_rad}" upper="${120.0 * deg_to_rad}" effort="${arm_3_max_effort}" velocity="${arm_3_max_vel}" />
-      <dynamics friction="${arm_friction}" damping="${arm_damping}"/>
-      <safety_controller k_position="20"
-                         k_velocity="20"
-                         soft_lower_limit="${-120 * deg_to_rad + arm_eps}"
-                         soft_upper_limit="${120 * deg_to_rad - arm_eps}" />
+      <limit lower="${-110 * deg_to_rad}" upper="${110.0 * deg_to_rad}" effort="${arm_3_max_effort}" velocity="${arm_3_max_vel}" />
+      <dynamics friction="${arm_friction}" damping="${arm_damping}"/>
+      <safety_controller k_position="20"
+                         k_velocity="20"
+                         soft_lower_limit="${-110 * deg_to_rad + arm_eps}"
+                         soft_upper_limit="${110 * deg_to_rad - arm_eps}" />
     </joint>
     <!--************************-->
@@ -208,10 +208,10 @@
       <xacro:property name="arm_4_upper_limit"       value="135.0"/>
       <xacro:property name="arm_4_lower_limit"       value="-5.0"/>
-      <limit lower="${0 * deg_to_rad}" upper="${135 * deg_to_rad}" effort="${arm_4_max_effort}" velocity="${arm_4_max_vel}" />
-      <dynamics friction="${arm_friction}" damping="${arm_damping}"/>
-      <safety_controller k_position="20"
-                         k_velocity="20"
-                         soft_lower_limit="${0 * deg_to_rad + arm_eps}"
-                         soft_upper_limit="${135 * deg_to_rad - arm_eps}" />
+      <limit lower="${3 * deg_to_rad}" upper="${90 * deg_to_rad}" effort="${arm_4_max_effort}" velocity="${arm_4_max_vel}" />
+      <dynamics friction="${arm_friction}" damping="${arm_damping}"/>
+      <safety_controller k_position="20"
+                         k_velocity="20"
+                         soft_lower_limit="${3 * deg_to_rad + arm_eps}"
+                         soft_upper_limit="${90 * deg_to_rad - arm_eps}" />
     </joint>
     <link name="${name}_${side}_5_link">
@@ -244,11 +244,11 @@
       <xacro:property name="arm_5_upper_limit"       value="135.0"/>
       <xacro:property name="arm_5_lower_limit"       value="-5.0"/>
-      <limit lower="${-120 * deg_to_rad}" upper="${120 * deg_to_rad}"
+      <limit lower="${-110 * deg_to_rad}" upper="${110 * deg_to_rad}"
         effort="${arm_5_max_effort}" velocity="${arm_5_max_vel}" />
       <dynamics friction="${arm_friction}" damping="${arm_damping}"/>
       <safety_controller k_position="20"
                          k_velocity="20"
-                         soft_lower_limit="${-120.0 * deg_to_rad + arm_eps}"
-                         soft_upper_limit="${120.0 * deg_to_rad - arm_eps}" />
+                         soft_lower_limit="${-110.0 * deg_to_rad + arm_eps}"
+                         soft_upper_limit="${110.0 * deg_to_rad - arm_eps}" />
     </joint>
   <!-- hand Link -->

Commit message: Update joint limits and wheel radius

File: ari_description/urdf/arm/arm_v2.urdf.xacro (robot description, xacro)
@@ -25,4 +25,14 @@
   <xacro:property name="arm_4_max_effort"   value="5" />
   <xacro:property name="arm_5_max_effort"   value="5" />
+  <xacro:property name="arm_1_lower_limit"  value="${-115.0 * deg_to_rad}"/>
+  <xacro:property name="arm_1_upper_limit"  value="${115.0 * deg_to_rad}"/>
+  <xacro:property name="arm_2_lower_limit"  value="${5.0 * deg_to_rad}"/>
+  <xacro:property name="arm_2_upper_limit"  value="${95.0 * deg_to_rad}"/>
+  <xacro:property name="arm_3_lower_limit"  value="${-115.0 * deg_to_rad}"/>
+  <xacro:property name="arm_3_upper_limit"  value="${115.0 * deg_to_rad}"/>
+  <xacro:property name="arm_4_lower_limit"  value="${5.0 * deg_to_rad}"/>
+  <xacro:property name="arm_4_upper_limit"  value="${95.0 * deg_to_rad}"/>
+  <xacro:property name="arm_5_lower_limit"  value="${-115.0 * deg_to_rad}"/>
+  <xacro:property name="arm_5_upper_limit"  value="${115.0 * deg_to_rad}"/>
   <xacro:property name="arm_eps"            value="0.07" />
   <xacro:macro name="ari_arm" params="name parent side reflect end_effector *origin">
@@ -94,10 +104,10 @@
       <origin xyz="0.0 0.0047319 -0.00041399" rpy="${(-90 - 5.0) * deg_to_rad} 0.0 0.0"/>
       <axis xyz="0 0 ${-1 * reflect}" />
-      <limit lower="${-110.0 * deg_to_rad}" upper="${110.0 * deg_to_rad}" effort="${arm_1_max_effort}" velocity="${arm_1_max_vel}" />
-      <dynamics friction="${arm_friction}" damping="${arm_damping}"/>
-      <safety_controller k_position="20"
-                         k_velocity="20"
-                         soft_lower_limit="${-110.0 * deg_to_rad + arm_eps}"
-                         soft_upper_limit="${110.0 * deg_to_rad - arm_eps}" />
+      <limit lower="${arm_1_lower_limit}" upper="${arm_1_upper_limit}"  effort="${arm_1_max_effort}" velocity="${arm_1_max_vel}" />
+      <dynamics friction="${arm_friction}" damping="${arm_damping}"/>
+      <safety_controller k_position="20"
+                         k_velocity="20"
+                         soft_lower_limit="${arm_1_lower_limit + arm_eps}"
+                         soft_upper_limit="${arm_1_upper_limit - arm_eps}" />
     </joint>
    <link name="${name}_${side}_2_link">
@@ -129,10 +139,10 @@
               rpy="0 ${1.5708 * 1} 0" />
       <axis xyz="0 0 1" />
-      <limit lower="${2 * deg_to_rad}" upper="${95 * deg_to_rad}" effort="${arm_2_max_effort}" velocity="${arm_2_max_vel}" />
-      <dynamics friction="${arm_friction}" damping="${arm_damping}"/>
-      <safety_controller k_position="20"
-                         k_velocity="20"
-                         soft_lower_limit="${2 * deg_to_rad  + arm_eps}"
-                         soft_upper_limit="${95 * deg_to_rad - arm_eps}" />
+      <limit lower="${arm_2_lower_limit}" upper="${arm_2_upper_limit}" effort="${arm_2_max_effort}" velocity="${arm_2_max_vel}" />
+      <dynamics friction="${arm_friction}" damping="${arm_damping}"/>
+      <safety_controller k_position="20"
+                         k_velocity="20"
+                         soft_lower_limit="${arm_2_lower_limit  + arm_eps}"
+                         soft_upper_limit="${arm_2_upper_limit - arm_eps}" />
     </joint>
     <link name="${name}_${side}_3_link">
@@ -164,10 +174,10 @@
               rpy="${(90 - 5.0) * deg_to_rad} ${90 * deg_to_rad} 0" />
       <axis xyz="0 0 ${reflect}" />
-      <limit lower="${-110 * deg_to_rad}" upper="${110.0 * deg_to_rad}" effort="${arm_3_max_effort}" velocity="${arm_3_max_vel}" />
-      <dynamics friction="${arm_friction}" damping="${arm_damping}"/>
-      <safety_controller k_position="20"
-                         k_velocity="20"
-                         soft_lower_limit="${-110 * deg_to_rad + arm_eps}"
-                         soft_upper_limit="${110 * deg_to_rad - arm_eps}" />
+      <limit lower="${arm_3_lower_limit }" upper="${arm_3_upper_limit }" effort="${arm_3_max_effort}" velocity="${arm_3_max_vel}" />
+      <dynamics friction="${arm_friction}" damping="${arm_damping}"/>
+      <safety_controller k_position="20"
+                         k_velocity="20"
+                         soft_lower_limit="${arm_3_lower_limit  + arm_eps}"
+                         soft_upper_limit="${arm_3_upper_limit - arm_eps}" />
     </joint>
     <!--************************-->
@@ -206,12 +216,10 @@
               rpy="${90 * deg_to_rad} ${-90 * deg_to_rad} 0" />
       <axis xyz="0 0 ${-1 * reflect}" />
-      <xacro:property name="arm_4_upper_limit"       value="135.0"/>
-      <xacro:property name="arm_4_lower_limit"       value="-5.0"/>
-      <limit lower="${3 * deg_to_rad}" upper="${90 * deg_to_rad}" effort="${arm_4_max_effort}" velocity="${arm_4_max_vel}" />
-      <dynamics friction="${arm_friction}" damping="${arm_damping}"/>
-      <safety_controller k_position="20"
-                         k_velocity="20"
-                         soft_lower_limit="${3 * deg_to_rad + arm_eps}"
-                         soft_upper_limit="${90 * deg_to_rad - arm_eps}" />
+      <limit lower="${arm_4_lower_limit}" upper="${arm_4_upper_limit}" effort="${arm_4_max_effort}" velocity="${arm_4_max_vel}" />
+      <dynamics friction="${arm_friction}" damping="${arm_damping}"/>
+      <safety_controller k_position="20"
+                         k_velocity="20"
+                         soft_lower_limit="${arm_4_lower_limit  + arm_eps}"
+                         soft_upper_limit="${arm_4_upper_limit - arm_eps}" />
     </joint>
     <link name="${name}_${side}_5_link">
@@ -242,13 +250,11 @@
       <child link="${name}_${side}_5_link" />
       <axis xyz="0 0 ${reflect}" />
-      <xacro:property name="arm_5_upper_limit"       value="135.0"/>
-      <xacro:property name="arm_5_lower_limit"       value="-5.0"/>
-      <limit lower="${-110 * deg_to_rad}" upper="${110 * deg_to_rad}"
+      <limit lower="${arm_5_lower_limit}" upper="${arm_5_upper_limit}"
         effort="${arm_5_max_effort}" velocity="${arm_5_max_vel}" />
       <dynamics friction="${arm_friction}" damping="${arm_damping}"/>
       <safety_controller k_position="20"
                          k_velocity="20"
-                         soft_lower_limit="${-110.0 * deg_to_rad + arm_eps}"
-                         soft_upper_limit="${110.0 * deg_to_rad - arm_eps}" />
+                         soft_lower_limit="${arm_5_lower_limit  + arm_eps}"
+                         soft_upper_limit="${arm_5_upper_limit - arm_eps}" />
     </joint>
   <!-- hand Link -->

File: ari_description/urdf/base/base_v2.urdf.xacro (robot description, xacro)
@@ -14,5 +14,5 @@
   <xacro:include filename="$(find ari_description)/urdf/base/docking_link_v2.urdf.xacro"/>
   <!-- Wheel characteristics -->
-  <xacro:property name="wheel_radius"     value="0.11"/>
+  <xacro:property name="wheel_radius"     value="0.1"/>
   <xacro:property name="wheel_width"      value="0.06"/>
   <xacro:property name="wheel_separation" value="0.4668"/>
