Commit message: update joint limits

File: ari_description/urdf/arm/arm_v2.urdf.xacro (robot description, xacro)
@@ -25,12 +25,12 @@
   <xacro:property name="arm_4_max_effort"   value="5" />
   <xacro:property name="arm_5_max_effort"   value="5" />
-  <xacro:property name="arm_1_lower_limit"  value="${-115.0 * deg_to_rad}"/>
-  <xacro:property name="arm_1_upper_limit"  value="${115.0 * deg_to_rad}"/>
-  <xacro:property name="arm_2_lower_limit"  value="${5.0 * deg_to_rad}"/>
-  <xacro:property name="arm_2_upper_limit"  value="${95.0 * deg_to_rad}"/>
-  <xacro:property name="arm_3_lower_limit"  value="${-115.0 * deg_to_rad}"/>
-  <xacro:property name="arm_3_upper_limit"  value="${115.0 * deg_to_rad}"/>
-  <xacro:property name="arm_4_lower_limit"  value="${5.0 * deg_to_rad}"/>
-  <xacro:property name="arm_4_upper_limit"  value="${95.0 * deg_to_rad}"/>
+  <xacro:property name="arm_1_lower_limit"  value="${-120.0 * deg_to_rad}"/>
+  <xacro:property name="arm_1_upper_limit"  value="${120.0 * deg_to_rad}"/>
+  <xacro:property name="arm_2_lower_limit"  value="${1.0 * deg_to_rad}"/>
+  <xacro:property name="arm_2_upper_limit"  value="${100.0 * deg_to_rad}"/>
+  <xacro:property name="arm_3_lower_limit"  value="${-120.0 * deg_to_rad}"/>
+  <xacro:property name="arm_3_upper_limit"  value="${120.0 * deg_to_rad}"/>
+  <xacro:property name="arm_4_lower_limit"  value="${1.0 * deg_to_rad}"/>
+  <xacro:property name="arm_4_upper_limit"  value="${100.0 * deg_to_rad}"/>
   <xacro:property name="arm_5_lower_limit"  value="${-115.0 * deg_to_rad}"/>
   <xacro:property name="arm_5_upper_limit"  value="${115.0 * deg_to_rad}"/>

Commit message: Fix CoM for arm_right_1_link

File: ari_description/urdf/arm/arm_v2.urdf.xacro (robot description, xacro)
@@ -75,5 +75,5 @@
     <link name="${name}_${side}_1_link">
       <inertial>
-        <origin xyz="-0.00734678702660377 ${-2.69505911157866E-06 * reflect} 0.0810729999795757" rpy="0.0 0.0 0.0"/>
+        <origin xyz="${-0.00734678702660377*reflect} ${-2.69505911157866E-06 * reflect} 0.0810729999795757" rpy="0.0 0.0 0.0"/>
         <mass value="0.626384555512818" />
         <inertia

Commit message: Update limits

File: ari_description/urdf/arm/arm_v2.urdf.xacro (robot description, xacro)
@@ -26,13 +26,13 @@
   <xacro:property name="arm_1_lower_limit"  value="${-120.0 * deg_to_rad}"/>
   <xacro:property name="arm_1_upper_limit"  value="${120.0 * deg_to_rad}"/>
-  <xacro:property name="arm_2_lower_limit"  value="${1.0 * deg_to_rad}"/>
+  <xacro:property name="arm_2_lower_limit"  value="${0.0 * deg_to_rad}"/>
   <xacro:property name="arm_2_upper_limit"  value="${100.0 * deg_to_rad}"/>
   <xacro:property name="arm_3_lower_limit"  value="${-120.0 * deg_to_rad}"/>
   <xacro:property name="arm_3_upper_limit"  value="${120.0 * deg_to_rad}"/>
-  <xacro:property name="arm_4_lower_limit"  value="${1.0 * deg_to_rad}"/>
+  <xacro:property name="arm_4_lower_limit"  value="${0.0 * deg_to_rad}"/>
   <xacro:property name="arm_4_upper_limit"  value="${100.0 * deg_to_rad}"/>
-  <xacro:property name="arm_5_lower_limit"  value="${-115.0 * deg_to_rad}"/>
-  <xacro:property name="arm_5_upper_limit"  value="${115.0 * deg_to_rad}"/>
-  <xacro:property name="arm_eps"            value="0.07" />
+  <xacro:property name="arm_5_lower_limit"  value="${-120.0 * deg_to_rad}"/>
+  <xacro:property name="arm_5_upper_limit"  value="${120.0 * deg_to_rad}"/>
+  <xacro:property name="arm_eps"            value="0.05" />
   <xacro:macro name="ari_arm" params="name parent side reflect end_effector *origin">
     <!--************************-->
