Commit message: Added the head limit and the microphone urdf

File: ari_description/urdf/head/head.urdf.xacro (robot description, xacro)
@@ -22,5 +22,5 @@
   <xacro:property name="head_1_upper_limit" value="75"/>
   <xacro:property name="head_2_lower_limit" value="-15"/>
-  <xacro:property name="head_2_upper_limit" value="45"/>
+  <xacro:property name="head_2_upper_limit" value="35"/>
   <!--************************-->
   <!--     HEAD_1 (PAN)       -->
@@ -111,11 +111,4 @@
                          soft_upper_limit="${head_2_upper_limit * deg_to_rad}" />
     </joint>
-    <!--gazebo reference="${name}_link">
-      <mu1>0.9</mu1>
-      <mu2>0.9</mu2>
-    </gazebo>
-    <gazebo reference="${name}_joint">
-       <implicitSpringDamper>1</implicitSpringDamper>
-    </gazebo-->
     <xacro:head_transmission name="${name}" reduction="1" offset_value="${head_2_joint_offset}"/>
   </xacro:macro>

File: ari_description/urdf/torso/torso_sensors.urdf.xacro (robot description, xacro)
@@ -12,5 +12,5 @@
   <xacro:include filename="$(find realsense_gazebo_plugin)/urdf/d435.urdf.xacro" />
   <xacro:include filename="$(find realsense_gazebo_plugin)/urdf/t265.urdf.xacro" />
-  <!--xacro:include filename="$(find ari_description)/urdf/sensors/microphone.urdf.xacro"/-->
+  <xacro:include filename="$(find ari_description)/urdf/sensors/microphone.urdf.xacro"/>
   <!--xacro:include filename="$(find ari_description_calibration)/urdf/calibration/calibration_constants.urdf.xacro" /-->
   <!--Constant parameters-->
@@ -40,7 +40,7 @@
   </sensor_t265_gazebo>
   <!-- Microphones -->
-  <!--xacro:microphone name="${name}_mic_front" parent="${parent}">
-    <origin xyz="0.23182 0.03902 0.195" rpy="0 0 0"/>
-  </xacro:microphone-->
+  <xacro:microphone name="${name}_mic_front" parent="${parent}">
+    <origin xyz="-0.12173 -3.5497E-05 0.80332" rpy="${80 * deg_to_rad} 0 ${90 * deg_to_rad}"/>
+  </xacro:microphone>
  </xacro:macro>
 </robot>

Commit message: fix Raspi camera frame orientation

File: ari_description/urdf/head/head.urdf.xacro (robot description, xacro)
@@ -144,5 +144,5 @@
   </link>
   <joint name="${name}_joint" type="fixed">
-    <origin xyz="0.0633629998680001 0.181996035631448 0" rpy="${-90 * deg_to_rad} 0 0" />
+    <origin xyz="0.0633629998680001 0.181996035631448 0" rpy="${90 * deg_to_rad} ${-90 * deg_to_rad} ${90 * deg_to_rad}" />
     <parent link="${parent}" />
     <child link="${name}_link" />

Commit message: Revert "fix Raspi camera frame orientation"
This reverts commit 1b4612c5b6826d16f8e8d936be78decd74e0ae8a.

File: ari_description/urdf/head/head.urdf.xacro (robot description, xacro)
@@ -144,5 +144,5 @@
   </link>
   <joint name="${name}_joint" type="fixed">
-    <origin xyz="0.0633629998680001 0.181996035631448 0" rpy="${90 * deg_to_rad} ${-90 * deg_to_rad} ${90 * deg_to_rad}" />
+    <origin xyz="0.0633629998680001 0.181996035631448 0" rpy="${-90 * deg_to_rad} 0 0" />
     <parent link="${parent}" />
     <child link="${name}_link" />

Commit message: added head_front_camera_optic_frame

File: ari_description/urdf/head/head.urdf.xacro (robot description, xacro)
@@ -149,4 +149,11 @@
     <axis xyz="0 0 0" />
   </joint>
+  <joint name="${name}_optical_joint" type="fixed">
+    <origin xyz="0.0 0.0 0.0" rpy="${-90 * deg_to_rad} 0 ${-90 * deg_to_rad}" />
+    <parent link="${name}_link" />
+    <child link="${name}_optical_frame" />
+    <axis xyz="0 0 0" />
+  </joint>
+  <link name="${name}_optical_frame"/>
   <!-- Gazebo plugin -->
   <xacro:rpi_camera_gazebo name="${name}" topic="${name}"/>

Commit message: Update Rpi camera plugin to use the parsed frame

File: ari_description/urdf/head/head.urdf.xacro (robot description, xacro)
@@ -157,5 +157,5 @@
   <link name="${name}_optical_frame"/>
   <!-- Gazebo plugin -->
-  <xacro:rpi_camera_gazebo name="${name}" topic="${name}"/>
+  <xacro:rpi_camera_gazebo name="${name}" topic="${name}" frame="${name}_optical_frame"/>
   </xacro:macro>
   <xacro:macro name="head" params="name parent">

File: ari_description/urdf/sensors/rpi_camera.gazebo.xacro (robot description, xacro)
@@ -8,5 +8,5 @@
 -->
 <robot xmlns:xacro="http://ros.org/wiki/xacro">
-  <xacro:macro name="rpi_camera_gazebo" params="name:=camera topic:=camera">
+  <xacro:macro name="rpi_camera_gazebo" params="name:=camera topic:=camera frame:=camera_optic_frame">
     <gazebo reference="${name}_link">
       <sensor type="camera" name="${name}_pi_camera">
@@ -38,5 +38,5 @@
           <imageTopicName>image</imageTopicName>
           <cameraInfoTopicName>camera_info</cameraInfoTopicName>
-          <frameName>${name}_link</frameName>
+          <frameName>${frame}</frameName>
           <hackBaseline>0.07</hackBaseline>
           <distortionK1>0.00000001</distortionK1>

Commit message: Reduce head_2 upper limit to avoid collisions at head_1 limits

File: ari_description/urdf/head/head.urdf.xacro (robot description, xacro)
@@ -22,5 +22,5 @@
   <xacro:property name="head_1_upper_limit" value="75"/>
   <xacro:property name="head_2_lower_limit" value="-15"/>
-  <xacro:property name="head_2_upper_limit" value="35"/>
+  <xacro:property name="head_2_upper_limit" value="25"/>
   <!--************************-->
   <!--     HEAD_1 (PAN)       -->

Commit message: Modify URDF to include optional head realsense camera, location still to be defined

File: ari_description/urdf/head/head.urdf.xacro (robot description, xacro)
@@ -12,4 +12,5 @@
   <xacro:include filename="$(find ari_description)/urdf/head/head.transmission.xacro" />
   <xacro:include filename="$(find ari_description)/urdf/sensors/rpi_camera.gazebo.xacro" />
+  <xacro:include filename="$(find realsense2_description)/urdf/_d435.urdf.xacro" />
   <!--Constant parameters-->
   <xacro:property name="head_1_joint_offset" value="0.0" />
@@ -23,4 +24,11 @@
   <xacro:property name="head_2_lower_limit" value="-15"/>
   <xacro:property name="head_2_upper_limit" value="25"/>
+  <!--Constant parameters-->
+  <xacro:property name="head_realsense_camera_position_x" value="0.05215" />
+  <xacro:property name="head_realsense_camera_position_y" value="0.1675" />
+  <xacro:property name="head_realsense_camera_position_z" value="0.0" />
+  <xacro:property name="head_realsense_camera_orientation_r" value="${-90 * deg_to_rad}" />
+  <xacro:property name="head_realsense_camera_orientation_p" value="0.0" />
+  <xacro:property name="head_realsense_camera_orientation_y" value="0.0" />
   <!--************************-->
   <!--     HEAD_1 (PAN)       -->
@@ -120,4 +128,12 @@
   <!--      HEAD_CAMERA       -->
   <!--************************-->
+  <!-- Optional head realsense camera -->
+  <xacro:macro name="head_rgbd" params="name parent">
+    <sensor_d435 parent="head_2_link" name="head_front_camera" topics_ns="head_front_camera">
+      <origin xyz="${head_realsense_camera_position_x} ${head_realsense_camera_position_y} ${head_realsense_camera_position_z}"
+            rpy="${head_realsense_camera_orientation_r} ${head_realsense_camera_orientation_p} ${head_realsense_camera_orientation_y}"/>
+    </sensor_d435>
+  </xacro:macro>
+  <!-- Head RGB camera -->
   <xacro:macro name="head_front_camera" params="name parent">
   <link name="${name}_link">
@@ -149,11 +165,14 @@
     <axis xyz="0 0 0" />
   </joint>
-  <joint name="${name}_optical_joint" type="fixed">
+  <joint name="${name}_color_optical_joint" type="fixed">
     <origin xyz="0.0 0.0 0.0" rpy="${-90 * deg_to_rad} 0 ${-90 * deg_to_rad}" />
     <parent link="${name}_link" />
-    <child link="${name}_optical_frame" />
+    <child link="${name}_color_optical_frame" />
     <axis xyz="0 0 0" />
   </joint>
-  <link name="${name}_optical_frame"/>
+  <link name="${name}_color_optical_frame"/>
+  <!-- Gazebo plugin -->
+  <xacro:rpi_camera_gazebo name="${name}" topic="${name}/color" frame="${name}_color_optical_frame"/>
+  </xacro:macro>
   <joint name="ear_led_left_link" type="fixed">
     <origin xyz="0.021 0.095 0.192" rpy="-0.1 0 0.0" />
@@ -184,11 +203,13 @@
     </inertial>
   </link>
-  <!-- Gazebo plugin -->
-  <xacro:rpi_camera_gazebo name="${name}" topic="${name}" frame="${name}_optical_frame"/>
-  </xacro:macro>
   <xacro:macro name="head" params="name parent">
     <xacro:head_1 name="${name}_1" parent="${parent}" />
     <xacro:head_2 name="${name}_2" parent="${name}_1_link"/>
-    <xacro:head_front_camera name="${name}_front_camera" parent="${name}_2_link"/>
-  </xacro:macro>
+    <xacro:if value="${camera_model == 'head-rgb'}">
+      <xacro:head_front_camera name="${name}_front_camera" parent="${name}_2_link"/>
+    </xacro:if>
+    <xacro:if value="${camera_model == 'head-rgbd'}">
+      <xacro:head_rgbd name="${name}_rgbd" parent="${name}_2_link"/>
+    </xacro:if>
+ </xacro:macro>
 </robot>

Commit message: Fix urdf structure

File: ari_description/urdf/head/head.urdf.xacro (robot description, xacro)
@@ -175,4 +175,7 @@
   <xacro:rpi_camera_gazebo name="${name}" topic="${name}/color" frame="${name}_color_optical_frame"/>
   </xacro:macro>
+  <!-- Gazebo plugin -->
+  <xacro:rpi_camera_gazebo name="${name}" topic="${name}" frame="${name}_optical_frame"/>
+  </xacro:macro>
   <joint name="ear_led_left_link" type="fixed">
     <origin xyz="0.021 0.095 0.192" rpy="-0.1 0 0.0" />

Commit message: Modify URDF for head camera and fix topic names

File: ari_description/urdf/head/head.urdf.xacro (robot description, xacro)
@@ -175,7 +175,4 @@
   <xacro:rpi_camera_gazebo name="${name}" topic="${name}/color" frame="${name}_color_optical_frame"/>
   </xacro:macro>
-  <!-- Gazebo plugin -->
-  <xacro:rpi_camera_gazebo name="${name}" topic="${name}" frame="${name}_optical_frame"/>
-  </xacro:macro>
   <joint name="ear_led_left_link" type="fixed">
     <origin xyz="0.021 0.095 0.192" rpy="-0.1 0 0.0" />

Commit message: added frames for eyes of ari

File: ari_description/urdf/head/head.urdf.xacro (robot description, xacro)
@@ -238,4 +238,23 @@
     </inertial>
   </link>
+   <!-- EYE FRAMES -->
+  <link name="sellion_link"/>
+  <joint name="sellion_joint" type="fixed">
+    <origin xyz="0.04 0.09205 0" rpy="0 0 0"/>
+    <child link="sellion_link" />
+    <parent link="head_2_link"/>
+  </joint>
+  <link name="right_eye_link"/>
+  <joint name="right_eye_joint" type="fixed">
+    <origin xyz="0.0 0 0.0344 " rpy="0 0 0"/>
+    <child link="right_eye_link" />
+    <parent link="sellion_link"/>
+  </joint>
+  <link name="left_eye_link"/>
+  <joint name="left_eye_joint" type="fixed">
+    <origin xyz="0 0 -0.0344 " rpy="0 0 0"/>
+    <child link="left_eye_link" />
+    <parent link="sellion_link"/>
+  </joint>
   <xacro:macro name="head" params="name parent robot_model">
     <xacro:head_1 name="${name}_1" parent="${parent}" robot_model="${robot_model}" />

Commit message: Change link names and z-axis pointing up now

File: ari_description/urdf/head/head.urdf.xacro (robot description, xacro)
@@ -239,20 +239,21 @@
   </link>
    <!-- EYE FRAMES -->
+  <!-- Eyes are located 3cm behind the screen-->
   <link name="sellion_link"/>
   <joint name="sellion_joint" type="fixed">
-    <origin xyz="0.04 0.09205 0" rpy="0 0 0"/>
+    <origin xyz="0.04 0.09205 0" rpy="${-90 * deg_to_rad} 0 0"/>
     <child link="sellion_link" />
     <parent link="head_2_link"/>
   </joint>
-  <link name="right_eye_link"/>
-  <joint name="right_eye_joint" type="fixed">
-    <origin xyz="0.0 0 0.0344 " rpy="0 0 0"/>
-    <child link="right_eye_link" />
+  <link name="eye_right_link"/>
+  <joint name="eye_right_joint" type="fixed">
+    <origin xyz="0.0 0.0344 0" rpy="0 0 0"/>
+    <child link="eye_right_link" />
     <parent link="sellion_link"/>
   </joint>
-  <link name="left_eye_link"/>
-  <joint name="left_eye_joint" type="fixed">
-    <origin xyz="0 0 -0.0344 " rpy="0 0 0"/>
-    <child link="left_eye_link" />
+  <link name="eye_left_link"/>
+  <joint name="eye_left_joint" type="fixed">
+    <origin xyz="0 -0.0344 0" rpy="0 0 0"/>
+    <child link="eye_left_link" />
     <parent link="sellion_link"/>
   </joint>

Commit message: Change path for hokuyo and lidar sensors

File: ari_description/urdf/head/head.urdf.xacro (robot description, xacro)
@@ -10,5 +10,5 @@
   <!--File includes-->
   <xacro:include filename="$(find ari_description)/urdf/deg_to_rad.xacro" />
-  <xacro:include filename="$(find ari_description)/urdf/sensors/rpi_camera.gazebo.xacro" />
+  <xacro:include filename="$(find pal_urdf_utils)/urdf/sensors/ari/rpi_camera.gazebo.xacro" />
 <!-- TODO ROS2; disabled until realsense camera available
     <xacro:include filename="$(find realsense2_description)/urdf/_d435.urdf.xacro" />
@@ -171,5 +171,5 @@
       <origin rpy="0 0 0" xyz="0 0 0" />
       <geometry>
-        <mesh filename="package://ari_description/meshes/sensors/${name}.stl" scale="1 1 1"/>
+        <mesh filename="$(find pal_urdf_utils)/meshes/sensors/ari/${name}.stl" scale="1 1 1"/>
       </geometry>
       <material name="DarkGrey"/>
@@ -178,5 +178,5 @@
       <origin rpy="0 0 0" xyz="0 0 0" />
       <geometry>
-        <mesh filename="package://ari_description/meshes/sensors/${name}.stl" scale="1 1 1"/>
+        <mesh filename="$(find pal_urdf_utils)/meshes/sensors/ari/${name}.stl" scale="1 1 1"/>
       </geometry>
     </collision>

File: ari_description/urdf/torso/torso_sensors.urdf.xacro (robot description, xacro)
@@ -14,9 +14,9 @@
   <xacro:include filename="$(find realsense2_description)/urdf/_t265.urdf.xacro" />
 -->
-  <xacro:include filename="$(find ari_description)/urdf/sensors/microphone.urdf.xacro"/>
-  <xacro:include filename="$(find ari_description)/urdf/sensors/imx179_camera.gazebo.xacro"/>
-  <xacro:include filename="$(find pmb2_description)/urdf/sensors/sick_tim571_laser.urdf.xacro"/>
-  <xacro:include filename="$(find ari_description)/urdf/sensors/ydlidar_tg30_laser.urdf.xacro"/>
-  <xacro:include filename="$(find ari_description)/urdf/sensors/ydlidar_tg15_laser.urdf.xacro"/>
+  <xacro:include filename="$(find pal_urdf_utils)/urdf/sensors/microphone.urdf.xacro"/>
+  <xacro:include filename="$(find pal_urdf_utils)/urdf/sensors/ari/imx179_camera.gazebo.xacro"/>
+  <xacro:include filename="$(find pal_urdf_utils)/urdf/sensors/bases/sick_tim571_laser.urdf.xacro"/>
+  <xacro:include filename="$(find pal_urdf_utils)/urdf/sensors/ari/ydlidar_tg30_laser.urdf.xacro"/>
+  <xacro:include filename="$(find pal_urdf_utils)/urdf/sensors/ari/ydlidar_tg15_laser.urdf.xacro"/>
   <xacro:macro name="torso_sensors" params="name parent robot_model use_nominal_extrinsics laser_model">
     <xacro:if value="${robot_model == 'v1'}">

Commit message: Change path for camera meshes

File: ari_description/urdf/head/head.urdf.xacro (robot description, xacro)
@@ -171,5 +171,5 @@
       <origin rpy="0 0 0" xyz="0 0 0" />
       <geometry>
-        <mesh filename="$(find pal_urdf_utils)/meshes/sensors/ari/${name}.stl" scale="1 1 1"/>
+        <mesh filename="$(find pal_urdf_utils)/meshes/camera/${name}.stl" scale="1 1 1"/>
       </geometry>
       <material name="DarkGrey"/>
@@ -178,5 +178,5 @@
       <origin rpy="0 0 0" xyz="0 0 0" />
       <geometry>
-        <mesh filename="$(find pal_urdf_utils)/meshes/sensors/ari/${name}.stl" scale="1 1 1"/>
+        <mesh filename="$(find pal_urdf_utils)/meshes/camera/${name}.stl" scale="1 1 1"/>
       </geometry>
     </collision>

Commit message: Fix meshes paths

File: ari_description/urdf/head/head.urdf.xacro (robot description, xacro)
@@ -169,5 +169,5 @@
       <origin rpy="0 0 0" xyz="0 0 0" />
       <geometry>
-        <mesh filename="$(find pal_urdf_utils)/meshes/camera/${name}.stl" scale="1 1 1"/>
+        <mesh filename="package://pal_urdf_utils/meshes/camera/${name}.stl" scale="1 1 1"/>
       </geometry>
       <material name="DarkGrey"/>
@@ -176,5 +176,5 @@
       <origin rpy="0 0 0" xyz="0 0 0" />
       <geometry>
-        <mesh filename="$(find pal_urdf_utils)/meshes/camera/${name}.stl" scale="1 1 1"/>
+        <mesh filename="package://pal_urdf_utils/meshes/camera/${name}.stl" scale="1 1 1"/>
       </geometry>
     </collision>

Commit message: Rotate head 2 limiits

File: ari_description/urdf/head/head.urdf.xacro (robot description, xacro)
@@ -21,6 +21,6 @@
   <xacro:property name="head_1_lower_limit" value="-75"/>
   <xacro:property name="head_1_upper_limit" value="75"/>
-  <xacro:property name="head_2_lower_limit" value="-15"/>
-  <xacro:property name="head_2_upper_limit" value="25"/>
+  <xacro:property name="head_2_lower_limit" value="-25"/>
+  <xacro:property name="head_2_upper_limit" value="15"/>
   <!--Constant parameters-->
   <xacro:property name="head_realsense_camera_position_x" value="0.05215" />
