Commit message: update and delete xacro files

File: ari_description/urdf/base/base_v2.urdf.xacro (robot description, xacro)
@@ -119,10 +119,3 @@
     <origin xyz="-0.600830 0 0.039" rpy="0 0 0" />
   </xacro:docking_link>
-<!--   <xacro:torso_rgbd name="torso_rgbd">
-    <origin xyz="-0.13799 -0.00034911 1.0305" rpy="0 0.75049 0" />
-  </xacro:torso_rgbd>
-  <xacro:torso_265 name="torso_265">
-    <origin xyz="-0.31955 0.009 1.0599" rpy="0 0.2618 3.1416" />
-  </xacro:torso_265>
- -->
 </robot>

File: ari_description/urdf/head/head_v2.urdf.xacro (robot description, xacro)
@@ -10,5 +10,5 @@
   <!--File includes-->
   <xacro:include filename="$(find ari_description)/urdf/deg_to_rad.xacro" />
-  <xacro:include filename="$(find ari_description)/urdf/head/head_v2.transmission.xacro" />
+  <xacro:include filename="$(find ari_description)/urdf/head/head.transmission.xacro" />
   <xacro:include filename="$(find ari_description)/urdf/sensors/rpi_camera.gazebo.xacro" />
   <xacro:include filename="$(find realsense2_description)/urdf/_d435.urdf.xacro" />

File: ari_description/urdf/wheels/caster_v2.urdf.xacro (robot description, xacro)
@@ -8,5 +8,5 @@
 -->
 <robot xmlns:xacro="http://ros.org/wiki/xacro">
-  <xacro:include filename="$(find ari_description)/urdf/wheels/caster_v2.gazebo.xacro"/>
+  <xacro:include filename="$(find ari_description)/urdf/wheels/caster.gazebo.xacro"/>
   <xacro:macro name="caster" params="side reflect radius width separation_x offset_y offset_z parent">
     <link name="caster_${side}_link">
@@ -28,5 +28,5 @@
         <origin xyz="0 0 0" rpy="0 0 0"/>
         <geometry>
-          <cylinder radius="${radius}" length="${width}"/>
+          <mesh filename="package://ari_description/meshes/wheels/caster_v2.stl" scale="1 ${reflect} 1"/>
         </geometry>
       </collision>

File: ari_description/urdf/wheels/wheel_v2.urdf.xacro (robot description, xacro)
@@ -22,5 +22,5 @@
         <origin xyz="0 0 0" rpy="0 0 0"/>
         <geometry>
-        <mesh filename="package://ari_description/meshes/wheels/wheel_${side}_v2.stl"/>
+          <mesh filename="package://ari_description/meshes/wheels/wheel_${side}_v2.stl"/>
         </geometry>
         <material name="White"/>
@@ -29,5 +29,5 @@
         <origin xyz="0 0 0" rpy="0 0 0"/>
         <geometry>
-          <cylinder radius="${radius}" length="${width}"/>
+          <mesh filename="package://ari_description/meshes/wheels/wheel_${side}_v2.stl"/>
         </geometry>
       </collision>
