Commit message: Remove docking and head base stl to avoid collision errors

File: ari_description/urdf/base/docking_link_v2.urdf.xacro (robot description, xacro)
@@ -17,5 +17,5 @@
                    iyy="2.2318E-05" iyz="1.0152E-09" izz="3.4652E-05" />
       </inertial>
-      <visual>
+<!--       <visual>
         <origin xyz="0 0 0" rpy="0 0 0" />
         <geometry>
@@ -31,5 +31,5 @@
           <mesh filename="package://ari_description/meshes/base/docking_joint_v2.stl" />
         </geometry>
-      </collision>
+      </collision>       -->
   </link>
   <joint name="${name}_joint" type="fixed">

File: ari_description/urdf/head/head_v2.urdf.xacro (robot description, xacro)
@@ -43,5 +43,5 @@
                izz="0.000359230346366051" />
     </inertial>
-    <visual>
+<!--     <visual>
       <origin xyz="0 0 0" rpy="0 0 0" />
       <geometry>
@@ -57,5 +57,5 @@
           <mesh filename="package://ari_description/meshes/head/head_base_v2.stl" scale="1 1 1"/>
       </geometry>
-    </collision>
+    </collision> -->
   </link>
   <joint name="${name}_joint" type="fixed">

Commit message: Update collision geometry for docking link

File: ari_description/urdf/base/docking_link_v2.urdf.xacro (robot description, xacro)
@@ -8,4 +8,7 @@
 -->
 <robot xmlns:xacro="http://ros.org/wiki/xacro">
+  <xacro:include filename="$(find ari_description)/urdf/deg_to_rad.xacro" />
+  <xacro:property name="docking_radius"     value="0.045"/>
+  <xacro:property name="docking_width"      value="0.01"/>
   <xacro:macro name="docking_link" params="name *origin">
   <!-- Docking Link -->
@@ -17,5 +20,5 @@
                    iyy="2.2318E-05" iyz="1.0152E-09" izz="3.4652E-05" />
       </inertial>
-<!--       <visual>
+      <visual>
         <origin xyz="0 0 0" rpy="0 0 0" />
         <geometry>
@@ -27,9 +30,9 @@
       </visual>
       <collision>
-        <origin xyz="0 0 0" rpy="0 0 0" />
+        <origin xyz="0 0 0" rpy="0 ${90 * deg_to_rad} 0"/>
         <geometry>
-          <mesh filename="package://ari_description/meshes/base/docking_joint_v2.stl" />
+          <cylinder radius="${docking_radius}" length="${docking_width}"/>
         </geometry>
-      </collision>       -->
+      </collision>
   </link>
   <joint name="${name}_joint" type="fixed">
