Commit message: Created the bringup and the controller configuration and added the t265 camera to the back of the torso

File: ari_description/urdf/base/base.urdf.xacro (robot description, xacro)
@@ -13,14 +13,10 @@
   <!--xacro:include filename="$(find ari_description)/urdf/sensors/microphone.urdf.xacro"/-->
   <!-- Wheel characteristics -->
-  <xacro:property name="wheel_radius"     value="0.0"/>
-  <xacro:property name="wheel_width"     value="0.0"/>
-  <xacro:property name="wheel_torque"     value="0.0"/>
-  <xacro:property name="wheel_velocity"     value="0.0"/>
-  <!--xacro:property name="wheel_radius"     value="0.101"/>
+  <xacro:property name="wheel_radius"     value="0.101"/>
   <xacro:property name="wheel_width"      value="0.040"/>
   <xacro:property name="wheel_separation" value="0.4554"/>
   <xacro:property name="wheel_pair_separation" value="0.420"/>
   <xacro:property name="wheel_torque"     value="6.0"/>
-  <xacro:property name="wheel_velocity"   value="1.0"/-->
+  <xacro:property name="wheel_velocity"   value="1.0"/>
   <xacro:macro name="base" params="name">
   <!-- Base -->

File: ari_description/urdf/head/head.urdf.xacro (robot description, xacro)
@@ -14,5 +14,5 @@
   <xacro:property name="head_1_joint_offset" value="0.0" />
   <xacro:property name="head_2_joint_offset" value="0.0" />
-  <!--xacro:property name="head_friction" value="1.0" />
+  <xacro:property name="head_friction" value="1.0" />
   <xacro:property name="head_damping"  value="0.5" />
   <xacro:property name="head_max_vel"  value="3.0" />
@@ -20,6 +20,6 @@
   <xacro:property name="head_1_lower_limit" value="-75"/>
   <xacro:property name="head_1_upper_limit" value="75"/>
-  <xacro:property name="head_2_lower_limit" value="-60"/>
-  <xacro:property name="head_2_upper_limit" value="45"/-->
+  <xacro:property name="head_2_lower_limit" value="-20"/>
+  <xacro:property name="head_2_upper_limit" value="45"/>
   <!--************************-->
   <!--     HEAD_1 (PAN)       -->
@@ -54,11 +54,10 @@
       <origin xyz="0 0 0"  rpy="0 0 0" />
       <axis xyz="0 0 1" />
-      <limit lower="0" upper="0" effort="0" velocity="0" />
-      <!--limit lower="${head_1_lower_limit * deg_to_rad}" upper="${head_1_upper_limit * deg_to_rad}" effort="5.197" velocity="${head_max_vel}" /-->
-      <!--dynamics damping="${head_damping}" friction="${head_friction}"/-->
-      <!--safety_controller k_position="20"
+      <limit lower="${head_1_lower_limit * deg_to_rad}" upper="${head_1_upper_limit * deg_to_rad}" effort="5.197" velocity="${head_max_vel}" />
+      <dynamics damping="${head_damping}" friction="${head_friction}"/>
+      <safety_controller k_position="20"
                          k_velocity="20"
                          soft_lower_limit="${head_1_lower_limit * deg_to_rad + head_eps}"
-                         soft_upper_limit="${head_1_upper_limit * deg_to_rad - head_eps}" /-->
+                         soft_upper_limit="${head_1_upper_limit * deg_to_rad - head_eps}" />
     </joint>
     <gazebo reference="${name}_link">
@@ -104,12 +103,18 @@
       <origin xyz="-0.183 0 1.2845"  rpy="${90.0 * deg_to_rad} 0 0" />
       <axis xyz="0 0 -1" />
-      <limit lower="0" upper="0" effort="0" velocity="0" />
-      <!--limit lower="${head_2_lower_limit * deg_to_rad}" upper="${head_2_upper_limit * deg_to_rad}" effort="2.77" velocity="${head_max_vel}" /-->
-      <!--dynamics damping="${head_damping}" friction="${head_friction}"/-->
-      <!--safety_controller k_position="20"
+      <limit lower="${head_2_lower_limit * deg_to_rad}" upper="${head_2_upper_limit * deg_to_rad}" effort="2.77" velocity="${head_max_vel}" />
+      <dynamics damping="${head_damping}" friction="${head_friction}"/>
+      <safety_controller k_position="20"
                          k_velocity="20"
                          soft_lower_limit="${head_2_lower_limit * deg_to_rad + head_eps}"
-                         soft_upper_limit="${head_2_upper_limit * deg_to_rad}" /-->
+                         soft_upper_limit="${head_2_upper_limit * deg_to_rad}" />
     </joint>
+    <!--gazebo reference="${name}_link">
+      <mu1>0.9</mu1>
+      <mu2>0.9</mu2>
+    </gazebo>
+    <gazebo reference="${name}_joint">
+       <implicitSpringDamper>1</implicitSpringDamper>
+    </gazebo-->
     <xacro:head_transmission name="${name}" reduction="1" offset_value="${head_2_joint_offset}"/>
   </xacro:macro>

File: ari_description/urdf/torso/torso_sensors.urdf.xacro (robot description, xacro)
@@ -11,4 +11,5 @@
   <xacro:include filename="$(find ari_description)/urdf/deg_to_rad.xacro" />
   <xacro:include filename="$(find realsense_gazebo_plugin)/urdf/d435.urdf.xacro" />
+  <xacro:include filename="$(find realsense_gazebo_plugin)/urdf/t265.urdf.xacro" />
   <!--xacro:include filename="$(find ari_description_calibration)/urdf/calibration/calibration_constants.urdf.xacro" /-->
   <!--Constant parameters-->
@@ -19,4 +20,10 @@
   <xacro:property name="torso_front_camera_orientation_p" value="${42.5 * deg_to_rad}" />
   <xacro:property name="torso_front_camera_orientation_y" value="0.0" />
+  <xacro:property name="torso_back_camera_position_x" value="-0.3275" />
+  <xacro:property name="torso_back_camera_position_y" value="0.009" />
+  <xacro:property name="torso_back_camera_position_z" value="1.0337" />
+  <xacro:property name="torso_back_camera_orientation_r" value="${75 * deg_to_rad}" />
+  <xacro:property name="torso_back_camera_orientation_p" value="0.0" />
+  <xacro:property name="torso_back_camera_orientation_y" value="${90 * deg_to_rad}" />
   <xacro:macro name="torso_sensors" params="name parent">
   <!-- Torso sensors -->
@@ -27,5 +34,9 @@
   </sensor_d435_gazebo>
   <!-- Torso back camera -->
-  <link name="${name}_camera_2_link">
+  <sensor_t265_gazebo parent="${parent}" name="${name}_back_camera" topics_ns="${name}_back_camera">
+    <origin xyz="${torso_back_camera_position_x} ${torso_back_camera_position_y} ${torso_back_camera_position_z}"
+            rpy="${torso_back_camera_orientation_r} ${torso_back_camera_orientation_p} ${torso_back_camera_orientation_y}"/>
+  </sensor_t265_gazebo>
+  <!--link name="${name}_camera_2_link">
     <inertial>
       <origin xyz="0 0 0" rpy="0 0 0"/>
@@ -54,5 +65,5 @@
     <child link="${name}_camera_2_link" />
     <axis xyz="0 0 0" />
-  </joint>
+  </joint-->
  </xacro:macro>
 </robot>

Commit message: Added the caster wheels, modified the urdf files, fixed the problem with the head_1_joint, added the head_camera

File: ari_description/urdf/base/base.urdf.xacro (robot description, xacro)
@@ -21,20 +21,18 @@
   <xacro:property name="wheel_velocity"   value="1.0"/>
   <!-- Caster wheel characteristics -->
-  <xacro:property name="caster_radius"       value="0.025"/>
-  <xacro:property name="caster_width"        value="0.015"/>
-  <xacro:property name="caster_separation_x" value="0.343"/>
-  <xacro:property name="caster_separation_y" value="0.204"/>
-  <xacro:property name="caster_offset_x"     value="-0.002"/>
-  <xacro:property name="caster_offset_y"     value="0.0"/>
-  <xacro:property name="caster_offset_z"     value="-0.0335"/>
+  <xacro:property name="caster_radius"       value="0.045"/>
+  <xacro:property name="caster_width"        value="0.055"/>
+  <xacro:property name="caster_separation_x" value="0.91"/>
+  <xacro:property name="caster_separation_y" value="0.205"/>
+  <xacro:property name="caster_offset_z"     value="-0.08"/>
   <xacro:macro name="base" params="name">
   <!-- Base -->
   <link name="${name}_link">
     <inertial>
-      <origin xyz="-0.1896 -0.003234 0.27382" rpy="0 0 0"/>
-      <mass value="43.891"/>
-      <inertia ixx="0.71827" ixy="-7.1158E-05" ixz="0.054913"
-               iyy="0.74483" iyz="-9.085E-06"
-               izz="0.45676"/>
+      <origin xyz="-0.18664 -0.0032701 0.2776" rpy="0 0 0"/>
+      <mass value="43.407"/>
+      <inertia ixx="0.71785" ixy="-7.1158E-05" ixz="0.054913"
+               iyy="0.74432" iyz="-9.0871E-06"
+               izz="0.45635"/>
     </inertial>
     <visual>
@@ -78,6 +76,8 @@
   <xacro:wheel side="left"  reflect="-1.0" radius="${wheel_radius}" width="${wheel_width}" torque="${wheel_torque}" velocity="${wheel_velocity}" separation="${wheel_separation}" parent="${name}"/>
   <!-- Casters wheels -->
-  <!--xacro:caster side="back_right"  radius="${caster_radius}" width="${caster_width}" separation_x="${-caster_separation_x}" separation_y="${ caster_separation_y}" offset_x="${caster_offset_x}" offset_y="${caster_offset_y}" offset_z="${caster_offset_z}" parent="${name}"/>
-  <xacro:caster side="back_left"   radius="${caster_radius}" width="${caster_width}" separation_x="${-caster_separation_x}" separation_y="${-caster_separation_y}" offset_x="${caster_offset_x}" offset_y="${caster_offset_y}" offset_z="${caster_offset_z}" parent="${name}"/-->
+  <xacro:caster side="right" reflect=" 1.0" radius="${caster_radius}" width="${caster_width}" separation_x="${caster_separation_x}" separation_y="${caster_separation_y}"
+                offset_z="${caster_offset_z}" parent="${name}"/>
+  <xacro:caster side="left"  reflect="-1.0" radius="${caster_radius}" width="${caster_width}" separation_x="${caster_separation_x}" separation_y="${caster_separation_y}"
+                offset_z="${caster_offset_z}" parent="${name}"/>
   </xacro:macro>
 </robot>

File: ari_description/urdf/head/head.urdf.xacro (robot description, xacro)
@@ -29,5 +29,5 @@
     <link name="${name}_link">
       <inertial>
-        <origin xyz="-0.21358 0.00089501 1.2715" rpy="0 0 0"/>
+        <origin xyz="0.011917 0.00089501 0.08" rpy="0 0 0"/>
         <mass value="0.35824"/>
         <inertia ixx="0.00038949" ixy="-2.99E-07" ixz="-1.0058E-05"
@@ -53,5 +53,5 @@
       <parent link="${parent}"/>
       <child link="${name}_link"/>
-      <origin xyz="0 0 0"  rpy="0 0 0" />
+      <origin xyz="-0.2255 0 1.1915"  rpy="0 0 0" />
       <axis xyz="0 0 1" />
       <limit lower="${head_1_lower_limit * deg_to_rad}" upper="${head_1_upper_limit * deg_to_rad}" effort="5.197" velocity="${head_max_vel}" />
@@ -78,9 +78,9 @@
     <link name="${name}_link">
       <inertial>
-        <origin xyz="-0.0069656 0.102 -0.00084474" rpy="0 0 0"/>
+        <origin xyz="-0.00696564558843529 0.101996367574138 -0.0008447177604265" rpy="0 0 0"/>
         <mass value="0.87177"/>
-        <inertia ixx="0.0034812" ixy="-0.00057471" ixz="3.5243E-08"
-                 iyy="0.0023942" iyz="2.1773E-07"
-                 izz="0.0029851"/>
+        <inertia ixx="0.00348124070979026" ixy="-0.000574703524917147" ixz="3.53158443864736E-08"
+                 iyy="0.0023941695403699" iyz="2.1916879659837E-07"
+                 izz="0.00298511989538667"/>
       </inertial>
       <visual>
@@ -102,5 +102,5 @@
       <parent link="${parent}"/>
       <child link="${name}_link"/>
-      <origin xyz="-0.183 0 1.2845"  rpy="${90.0 * deg_to_rad} 0 0" />
+      <origin xyz="0.0425000000000001 0 0.093"  rpy="${90.0 * deg_to_rad} 0 0" />
       <axis xyz="0 0 -1" />
       <limit lower="${head_2_lower_limit * deg_to_rad}" upper="${head_2_upper_limit * deg_to_rad}" effort="2.77" velocity="${head_max_vel}" />
@@ -120,7 +120,41 @@
     <xacro:head_transmission name="${name}" reduction="1" offset_value="${head_2_joint_offset}"/>
   </xacro:macro>
+  <!--************************-->
+  <!--      HEAD_CAMERA       -->
+  <!--************************-->
+  <xacro:macro name="head_camera" params="name parent">
+  <link name="${name}_link">
+    <inertial>
+      <origin xyz="-0.00619317919404934 -4.45435622691566E-05 -8.22112600169511E-05" rpy="0 0 0"/>
+      <mass value="0.00115745344894968"/>
+      <inertia ixx="6.76913771029748E-08" ixy="2.52492243040059E-13" ixz="-3.60412180500293E-11"
+               iyy="2.88827920072855E-08" iyz="-1.65336506314803E-13"
+               izz="3.97290092554434E-08"/>
+    </inertial>
+    <visual>
+      <origin rpy="0 0 0" xyz="0 0 0" />
+      <geometry>
+        <mesh filename="package://ari_description/meshes/sensors/${name}.stl" scale="1 1 1"/>
+      </geometry>
+      <material name="DarkGrey"/>
+    </visual>
+    <collision>
+      <origin rpy="0 0 0" xyz="0 0 0" />
+      <geometry>
+        <mesh filename="package://ari_description/meshes/sensors/${name}.stl" scale="1 1 1"/>
+      </geometry>
+    </collision>
+  </link>
+  <joint name="${name}_joint" type="fixed">
+    <origin xyz="0.0633629998680001 0.181996035631448 0" rpy="${-90 * deg_to_rad} 0 0" />
+    <parent link="${parent}" />
+    <child link="${name}_link" />
+    <axis xyz="0 0 0" />
+  </joint>
+  </xacro:macro>
   <xacro:macro name="head" params="name parent">
     <xacro:head_1 name="${name}_1" parent="${parent}" />
     <xacro:head_2 name="${name}_2" parent="${name}_1_link"/>
+    <xacro:head_camera name="${name}_camera" parent="${name}_2_link"/>
   </xacro:macro>
 </robot>

File: ari_description/urdf/torso/torso_sensors.urdf.xacro (robot description, xacro)
@@ -38,32 +38,4 @@
             rpy="${torso_back_camera_orientation_r} ${torso_back_camera_orientation_p} ${torso_back_camera_orientation_y}"/>
   </sensor_t265_gazebo>
-  <!--link name="${name}_camera_2_link">
-    <inertial>
-      <origin xyz="0 0 0" rpy="0 0 0"/>
-      <mass value="0"/>
-      <inertia ixx="0" ixy="0" ixz="0"
-               iyy="0" iyz="0"
-               izz="0"/>
-    </inertial>
-    <visual>
-      <origin rpy="0 0 0" xyz="0 0 0" />
-      <geometry>
-        <mesh filename="package://ari_description/meshes/sensors/${name}_camera_2.stl" scale="1 1 1"/>
-      </geometry>
-      <material name="White"/>
-    </visual>
-    <collision>
-      <origin rpy="0 0 0" xyz="0 0 0" />
-      <geometry>
-        <mesh filename="package://ari_description/meshes/sensors/${name}_camera_2.stl" scale="1 1 1"/>
-      </geometry>
-    </collision>
-  </link>
-  <joint name="${name}_camera_2_joint" type="fixed">
-    <origin rpy="0 0.26179938779914 -3.14159265358979" xyz="-0.327497577576678 0.00899999999999999 1.03369506830427" />
-    <parent link="${parent}" />
-    <child link="${name}_camera_2_link" />
-    <axis xyz="0 0 0" />
-  </joint-->
  </xacro:macro>
 </robot>

File: ari_description/urdf/wheels/caster.urdf.xacro (robot description, xacro)
@@ -9,41 +9,19 @@
 <robot xmlns:xacro="http://ros.org/wiki/xacro">
   <xacro:include filename="$(find ari_description)/urdf/wheels/caster.gazebo.xacro"/>
-  <xacro:macro name="caster" params="side radius width separation_x separation_y offset_x offset_y offset_z parent">
-    <link name="caster_${side}_1_link">
+  <xacro:macro name="caster" params="side reflect radius width separation_x separation_y offset_z parent">
+    <link name="caster_${side}_link">
       <inertial>
-        <origin xyz="-0.00634599 0.00005347 -0.02037519" rpy="0 0 0"/>
-        <mass value="0.05144761"/>
-        <inertia  ixx="0.00001513" ixy="-0.00000003" ixz="0.00000267"
-                  iyy="0.00001309" iyz="-0.00000005"
-                  izz="0.00001198"/>
+        <origin xyz="${1.4445E-06 * reflect} 0.016213 ${-0.00019766 * reflect}" rpy="0 0 0"/>
+        <mass value="0.24242"/>
+        <inertia  ixx="0.0002099" ixy="${-5.5806E-09 * reflect}" ixz="-6.9375E-11"
+                  iyy="0.00020239" iyz="${-2.6771E-09 * reflect}"
+                  izz="0.00025496"/>
       </inertial>
       <visual>
         <origin xyz="0 0 0" rpy="0 0 0"/>
         <geometry>
-          <mesh filename="package://ari_description/meshes/wheels/caster_1.stl"/>
+          <mesh filename="package://ari_description/meshes/wheels/caster_${side}.stl"/>
         </geometry>
         <material name="Grey"/>
-      </visual>
-      <!--collision>
-        <origin xyz="0 0 0" rpy="0 0 0"/>
-        <geometry>
-          <cylinder radius="${radius}" length="${width}"/>
-        </geometry>
-      </collision-->
-    </link>
-    <link name="caster_${side}_2_link">
-      <inertial>
-        <origin xyz="0 0 0" rpy="0 0 0"/>
-        <mass value="0.08855784"/>
-        <inertia  ixx="0.00001075" ixy="0" ixz="0"
-                  iyy="0.00001541" iyz="0"
-                  izz="0.00001075"/>
-        </inertial>
-      <visual>
-        <origin xyz="0 0 0" rpy="0 0 0"/>
-        <geometry>
-          <mesh filename="package://pmb2_description/meshes/wheels/caster_2.stl"/>
-        </geometry>
-        <material name="DarkGrey"/>
       </visual>
       <collision>
@@ -54,16 +32,10 @@
       </collision>
     </link>
-    <joint name="caster_${side}_1_joint" type="continuous">
+    <joint name="caster_${side}_joint" type="continuous">
       <parent link="${parent}_link"/>
-      <child link="caster_${side}_1_link"/>
-      <origin xyz="${offset_x + separation_x / 2} ${offset_y - separation_y / 2} ${offset_z}" rpy="0 0 0"/>
-      <axis xyz="0 0 1"/>
+      <child link="caster_${side}_link"/>
+      <origin xyz="${-separation_x / 2} ${-separation_y / 2 * reflect} ${offset_z}" rpy="${90.0 * deg_to_rad} 0 0"/>
+      <axis xyz="0 0 -1"/>
       <dynamics damping="0.005" friction="0.0"/>
-    </joint>
-    <joint name="caster_${side}_2_joint" type="continuous">
-      <parent link="caster_${side}_1_link"/>
-      <child link="caster_${side}_2_link"/>
-      <origin xyz="-0.016 0.0000 -0.040" rpy="${-90.0 * deg_to_rad} 0 0"/>
-      <axis xyz="0 0 1"/>
     </joint>
     <!-- Gazebo extensions -->

File: ari_description/urdf/wheels/wheel.urdf.xacro (robot description, xacro)
@@ -13,9 +13,9 @@
     <link name="wheel_${side}_link">
       <inertial>
-        <origin xyz="-5.88442419331937E-06 -7.00561276577305E-05 ${-0.0022290297150058 * reflect}" rpy="0 0 0"/>
-        <mass value="1.65650861485769"/>
-        <inertia ixx="0.00630296404438552" ixy="1.03127988436767E-10" ixz="${-7.08413960046181E-07 * reflect}"
-                 iyy="0.00630218683572695" iyz="${-5.36273885065753E-08 * reflect}"
-                 izz="0.0111537170515013"/>
+        <origin xyz="-5.88525464208667E-06 -7.00561297658359E-05 ${-0.00222902971508132 * reflect}" rpy="0 0 0"/>
+        <mass value="1.65651"/>
+        <inertia ixx="0.00630296404438488" ixy="1.03273612245952E-10" ixz="${-7.08413602420107E-07 * reflect}"
+                 iyy="0.00630218683572781" iyz="${-5.36273874221441E-08 * reflect}"
+                 izz="0.0111537170515009"/>
       </inertial>
       <visual>

Commit message: move rgbd laser frame farther

File: ari_description/urdf/base/base.urdf.xacro (robot description, xacro)
@@ -83,5 +83,5 @@
       <parent link="base_link"/>
       <child link="rgbd_laser_link"/>
-      <origin xyz="-1 0 0" rpy="0 0 0" />
+      <origin xyz="-1.1 0 0" rpy="0 0 0" />
   </joint>
   <link name="rgbd_laser_link">

Commit message: Add Led frames

File: ari_description/urdf/base/base.urdf.xacro (robot description, xacro)
@@ -92,3 +92,17 @@
       </inertial>
   </link>
+  <joint name="back_led_link" type="fixed">
+    <origin xyz="-0.12 0.0 -0.08" rpy="0.0 0.2 1.57" />
+    <child link="back_led_frame" />
+    <parent link="head_1_link"/>
+  </joint>
+  <link name="back_led_frame">
+    <inertial>
+      <origin xyz="0 0 0" rpy="0 0 0" />
+      <mass value="0.001" /> <!-- matrix below must not be zero, or Gazebo won't load -->
+      <inertia ixx="0.0001" ixy="0.0" ixz="0.0"
+               iyy="0.000001" iyz="0.0"
+               izz="0.0001" />
+    </inertial>
+  </link>
 </robot>

File: ari_description/urdf/head/head.urdf.xacro (robot description, xacro)
@@ -156,4 +156,32 @@
   </joint>
   <link name="${name}_optical_frame"/>
+  <joint name="ear_led_left_link" type="fixed">
+    <origin xyz="0.021 0.095 0.192" rpy="-0.1 0 0.0" />
+    <child link="ear_led_left_frame" />
+    <parent link="head_1_link"/>
+  </joint>
+  <link name="ear_led_left_frame">
+    <inertial>
+      <origin xyz="0 0 0" rpy="0 0 0" />
+      <mass value="0.001" /> <!-- matrix below must not be zero, or Gazebo won't load -->
+      <inertia ixx="0.0001" ixy="0.0" ixz="0.0"
+               iyy="0.000001" iyz="0.0"
+               izz="0.0001" />
+    </inertial>
+  </link>
+  <joint name="ear_led_right_link" type="fixed">
+    <origin xyz="0.021 -0.095 0.192" rpy="-0.1 0.0 3.14" />
+    <child link="ear_led_right_frame" />
+    <parent link="head_1_link"/>
+  </joint>
+  <link name="ear_led_right_frame">
+    <inertial>
+      <origin xyz="0 0 0" rpy="0 0 0" />
+      <mass value="0.001" /> <!-- matrix below must not be zero, or Gazebo won't load -->
+      <inertia ixx="0.0001" ixy="0.0" ixz="0.0"
+               iyy="0.000001" iyz="0.0"
+               izz="0.0001" />
+    </inertial>
+  </link>
   <!-- Gazebo plugin -->
   <xacro:rpi_camera_gazebo name="${name}" topic="${name}" frame="${name}_optical_frame"/>

Commit message: Added fixed frame to the urdf with the position of the docking interface for the parking planner node

File: ari_description/urdf/base/base.urdf.xacro (robot description, xacro)
@@ -106,3 +106,16 @@
     </inertial>
   </link>
+  <!-- Docking Link -->
+  <joint name="docking_joint" type="fixed">
+      <parent link="base_link"/>
+      <child link="docking_link"/>
+      <origin xyz="-0.6 0 0" rpy="0 0 0" />
+  </joint>
+  <link name="docking_link">
+      <inertial>
+          <origin xyz="0 0 0" rpy="0 0 0"/>
+          <mass value="0.0001" />
+          <inertia ixx="0.0001"  ixy="0"  ixz="0" iyy="0.0001" iyz="0" izz="0.0001" />
+      </inertial>
+  </link>
 </robot>

Commit message: reduced a bit the docking frame in order to guarantee that the parking planner is alway able to park

File: ari_description/urdf/base/base.urdf.xacro (robot description, xacro)
@@ -110,5 +110,5 @@
       <parent link="base_link"/>
       <child link="docking_link"/>
-      <origin xyz="-0.6 0 0" rpy="0 0 0" />
+      <origin xyz="-0.57 0 0" rpy="0 0 0" />
   </joint>
   <link name="docking_link">

Commit message: Updated docking_link distance based on mechanical specifications

File: ari_description/urdf/base/base.urdf.xacro (robot description, xacro)
@@ -110,5 +110,5 @@
       <parent link="base_link"/>
       <child link="docking_link"/>
-      <origin xyz="-0.57 0 0" rpy="0 0 0" />
+      <origin xyz="-0.6 0 0" rpy="0 0 0" />
   </joint>
   <link name="docking_link">

Commit message: URDF distance accuracy

File: ari_description/urdf/base/base.urdf.xacro (robot description, xacro)
@@ -110,5 +110,5 @@
       <parent link="base_link"/>
       <child link="docking_link"/>
-      <origin xyz="-0.6 0 0" rpy="0 0 0" />
+      <origin xyz="-0.602 0 0" rpy="0 0 0" />
   </joint>
   <link name="docking_link">
