Commit message: Fix ari base simulation wheels/caster

File: ari_description/urdf/base/base.urdf.xacro (robot description, xacro)
@@ -88,15 +88,4 @@
     <parent link="${name}_footprint"/>
   </joint>
-  <!-- gazebo parameters are given here for base_link thru base_footprint -->
-  <gazebo reference="${name}_footprint">
-    <kp>100000000.0</kp>
-    <kd>10.0</kd>
-    <mu1>0.1</mu1>
-    <mu2>0.1</mu2>
-    <fdir1>1 0 0</fdir1>
-    <maxVel>10.0</maxVel>
-    <minDepth>0.0005</minDepth>
-    <laserRetro>0</laserRetro>
-  </gazebo>
   <!-- Wheels -->
   <xacro:wheel side="right" reflect=" 1.0" radius="${wheel_radius}" width="${wheel_width}" torque="${wheel_torque}" velocity="${wheel_velocity}" separation="${wheel_separation}" parent="${name}"/>

File: ari_description/urdf/wheels/caster_v2.urdf.xacro (robot description, xacro)
@@ -8,7 +8,7 @@
 -->
 <robot xmlns:xacro="http://ros.org/wiki/xacro">
-  <xacro:include filename="$(find ari_description)/urdf/wheels/caster.gazebo.xacro"/>
+  <xacro:include filename="$(find ari_description)/urdf/wheels/caster_v2.gazebo.xacro"/>
   <xacro:macro name="caster" params="side reflect radius width separation_x offset_y offset_z parent">
-    <link name="caster_${side}_link">
+    <link name="caster_${side}_1_link">
       <inertial>
         <origin xyz="-0.016512 0 -0.029897" rpy="0 0 0"/>
@@ -25,15 +25,30 @@
         <material name="Grey"/>
       </visual>
-      <collision>
-        <origin xyz="-0.02 0 -0.023" rpy="${90 * deg_to_rad} 0 0"/>
-        <geometry>
-          <cylinder radius="${radius}" length="${width}"/>
-        </geometry>
-      </collision>
     </link>
-    <joint name="caster_${side}_joint" type="continuous">
+    <link name="caster_${side}_2_link">
+      <inertial>
+        <origin xyz="0 0 0" rpy="0 0 0"/>
+          <mass value="0.08855784"/>
+          <inertia  ixx="0.00001075" ixy="0" ixz="0"
+                       iyy="0.00001541" iyz="0"
+                       izz="0.00001075"/>
+          </inertial>
+          <collision>
+            <origin xyz="0.0 0.0 0.0" rpy="0 0 0"/>
+            <geometry>
+               <sphere radius="${radius}" />
+             </geometry>
+           </collision>
+      </link>
+    <joint name="caster_${side}_1_joint" type="continuous">
       <parent link="${parent}_link"/>
-      <child link="caster_${side}_link"/>
+      <child link="caster_${side}_1_link"/>
       <origin xyz="${-separation_x / 2} ${-offset_y * reflect} ${offset_z}" rpy="${0.0 * deg_to_rad} 0 0"/>
+      <axis xyz="0 0 1"/>
+    </joint>
+    <joint name="caster_${side}_2_joint" type="continuous">
+      <parent link="caster_${side}_1_link"/>
+      <child link="caster_${side}_2_link"/>
+      <origin xyz="-0.02 0 -0.023" rpy="${-90.0*deg_to_rad} 0 0"/>
       <axis xyz="0 0 1"/>
     </joint>

File: ari_description/urdf/wheels/wheel.gazebo.xacro (robot description, xacro)
@@ -13,11 +13,13 @@
       <kp>1000000.0</kp>
       <kd>1000.0</kd>
-      <mu1>1.0</mu1>
-      <mu2>0.1</mu2> <!-- Frictionless wheels 0.0-->
-      <fdir1>1 0 0</fdir1>
+      <mu1>1000000000.0</mu1>
+      <mu2>1000000000.0</mu2> <!-- Frictionless wheels 0.0-->
+      <!--<fdir1>1 0 0</fdir1>-->
       <maxVel>1.0</maxVel>
-      <minDepth>0.00</minDepth>
+      <minDepth>0.002</minDepth>
+      <material>Gazebo/DarkGrey</material>
+    </gazebo>
+    <gazebo reference="wheel_${side}_joint">
       <implicitSpringDamper>1</implicitSpringDamper>
-      <material>Gazebo/DarkGrey</material>
     </gazebo>
   </xacro:macro>

Commit message: added colorized meshes for ARIv2
ARIv2 only, as ARIv1 mesh does not lend itself well to colors

File: ari_description/urdf/base/base.urdf.xacro (robot description, xacro)
@@ -60,5 +60,5 @@
         </xacro:if>
         <xacro:if value="${robot_model == 'v2'}">
-          <mesh filename="package://ari_description/meshes/base/base_v2.stl" />
+          <mesh filename="package://ari_description/meshes/base/base_v2.dae" />
         </xacro:if>
       </geometry>

File: ari_description/urdf/head/head.urdf.xacro (robot description, xacro)
@@ -110,5 +110,10 @@
         <origin xyz="0 0 0" rpy="0 0 0" />
         <geometry>
-          <mesh filename="package://ari_description/meshes/head/head_2.stl" scale="1 1 1"/>
+          <xacro:if value="${robot_model == 'v1'}">
+            <mesh filename="package://ari_description/meshes/head/head_2.stl" scale="1 1 1"/>
+          </xacro:if>
+          <xacro:if value="${robot_model == 'v2'}">
+            <mesh filename="package://ari_description/meshes/head/head_2.dae" scale="1 1 1"/>
+          </xacro:if>
         </geometry>
         <material name="White" />

Commit message: removed useless link

File: ari_description/urdf/base/base.urdf.xacro (robot description, xacro)
@@ -115,17 +115,4 @@
   </link>
   </xacro:macro>
-  <!-- RGBD Laser Link -->
-  <joint name="rgbd_laser_joint" type="fixed">
-      <parent link="base_link"/>
-      <child link="rgbd_laser_link"/>
-      <origin xyz="-1.1 0 0" rpy="0 0 0" />
-  </joint>
-  <link name="rgbd_laser_link">
-      <inertial>
-          <origin xyz="0 0 0" rpy="0 0 0"/>
-          <mass value="0.0001" />
-          <inertia ixx="0.0001"  ixy="0"  ixz="0" iyy="0.0001" iyz="0" izz="0.0001" />
-      </inertial>
-  </link>
   <joint name="back_led_link" type="fixed">
     <origin xyz="-0.12 0.0 -0.08" rpy="0.0 0.2 1.57" />

Commit message: fix ros2 control interface and added assisted_teleop

File: ari_description/urdf/base/base.urdf.xacro (robot description, xacro)
@@ -19,5 +19,5 @@
       <xacro:property name="wheel_separation" value="0.44"/>
       <xacro:property name="wheel_torque"     value="6.0"/>
-      <xacro:property name="wheel_velocity"   value="1.0"/>
+      <xacro:property name="wheel_velocity"   value="100.0"/>
           <!-- Caster wheel characteristics -->
       <xacro:property name="caster_radius"       value="0.045"/>
@@ -36,5 +36,5 @@
   <xacro:property name="wheel_separation" value="0.4668"/>
   <xacro:property name="wheel_torque"     value="6.0"/>
-  <xacro:property name="wheel_velocity"   value="1.0"/>
+  <xacro:property name="wheel_velocity"   value="100.0"/>
   <!-- Caster wheel characteristics -->
   <xacro:property name="caster_radius"       value="0.040"/>

File: ari_description/urdf/wheels/wheel.ros2_control.xacro (robot description, xacro)
@@ -10,8 +10,5 @@
   <xacro:macro name="ros2_control_wheel" params="side">
     <joint name="wheel_${side}_joint">
-      <command_interface name="velocity">
-        <param name="min">-1</param>
-        <param name="max">1</param>
-      </command_interface>
+      <command_interface name="velocity"/>
       <state_interface name="position" />
     </joint>

File: ari_description/urdf/wheels/wheel.urdf.xacro (robot description, xacro)
@@ -44,5 +44,5 @@
       <origin xyz="0 ${-separation / 2 * reflect} 0" rpy="${90.0 * deg_to_rad} 0 0"/>
       <axis xyz="0 0 -1"/>
-      <limit effort="${torque}" velocity="${velocity / radius}"/>
+      <limit effort="${torque}" velocity="${velocity}"/>
     </joint>
     <!-- Transmission -->

File: ari_description/urdf/wheels/wheel_v2.urdf.xacro (robot description, xacro)
@@ -44,5 +44,5 @@
       <origin xyz="0 ${ -separation / 2 * reflect} 0" rpy="${90 * deg_to_rad} 0 0"/>
       <axis xyz="0 0 -1"/>
-      <limit effort="${torque}" velocity="${velocity / radius}"/>
+      <limit effort="${torque}" velocity="${velocity}"/>
     </joint>
     <!-- Transmission -->
