Commit message: Removed the torso back camera frames coordinates because it will be put in a static transform in the torso_back_camera launch

File: ari_description/urdf/torso/torso_sensors.urdf.xacro (robot description, xacro)
@@ -21,10 +21,10 @@
   <xacro:property name="torso_front_camera_orientation_p" value="${42.5 * deg_to_rad}" />
   <xacro:property name="torso_front_camera_orientation_y" value="0.0" />
-  <xacro:property name="torso_back_camera_position_x" value="-0.3275" />
-  <xacro:property name="torso_back_camera_position_y" value="0.009" />
-  <xacro:property name="torso_back_camera_position_z" value="1.0337" />
-  <xacro:property name="torso_back_camera_orientation_r" value="${75 * deg_to_rad}" />
+  <xacro:property name="torso_back_camera_position_x" value="0.0" />
+  <xacro:property name="torso_back_camera_position_y" value="0.0" />
+  <xacro:property name="torso_back_camera_position_z" value="0.0" />
+  <xacro:property name="torso_back_camera_orientation_r" value="0.0" />
   <xacro:property name="torso_back_camera_orientation_p" value="0.0" />
-  <xacro:property name="torso_back_camera_orientation_y" value="${90 * deg_to_rad}" />
+  <xacro:property name="torso_back_camera_orientation_y" value="0.0" />
   <xacro:macro name="torso_sensors" params="name parent">
   <!-- Torso sensors -->

Commit message: Restore torso back camera transform

File: ari_description/urdf/torso/torso_sensors.urdf.xacro (robot description, xacro)
@@ -21,10 +21,10 @@
   <xacro:property name="torso_front_camera_orientation_p" value="${42.5 * deg_to_rad}" />
   <xacro:property name="torso_front_camera_orientation_y" value="0.0" />
-  <xacro:property name="torso_back_camera_position_x" value="0.0" />
-  <xacro:property name="torso_back_camera_position_y" value="0.0" />
-  <xacro:property name="torso_back_camera_position_z" value="0.0" />
+  <xacro:property name="torso_back_camera_position_x" value="-0.3275" />
+  <xacro:property name="torso_back_camera_position_y" value="0.009" />
+  <xacro:property name="torso_back_camera_position_z" value="1.0337" />
   <xacro:property name="torso_back_camera_orientation_r" value="0.0" />
-  <xacro:property name="torso_back_camera_orientation_p" value="0.0" />
-  <xacro:property name="torso_back_camera_orientation_y" value="0.0" />
+  <xacro:property name="torso_back_camera_orientation_p" value="${15 * deg_to_rad}" />
+  <xacro:property name="torso_back_camera_orientation_y" value="${180 * deg_to_rad}" />
   <xacro:macro name="torso_sensors" params="name parent">
   <!-- Torso sensors -->

Commit message: Update laser distances

File: ari_description/urdf/torso/torso_sensors.urdf.xacro (robot description, xacro)
@@ -29,7 +29,7 @@
   <xacro:property name="torso_back_camera_orientation_y" value="${180 * deg_to_rad}" />
   <!-- Laser characteristics -->
-  <xacro:property name="base_laser_x" value="-0.334"/>
+  <xacro:property name="base_laser_x" value="-0.34"/>
   <xacro:property name="base_laser_y" value="0.0"/>
-  <xacro:property name="base_laser_z" value="0.565"/>
+  <xacro:property name="base_laser_z" value="0.564"/>
   <xacro:macro name="torso_sensors" params="name parent">
   <!-- Torso sensors -->

Commit message: Correct front fisheye pitch to new pose

File: ari_description/urdf/torso/torso_sensors.urdf.xacro (robot description, xacro)
@@ -57,5 +57,5 @@
     </link>
     <joint name="front_fisheye_camera_joint" type="fixed">
-      <origin xyz="-0.1418 0.0 1.1956" rpy="0 ${-39 * deg_to_rad} 0"/>
+      <origin xyz="-0.1418 0.0 1.1956" rpy="0 ${-19 * deg_to_rad} 0"/>
       <parent link="${parent}" />
       <child link="front_fisheye_camera_link" />

Commit message: Update lidar frame in case of ari-v2

File: ari_description/urdf/torso/torso_sensors.urdf.xacro (robot description, xacro)
@@ -17,8 +17,4 @@
   <xacro:include filename="$(find ari_description)/urdf/sensors/ydlidar_tg30_laser.urdf.xacro"/>
   <xacro:include filename="$(find ari_description)/urdf/sensors/ydlidar_tg15_laser.urdf.xacro"/>
-  <!-- Laser characteristics -->
-  <xacro:property name="base_laser_x" value="-0.34"/>
-  <xacro:property name="base_laser_y" value="0.0"/>
-  <xacro:property name="base_laser_z" value="0.564"/>
   <xacro:macro name="torso_sensors" params="name parent robot_model use_nominal_extrinsics">
     <xacro:if value="${robot_model == 'v1'}">
@@ -36,4 +32,8 @@
       <xacro:property name="torso_back_camera_orientation_p" value="${15 * deg_to_rad}" />
       <xacro:property name="torso_back_camera_orientation_y" value="${180 * deg_to_rad}" />
+        <!-- Laser characteristics -->
+      <xacro:property name="base_laser_x" value="-0.34"/>
+      <xacro:property name="base_laser_y" value="0.0"/>
+      <xacro:property name="base_laser_z" value="0.564"/>
     </xacro:if>
     <xacro:if value="${robot_model == 'v2'}">
@@ -51,4 +51,8 @@
       <xacro:property name="torso_back_camera_orientation_p" value="${15 * deg_to_rad}" />
       <xacro:property name="torso_back_camera_orientation_y" value="${180 * deg_to_rad}" />
+        <!-- Laser characteristics -->
+      <xacro:property name="base_laser_x" value="-0.39777"/>
+      <xacro:property name="base_laser_y" value="0.0"/>
+      <xacro:property name="base_laser_z" value="0.26848"/>
     </xacro:if>
   <!-- Torso sensors -->

Commit message: Correct yaw for ydlidar

File: ari_description/urdf/torso/torso_sensors.urdf.xacro (robot description, xacro)
@@ -135,5 +135,5 @@
     <!-- Theoretic FOV = 360 -->
     <xacro:ydlidar_tg30_laser name="${name}_laser" parent="${parent}" ros_topic="scan_raw" update_rate="10" min_angle="${-180 * deg_to_rad}" max_angle="${180 * deg_to_rad}" >
-      <origin xyz="${base_laser_x} ${base_laser_y} ${base_laser_z}" rpy="0 0 ${ 180 * deg_to_rad }" />
+      <origin xyz="${base_laser_x} ${base_laser_y} ${base_laser_z}" rpy="0 0 ${ 200 * deg_to_rad }" />
     </xacro:ydlidar_tg30_laser>
   </xacro:if>
@@ -142,5 +142,5 @@
     <!-- Theoretic FOV = 360 -->
     <xacro:ydlidar_tg15_laser name="${name}_laser" parent="${parent}" ros_topic="scan_raw" update_rate="10" min_angle="${-180 * deg_to_rad}" max_angle="${180 * deg_to_rad}" >
-      <origin xyz="${base_laser_x} ${base_laser_y} ${base_laser_z}" rpy="0 0 ${ 180 * deg_to_rad }" />
+      <origin xyz="${base_laser_x} ${base_laser_y} ${base_laser_z}" rpy="0 0 ${ 200 * deg_to_rad }" />
     </xacro:ydlidar_tg15_laser>
   </xacro:if>

Commit message: Fix min_angle and max_angle ydlidar

File: ari_description/urdf/torso/torso_sensors.urdf.xacro (robot description, xacro)
@@ -134,5 +134,5 @@
     <!-- Laser -->
     <!-- Theoretic FOV = 360 -->
-    <xacro:ydlidar_tg30_laser name="${name}_laser" parent="${parent}" ros_topic="scan_raw" update_rate="10" min_angle="${-180 * deg_to_rad}" max_angle="${180 * deg_to_rad}" >
+    <xacro:ydlidar_tg30_laser name="${name}_laser" parent="${parent}" ros_topic="scan_raw" update_rate="10" min_angle="${-70 * deg_to_rad}" max_angle="${110 * deg_to_rad}" >
       <origin xyz="${base_laser_x} ${base_laser_y} ${base_laser_z}" rpy="0 0 ${ 200 * deg_to_rad }" />
     </xacro:ydlidar_tg30_laser>
@@ -141,8 +141,8 @@
     <!-- Laser -->
     <!-- Theoretic FOV = 360 -->
-    <xacro:ydlidar_tg15_laser name="${name}_laser" parent="${parent}" ros_topic="scan_raw" update_rate="10" min_angle="${-180 * deg_to_rad}" max_angle="${180 * deg_to_rad}" >
+    <xacro:ydlidar_tg15_laser name="${name}_laser" parent="${parent}" ros_topic="scan_raw" update_rate="10" min_angle="${-70 * deg_to_rad}" max_angle="${110 * deg_to_rad}" >
       <origin xyz="${base_laser_x} ${base_laser_y} ${base_laser_z}" rpy="0 0 ${ 200 * deg_to_rad }" />
     </xacro:ydlidar_tg15_laser>
   </xacro:if>
- </xacro:macro>
+</xacro:macro>
 </robot>

Commit message: fix use sick position only with sick

File: ari_description/urdf/torso/torso_sensors.urdf.xacro (robot description, xacro)
@@ -33,7 +33,9 @@
       <xacro:property name="torso_back_camera_orientation_y" value="${180 * deg_to_rad}" />
       <!-- Laser characteristics -->
-      <xacro:property name="base_laser_x" value="-0.34"/>
-      <xacro:property name="base_laser_y" value="0.0"/>
-      <xacro:property name="base_laser_z" value="0.564"/>
+      <xacro:if value="${laser_model == 'sick-571'}">
+        <xacro:property name="base_laser_x" value="-0.34"/>
+        <xacro:property name="base_laser_y" value="0.0"/>
+        <xacro:property name="base_laser_z" value="0.564"/>
+      </xacro:if>
       <xacro:if value="${laser_model in ['ydlidar-tg30', 'ydlidar-tg15']}">
         <xacro:property name="base_laser_x" value="-0.39777"/>
