Commit message: remove differential transmission

File: ari_description/ros2_control/transmissions.urdf.xacro (robot description, xacro)
@@ -23,23 +23,3 @@
     </transmission>
   </xacro:macro>
-  <xacro:macro name="ari_differential_transmission"
-               params="name number_1 number_2 act_reduction_1 act_reduction_2 jnt_reduction_1 jnt_reduction_2 number_1_offset number_2_offset" >
-  <transmission name="${name}_${number_1}_${name}_${number_2}_wrist_trans">
-      <plugin>transmission_interface/DifferentialTransmission</plugin>
-      <actuator name="${name}_${number_1}_actuator" role="actuator1">
-      <mechanical_reduction>${act_reduction_1}</mechanical_reduction>
-      </actuator>
-      <actuator name="${name}_${number_2}_actuator" role="actuator2">
-        <mechanical_reduction>${act_reduction_2}</mechanical_reduction>
-      </actuator>
-      <joint name="${name}_${number_1}_joint" role="joint1">
-        <mechanical_reduction>${jnt_reduction_1}</mechanical_reduction>
-        <offset>${number_1_offset}</offset>
-      </joint>
-      <joint name="${name}_${number_2}_joint" role="joint2">
-        <mechanical_reduction>${jnt_reduction_2}</mechanical_reduction>
-        <offset>${number_2_offset}</offset>
-      </joint>
-    </transmission>
-  </xacro:macro>
 </robot>
