Commit message: add robot_model param

File: ari_description/ros2_control/ros2_control.urdf.xacro (robot description, xacro)
@@ -42,6 +42,6 @@
         <!-- arms -->
         <xacro:include filename="$(find ari_description)/urdf/arm/arm.ros2_control.xacro" />
-        <xacro:ros2_control_arm side="left" />
-        <xacro:ros2_control_arm side="right" />
+        <xacro:ros2_control_arm side="left" robot_model="${robot_model}" />
+        <xacro:ros2_control_arm side="right" robot_model="${robot_model}" />
       </ros2_control>
     </xacro:if>
@@ -56,6 +56,6 @@
         <!-- arms -->
         <xacro:include filename="$(find ari_description)/urdf/arm/arm.ros2_control.xacro" />
-        <xacro:ros2_control_arm side="left" />
-        <xacro:ros2_control_arm side="right" />
+        <xacro:ros2_control_arm side="left" robot_model="${robot_model}" />
+        <xacro:ros2_control_arm side="right" robot_model="${robot_model}" />
         <!-- head -->
         <xacro:include filename="$(find ari_description)/urdf/head/head.ros2_control.xacro" />

File: ari_description/urdf/arm/arm.ros2_control.xacro (robot description, xacro)
@@ -25,10 +25,11 @@
     <xacro:ari_simple_transmission name="${name}" reduction="${reduction}" offset_value="${offset}" />
   </xacro:macro>
-  <xacro:macro name="ros2_control_arm" params="side" >
-      <xacro:ros2_control_arm_segment name="arm_${side}_1" reduction="1.0" offset="${arm_1_joint_offset}" />
-      <xacro:ros2_control_arm_segment name="arm_${side}_2" reduction="1.0" offset="${arm_2_joint_offset}" />
-      <xacro:ros2_control_arm_segment name="arm_${side}_3" reduction="1.0" offset="${arm_3_joint_offset}" />
-      <xacro:ros2_control_arm_segment name="arm_${side}_4" reduction="1.0" offset="${arm_4_joint_offset}" />
-      <xacro:ros2_control_arm_segment name="arm_${side}_5" reduction="1.0" offset="${arm_5_joint_offset}" />
-  </xacro:macro>
+  <xacro:macro name="ros2_control_arm" params="side robot_model:=v1" > <xacro:ros2_control_arm_segment name="arm_${side}_1" reduction="1.0" offset="${arm_1_joint_offset}" />
+        <xacro:ros2_control_arm_segment name="arm_${side}_2" reduction="1.0" offset="${arm_2_joint_offset}" />
+        <xacro:ros2_control_arm_segment name="arm_${side}_3" reduction="1.0" offset="${arm_3_joint_offset}" />
+        <xacro:ros2_control_arm_segment name="arm_${side}_4" reduction="1.0" offset="${arm_4_joint_offset}" />
+        <xacro:if value="${robot_model != 'v1'}">
+            <xacro:ros2_control_arm_segment name="arm_${side}_5" reduction="1.0" offset="${arm_5_joint_offset}" />
+        </xacro:if>
+    </xacro:macro>
 </robot>

Commit message: fix ros2 parameter handling

File: ari_description/ros2_control/ros2_control.urdf.xacro (robot description, xacro)
@@ -18,9 +18,6 @@
     <xacro:arg name="description_calibration_dir" default="$(find ari_description)/urdf/calibration" />
     <xacro:property name="is_v2" value="${robot_model == 'v2'}" />
-    <!-- calibration offsets -->
     <xacro:include filename="$(arg description_calibration_dir)/calibration_constants.urdf.xacro" />
-    <!-- Simulation -->
     <xacro:if value="$(arg use_sim_time)">
-      <!-- Init the ROS 2 control gazebo interface -->
       <gazebo>
         <plugin filename="libgazebo_ros2_control.so" name="gazebo_ros2_control">
@@ -32,13 +29,10 @@
           <plugin>gazebo_ros2_control/GazeboSystem</plugin>
         </hardware>
-        <!-- wheels -->
         <xacro:include filename="$(find ari_description)/urdf/wheels/wheel.ros2_control.xacro" />
         <xacro:ros2_control_wheel side="right" />
         <xacro:ros2_control_wheel side="left" />
-        <!-- head -->
         <xacro:include filename="$(find ari_description)/urdf/head/head.ros2_control.xacro" />
         <xacro:ros2_control_head name="head_1" reduction="1.0" offset="${head_1_joint_offset}" />
         <xacro:ros2_control_head name="head_2" reduction="1.0" offset="${head_2_joint_offset}" />
-        <!-- arms -->
         <xacro:include filename="$(find ari_description)/urdf/arm/arm.ros2_control.xacro" />
         <xacro:ros2_control_arm side="left" robot_model="${robot_model}" />
@@ -46,7 +40,5 @@
       </ros2_control>
     </xacro:if>
-    <!-- Hardware -->
     <xacro:unless value="$(arg use_sim_time)">
-      <!-- Dynamixels system -->
       <ros2_control name="ros2_control_ari_system_dynamixel" type="system" rw_rate="200">
         <hardware>
@@ -54,14 +46,11 @@
           <param name="group">dynamixel</param>
         </hardware>
-        <!-- arms -->
         <xacro:include filename="$(find ari_description)/urdf/arm/arm.ros2_control.xacro" />
         <xacro:ros2_control_arm side="left" robot_model="${robot_model}" />
         <xacro:ros2_control_arm side="right" robot_model="${robot_model}" />
-        <!-- head -->
         <xacro:include filename="$(find ari_description)/urdf/head/head.ros2_control.xacro" />
         <xacro:ros2_control_head name="head_1" reduction="1.0" offset="${head_1_joint_offset}" />
         <xacro:ros2_control_head name="head_2" reduction="1.0" offset="${head_2_joint_offset}" />
       </ros2_control>
-      <!-- PapstK4 system -->
       <ros2_control name="ros2_control_ari_system_papstk4" type="system" rw_rate="50">
         <hardware>
@@ -69,10 +58,22 @@
           <param name="group">papstk4</param>
         </hardware>
-        <!-- wheels -->
         <xacro:include filename="$(find ari_description)/urdf/wheels/wheel.ros2_control.xacro" />
         <xacro:ros2_control_wheel side="right" />
         <xacro:ros2_control_wheel side="left" />
       </ros2_control>
-    </xacro:unless>
+      <xacro:if value="${robot_model == 'v1'}">
+        <xacro:include filename="$(find ari_description)/ros2_control/transmissions.urdf.xacro" />
+        <xacro:finger_transmissions_ros2
+            finger_name="hand_left"
+            act_name="hand_left_fingers_actuator"
+            start="0.0"
+            reduction="1.0" />
+        <xacro:finger_transmissions_ros2
+            finger_name="hand_right"
+            act_name="hand_right_fingers_actuator"
+            start="0.0"
+            reduction="1.0" />
+      </xacro:if>
+      </xacro:unless>
   </xacro:macro>
 </robot>

File: ari_description/ros2_control/transmissions.urdf.xacro (robot description, xacro)
@@ -16,10 +16,51 @@
     <transmission name="${name}_trans">
       <plugin>transmission_interface/SimpleTransmission</plugin>
-      <actuator name="${name}_actuator"  role="actuator1"/>
+      <actuator name="${name}_actuator" role="actuator1"/>
       <joint name="${name}_joint" role="joint1">
         <mechanical_reduction>${reduction}</mechanical_reduction>
         <offset>${offset_value}</offset>
-     </joint>
+      </joint>
     </transmission>
   </xacro:macro>
+  <xacro:macro name="finger_transmissions_ros2" params="finger_name act_name start reduction:=1.0">
+    <ros2_control name="${finger_name}_virtual_system" type="system">
+      <hardware>
+        <plugin>mock_components/GenericSystem</plugin>
+      </hardware>
+      <joint name="${finger_name}_virtual_1_joint">
+        <command_interface name="position"/>
+        <state_interface name="position"/>
+      </joint>
+      <transmission name="${finger_name}_virtual_1_trans">
+        <plugin>hey5_transmissions/Hey5Reducer</plugin>
+        <actuator name="${act_name}" role="actuator1">
+          <mechanical_reduction>${reduction}</mechanical_reduction>
+        </actuator>
+        <joint name="${finger_name}_virtual_1_joint" role="joint1">
+          <offset>0.0</offset>
+        </joint>
+        <param name="deadBandLower">0.0</param>
+        <param name="deadBandUpper">${start}</param>
+        <param name="saturationLower">0.0</param>
+        <param name="saturationUpper">3.0</param>
+      </transmission>
+      <joint name="${finger_name}_virtual_2_joint">
+        <command_interface name="position"/>
+        <state_interface name="position"/>
+      </joint>
+      <transmission name="${finger_name}_virtual_2_trans">
+        <plugin>hey5_transmissions/Hey5Reducer</plugin>
+        <actuator name="${act_name}" role="actuator1">
+          <mechanical_reduction>${reduction}</mechanical_reduction>
+        </actuator>
+        <joint name="${finger_name}_virtual_2_joint" role="joint1">
+          <offset>0.0</offset>
+        </joint>
+        <param name="deadBandLower">0.0</param>
+        <param name="deadBandUpper">${start}</param>
+        <param name="saturationLower">0.0</param>
+        <param name="saturationUpper">3.0</param>
+      </transmission>
+    </ros2_control>
+  </xacro:macro>
 </robot>

File: ari_description/urdf/arm/actuators.urdf.xacro (robot description, xacro)
@@ -12,9 +12,9 @@
     <xacro:actuator_impl parent="${parent}" name="${name}">
       <xacro:insert_block name="origin" />
-      <limit lower="${0 * deg_to_rad}" upper="${75 * deg_to_rad}" effort="4.0" velocity="2.5" /> <!-- TODO; Tune effort -->
+      <limit lower="${0 * deg_to_rad}" upper="${50 * deg_to_rad}" effort="4.0" velocity="2.5" /> <!-- TODO; Tune effort -->
       <safety_controller k_position="20"
                          k_velocity="20"
                          soft_lower_limit="${0.0 * deg_to_rad}"
-                         soft_upper_limit="${75.0 * deg_to_rad}" />
+                         soft_upper_limit="${50.0 * deg_to_rad}" />
     </xacro:actuator_impl>
   </xacro:macro>

File: ari_description/urdf/arm/arm.ros2_control.xacro (robot description, xacro)
@@ -13,4 +13,5 @@
  -->
 <robot xmlns:xacro="http://ros.org/wiki/xacro">
+  <xacro:include filename="$(find ari_description)/ros2_control/transmissions.urdf.xacro" />
   <xacro:macro name="ros2_control_arm_segment" params="name reduction offset" >
     <joint name="${name}_joint">
@@ -29,6 +30,13 @@
         <xacro:ros2_control_arm_segment name="arm_${side}_3" reduction="1.0" offset="${arm_3_joint_offset}" />
         <xacro:ros2_control_arm_segment name="arm_${side}_4" reduction="1.0" offset="${arm_4_joint_offset}" />
-        <xacro:if value="${robot_model != 'v1'}">
+        <xacro:if value="${robot_model == 'v2'}">
             <xacro:ros2_control_arm_segment name="arm_${side}_5" reduction="1.0" offset="${arm_5_joint_offset}" />
+        </xacro:if>
+        <xacro:if value="${robot_model == 'v1' and end_effector == 'ari-hand'}">
+            <joint name="hand_${side}_fingers_joint">
+              <command_interface name="position" />
+              <state_interface name="position" />
+            </joint>
+            <xacro:ari_simple_transmission name="hand_${side}_fingers" reduction="1.0" offset_value="0.0" />
         </xacro:if>
     </xacro:macro>
