Commit message: Fixed bugs and parameters

File: ari_description/gazebo/gazebo.urdf.xacro (robot description, xacro)
@@ -38,4 +38,18 @@
       </xacro:if>
     </plugin>
+    <!--plugin name="gazebo_diff_drive" filename="libgazebo_diff_drive.so">
+      <legacyMode>false</legacyMode>
+      <alwaysOn>true</alwaysOn>
+      <updateRate>20</updateRate>
+      <wheelSeparation>${wheel_separation}</wheelSeparation>
+      <wheelDiameter>${wheel_radius*2}</wheelDiameter>
+      <torque>${wheel_torque}</torque>
+      <commandTopic>/mobile_base_controller/cmd_vel</commandTopic>
+      <odometryTopic>odom</odometryTopic>
+      <odometryFrame>odom</odometryFrame>
+      <robotBaseFrame>base_footprint</robotBaseFrame>
+      <odometrySource>0</odometrySource>
+      <gravity>true</gravity>
+    </plugin-->
   </gazebo>
   <!--gazebo reference="base_imu_link"-->

File: ari_description/robots/ari.urdf.xacro (robot description, xacro)
@@ -10,15 +10,10 @@
         name="ari" >
   <!--xacro:arg name="arm" default="true"/--> <!-- true, false -->
-  <!--xacro:arg name="laser_model" default="sick-571"/--> <!-- false, hokuyo, sick-551, sick-561, sick-571-->
   <!--xacro:arg name="camera_model" default="orbbec-astra"/--> <!-- false, orbbec-astra, orbbec-astra-pro, asus-xtion -->
   <xacro:arg name="multiple" default="false"/>
   <xacro:arg name="namespace" default=""/>
-  <!--xacro:property name="laser_model" value="$(arg laser_model)" /-->
   <!--xacro:property name="camera_model" value="$(arg camera_model)" /-->
   <xacro:property name="is_multiple" value="$(arg multiple)" />
   <xacro:property name="nsp" value="$(arg namespace)" />
-  <!--xacro:if value="${laser_model not in ['false', False, 'sick-551', 'sick-561', 'sick-571', 'hokuyo']}">
-    <xacro:wrong_laser_model/>
-  </xacro:if-->
   <!--xacro:if value="${camera_model not in ['false', False, 'orbbec-astra', 'orbbec-astra-pro', 'asus-xtion']}">
     <xacro:wrong_camera_model/>
@@ -45,5 +40,5 @@
   <xacro:include filename="$(find ari_description)/urdf/materials.urdf.xacro" />
   <!-- Now we can start using the macros included above to define the actual robot -->
-  <xacro:base name="base"/> <!--microphone="true"/-->
+  <xacro:base name="base"/>
   <xacro:torso_sensors name="torso" parent="base_link"/> <!--camera_model="$(arg camera_model)"/-->
   <xacro:head name="head" parent="base_link"/>

File: ari_description/urdf/base/base.urdf.xacro (robot description, xacro)
@@ -11,12 +11,21 @@
   <xacro:include filename="$(find ari_description)/urdf/deg_to_rad.xacro" />
   <xacro:include filename="$(find ari_description)/urdf/wheels/wheel.urdf.xacro"/>
+  <xacro:include filename="$(find ari_description)/urdf/wheels/caster.urdf.xacro"/>
   <!--xacro:include filename="$(find ari_description)/urdf/sensors/microphone.urdf.xacro"/-->
+  <!--xacro:include filename="$(find ari_description)/urdf/sensors/imu.urdf.xacro"/-->
   <!-- Wheel characteristics -->
-  <xacro:property name="wheel_radius"     value="0.101"/>
-  <xacro:property name="wheel_width"      value="0.040"/>
-  <xacro:property name="wheel_separation" value="0.4554"/>
-  <xacro:property name="wheel_pair_separation" value="0.420"/>
+  <xacro:property name="wheel_radius"     value="0.125"/>
+  <xacro:property name="wheel_width"      value="0.075"/>
+  <xacro:property name="wheel_separation" value="0.44"/>
   <xacro:property name="wheel_torque"     value="6.0"/>
   <xacro:property name="wheel_velocity"   value="1.0"/>
+  <!-- Caster wheel characteristics -->
+  <xacro:property name="caster_radius"       value="0.025"/>
+  <xacro:property name="caster_width"        value="0.015"/>
+  <xacro:property name="caster_separation_x" value="0.343"/>
+  <xacro:property name="caster_separation_y" value="0.204"/>
+  <xacro:property name="caster_offset_x"     value="-0.002"/>
+  <xacro:property name="caster_offset_y"     value="0.0"/>
+  <xacro:property name="caster_offset_z"     value="-0.0335"/>
   <xacro:macro name="base" params="name">
   <!-- Base -->
@@ -66,6 +75,9 @@
   </gazebo>
   <!-- Wheels -->
-  <xacro:wheel side="right" reflect=" 1.0" radius="${wheel_radius}" width="${wheel_width}" torque="${wheel_torque}" velocity="${wheel_velocity}" parent="${name}"/>
-  <xacro:wheel side="left"  reflect="-1.0" radius="${wheel_radius}" width="${wheel_width}" torque="${wheel_torque}" velocity="${wheel_velocity}" parent="${name}"/>
+  <xacro:wheel side="right" reflect=" 1.0" radius="${wheel_radius}" width="${wheel_width}" torque="${wheel_torque}" velocity="${wheel_velocity}" separation="${wheel_separation}" parent="${name}"/>
+  <xacro:wheel side="left"  reflect="-1.0" radius="${wheel_radius}" width="${wheel_width}" torque="${wheel_torque}" velocity="${wheel_velocity}" separation="${wheel_separation}" parent="${name}"/>
+  <!-- Casters wheels -->
+  <!--xacro:caster side="back_right"  radius="${caster_radius}" width="${caster_width}" separation_x="${-caster_separation_x}" separation_y="${ caster_separation_y}" offset_x="${caster_offset_x}" offset_y="${caster_offset_y}" offset_z="${caster_offset_z}" parent="${name}"/>
+  <xacro:caster side="back_left"   radius="${caster_radius}" width="${caster_width}" separation_x="${-caster_separation_x}" separation_y="${-caster_separation_y}" offset_x="${caster_offset_x}" offset_y="${caster_offset_y}" offset_z="${caster_offset_z}" parent="${name}"/-->
   </xacro:macro>
 </robot>

File: ari_description/urdf/head/head.urdf.xacro (robot description, xacro)
@@ -11,4 +11,5 @@
   <xacro:include filename="$(find ari_description)/urdf/deg_to_rad.xacro" />
   <xacro:include filename="$(find tiago_description)/urdf/head/head.transmission.xacro" />
+  <!--xacro:include filename="$(find tiago_description_calibration)/urdf/calibration/calibration_constants.urdf.xacro" /-->
   <!--Constant parameters-->
   <xacro:property name="head_1_joint_offset" value="0.0" />

File: ari_description/urdf/wheels/caster.gazebo.xacro (robot description, xacro)
@@ -8,15 +8,26 @@
 -->
 <robot xmlns:xacro="http://ros.org/wiki/xacro">
-  <xacro:macro name="wheel_gazebo" params="side">
-    <!-- Contact model for the wheel surface -->
-    <gazebo reference="wheel_${side}_link">
+  <xacro:macro name="caster_gazebo" params="side">
+    <!-- Contact model for the caster wheel surface -->
+    <gazebo reference="caster_${side}_1_link">
       <kp>1000000.0</kp>
       <kd>1000.0</kd>
       <mu1>1.0</mu1>
-      <mu2>1.0</mu2> <!-- Frictionless wheels 0.0?-->
+      <mu2>1.0</mu2>
+      <fdir1>0 0 1</fdir1>
+      <maxVel>1.0</maxVel>
+      <minDepth>0.0</minDepth>
+      <implicitSpringDamper>0</implicitSpringDamper>
+      <material>Gazebo/DarkGrey</material>
+    </gazebo>
+    <gazebo reference="caster_${side}_2_link">
+      <kp>1000000.0</kp>
+      <kd>1000.0</kd>
+      <mu1>0.4</mu1>
+      <mu2>0.4</mu2>
       <fdir1>1 0 0</fdir1>
       <maxVel>1.0</maxVel>
       <minDepth>0.00</minDepth>
-      <implicitSpringDamper>1</implicitSpringDamper>
+      <implicitSpringDamper>0</implicitSpringDamper>
       <material>Gazebo/DarkGrey</material>
     </gazebo>

File: ari_description/urdf/wheels/wheel.urdf.xacro (robot description, xacro)
@@ -10,5 +10,5 @@
   <xacro:include filename="$(find ari_description)/urdf/wheels/wheel.transmission.xacro"/>
   <xacro:include filename="$(find ari_description)/urdf/wheels/wheel.gazebo.xacro"/>
-  <xacro:macro name="wheel" params="side reflect radius width torque velocity parent">
+  <xacro:macro name="wheel" params="side reflect radius width torque velocity separation parent">
     <link name="wheel_${side}_link">
       <inertial>
@@ -29,14 +29,21 @@
         <origin xyz="0 0 0" rpy="0 0 0"/>
         <geometry>
-          <mesh filename="package://ari_description/meshes/wheels/wheel_${side}.stl"/>
+          <cylinder radius="${radius}" length="${width}"/>
         </geometry>
       </collision>
+      <kinematic>0</kinematic>
+      <gravity>1</gravity>
     </link>
     <joint name="wheel_${side}_joint" type="continuous">
       <parent link="${parent}_link"/>
       <child link="wheel_${side}_link"/>
-      <origin xyz="0 ${-0.22 * reflect} 0" rpy="${90.0 * deg_to_rad} 0 0"/>
+      <origin xyz="0 ${-separation / 2 * reflect} 0" rpy="${90.0 * deg_to_rad} 0 0"/>
       <axis xyz="0 0 -1"/>
-      <!--limit effort="${torque}" velocity="${velocity / radius}"/-->
+      <limit effort="${torque}" velocity="${velocity / radius}"/>
+      <!--dynamics damping="100"/-->
+      <!--safety_controller k_position="0"
+        k_velocity="10"
+        soft_lower_limit="-0.005"
+        soft_upper_limit="0.005" /-->
     </joint>
     <!-- Transmission -->

Commit message: Fixed bugs and added the camera launch in the bringup and the microphone urdf

File: ari_description/gazebo/gazebo.urdf.xacro (robot description, xacro)
@@ -53,46 +53,4 @@
     </plugin-->
   </gazebo>
-  <!--gazebo reference="base_imu_link"-->
-    <!-- this is expected to be reparented to pelvis with appropriate offset
-         when imu_link is reduced by fixed joint reduction -->
-    <!-- todo: this is working with gazebo 1.4, need to write a unit test -->
-    <!--sensor name="imu_sensor" type="imu">
-      <always_on>1</always_on>
-      <update_rate>1000.0</update_rate>
-      <imu>
-        <noise>
-          <type>gaussian</type-->
-          <!-- Noise parameters from Boston Dynamics
-               (http://gazebosim.org/wiki/Sensor_noise):
-                 rates (rad/s): mean=0, stddev=2e-4
-                 accels (m/s/s): mean=0, stddev=1.7e-2
-                 rate bias (rad/s): 5e-6 - 1e-5
-                 accel bias (m/s/s): 1e-1
-               Experimentally, simulation provide rates with noise of
-               about 1e-3 rad/s and accels with noise of about 1e-1 m/s/s.
-               So we don't expect to see the noise unless number of inner iterations
-               are increased.
-               We will add bias.  In this model, bias is sampled once for rates
-               and once for accels at startup; the sign (negative or positive)
-               of each bias is then switched with equal probability.  Thereafter,
-               the biases are fixed additive offsets.  We choose
-               bias means and stddevs to produce biases close to the provided
-               data. -->
-          <!--rate>
-            <mean>0.0</mean>
-            <stddev>2e-4</stddev>
-            <bias_mean>0.0000075</bias_mean>
-            <bias_stddev>0.0000008</bias_stddev>
-          </rate>
-          <accel>
-            <mean>0.0</mean>
-            <stddev>1.7e-2</stddev>
-            <bias_mean>0.1</bias_mean>
-            <bias_stddev>0.001</bias_stddev>
-          </accel>
-        </noise>
-      </imu>
-    </sensor>
-  </gazebo-->
   <!-- define global properties -->
   <xacro:property name="M_PI" value="3.1415926535897931" />

File: ari_description/urdf/base/base.urdf.xacro (robot description, xacro)
@@ -12,6 +12,4 @@
   <xacro:include filename="$(find ari_description)/urdf/wheels/wheel.urdf.xacro"/>
   <xacro:include filename="$(find ari_description)/urdf/wheels/caster.urdf.xacro"/>
-  <!--xacro:include filename="$(find ari_description)/urdf/sensors/microphone.urdf.xacro"/-->
-  <!--xacro:include filename="$(find ari_description)/urdf/sensors/imu.urdf.xacro"/-->
   <!-- Wheel characteristics -->
   <xacro:property name="wheel_radius"     value="0.125"/>
@@ -24,5 +22,5 @@
   <xacro:property name="caster_width"        value="0.055"/>
   <xacro:property name="caster_separation_x" value="0.91"/>
-  <xacro:property name="caster_separation_y" value="0.205"/>
+  <xacro:property name="caster_offset_y"     value="0.1025"/>
   <xacro:property name="caster_offset_z"     value="-0.08"/>
   <xacro:macro name="base" params="name">
@@ -76,7 +74,7 @@
   <xacro:wheel side="left"  reflect="-1.0" radius="${wheel_radius}" width="${wheel_width}" torque="${wheel_torque}" velocity="${wheel_velocity}" separation="${wheel_separation}" parent="${name}"/>
   <!-- Casters wheels -->
-  <xacro:caster side="right" reflect=" 1.0" radius="${caster_radius}" width="${caster_width}" separation_x="${caster_separation_x}" separation_y="${caster_separation_y}"
+  <xacro:caster side="right" reflect=" 1.0" radius="${caster_radius}" width="${caster_width}" separation_x="${caster_separation_x}" offset_y="${caster_offset_y}"
                 offset_z="${caster_offset_z}" parent="${name}"/>
-  <xacro:caster side="left"  reflect="-1.0" radius="${caster_radius}" width="${caster_width}" separation_x="${caster_separation_x}" separation_y="${caster_separation_y}"
+  <xacro:caster side="left"  reflect="-1.0" radius="${caster_radius}" width="${caster_width}" separation_x="${caster_separation_x}" offset_y="${caster_offset_y}"
                 offset_z="${caster_offset_z}" parent="${name}"/>
   </xacro:macro>

File: ari_description/urdf/head/head.urdf.xacro (robot description, xacro)
@@ -21,5 +21,5 @@
   <xacro:property name="head_1_lower_limit" value="-75"/>
   <xacro:property name="head_1_upper_limit" value="75"/>
-  <xacro:property name="head_2_lower_limit" value="-20"/>
+  <xacro:property name="head_2_lower_limit" value="-15"/>
   <xacro:property name="head_2_upper_limit" value="45"/>
   <!--************************-->
@@ -55,5 +55,5 @@
       <origin xyz="-0.2255 0 1.1915"  rpy="0 0 0" />
       <axis xyz="0 0 1" />
-      <limit lower="${head_1_lower_limit * deg_to_rad}" upper="${head_1_upper_limit * deg_to_rad}" effort="5.197" velocity="${head_max_vel}" />
+      <limit lower="${head_1_lower_limit * deg_to_rad}" upper="${head_1_upper_limit * deg_to_rad}" effort="3.4" velocity="${head_max_vel}" />
       <dynamics damping="${head_damping}" friction="${head_friction}"/>
       <safety_controller k_position="20"
@@ -104,5 +104,5 @@
       <origin xyz="0.0425000000000001 0 0.093"  rpy="${90.0 * deg_to_rad} 0 0" />
       <axis xyz="0 0 -1" />
-      <limit lower="${head_2_lower_limit * deg_to_rad}" upper="${head_2_upper_limit * deg_to_rad}" effort="2.77" velocity="${head_max_vel}" />
+      <limit lower="${head_2_lower_limit * deg_to_rad}" upper="${head_2_upper_limit * deg_to_rad}" effort="3.26" velocity="${head_max_vel}" />
       <dynamics damping="${head_damping}" friction="${head_friction}"/>
       <safety_controller k_position="20"

File: ari_description/urdf/sensors/microphone.urdf.xacro (robot description, xacro)
@@ -8,17 +8,12 @@
 -->
 <robot xmlns:xacro="http://ros.org/wiki/xacro">
-  <xacro:macro name="wheel_gazebo" params="side">
-    <!-- Contact model for the wheel surface -->
-    <gazebo reference="wheel_${side}_link">
-      <kp>1000000.0</kp>
-      <kd>1000.0</kd>
-      <mu1>1.0</mu1>
-      <mu2>0.0</mu2> <!-- Frictionless wheels 0.0-->
-      <fdir1>1 0 0</fdir1>
-      <maxVel>1.0</maxVel>
-      <minDepth>0.00</minDepth>
-      <implicitSpringDamper>1</implicitSpringDamper>
-      <material>Gazebo/DarkGrey</material>
-    </gazebo>
+  <!-- Macro -->
+  <xacro:macro name="microphone" params="name parent *origin">
+    <link name="${name}_link"/>
+    <joint name="${name}_joint" type="fixed">
+      <xacro:insert_block name="origin"/>
+      <child link="${name}_link"/>
+      <parent link="${parent}"/>
+    </joint>
   </xacro:macro>
 </robot>

File: ari_description/urdf/torso/torso_sensors.urdf.xacro (robot description, xacro)
@@ -12,4 +12,5 @@
   <xacro:include filename="$(find realsense_gazebo_plugin)/urdf/d435.urdf.xacro" />
   <xacro:include filename="$(find realsense_gazebo_plugin)/urdf/t265.urdf.xacro" />
+  <!--xacro:include filename="$(find ari_description)/urdf/sensors/microphone.urdf.xacro"/-->
   <!--xacro:include filename="$(find ari_description_calibration)/urdf/calibration/calibration_constants.urdf.xacro" /-->
   <!--Constant parameters-->
@@ -38,4 +39,8 @@
             rpy="${torso_back_camera_orientation_r} ${torso_back_camera_orientation_p} ${torso_back_camera_orientation_y}"/>
   </sensor_t265_gazebo>
+  <!-- Microphones -->
+  <!--xacro:microphone name="${name}_mic_front" parent="${parent}">
+    <origin xyz="0.23182 0.03902 0.195" rpy="0 0 0"/>
+  </xacro:microphone-->
  </xacro:macro>
 </robot>

File: ari_description/urdf/wheels/caster.urdf.xacro (robot description, xacro)
@@ -9,5 +9,5 @@
 <robot xmlns:xacro="http://ros.org/wiki/xacro">
   <xacro:include filename="$(find ari_description)/urdf/wheels/caster.gazebo.xacro"/>
-  <xacro:macro name="caster" params="side reflect radius width separation_x separation_y offset_z parent">
+  <xacro:macro name="caster" params="side reflect radius width separation_x offset_y offset_z parent">
     <link name="caster_${side}_link">
       <inertial>
@@ -35,5 +35,5 @@
       <parent link="${parent}_link"/>
       <child link="caster_${side}_link"/>
-      <origin xyz="${-separation_x / 2} ${-separation_y / 2 * reflect} ${offset_z}" rpy="${90.0 * deg_to_rad} 0 0"/>
+      <origin xyz="${-separation_x / 2} ${-offset_y * reflect} ${offset_z}" rpy="${90.0 * deg_to_rad} 0 0"/>
       <axis xyz="0 0 -1"/>
       <dynamics damping="0.005" friction="0.0"/>

File: ari_description/urdf/wheels/wheel.urdf.xacro (robot description, xacro)
@@ -41,9 +41,4 @@
       <axis xyz="0 0 -1"/>
       <limit effort="${torque}" velocity="${velocity / radius}"/>
-      <!--dynamics damping="100"/-->
-      <!--safety_controller k_position="0"
-        k_velocity="10"
-        soft_lower_limit="-0.005"
-        soft_upper_limit="0.005" /-->
     </joint>
     <!-- Transmission -->

Commit message: add hand joints and transmission for underactuation

File: ari_description/gazebo/gazebo.urdf.xacro (robot description, xacro)
@@ -38,19 +38,20 @@
       </xacro:if>
     </plugin>
-    <!--plugin name="gazebo_diff_drive" filename="libgazebo_diff_drive.so">
-      <legacyMode>false</legacyMode>
-      <alwaysOn>true</alwaysOn>
-      <updateRate>20</updateRate>
-      <wheelSeparation>${wheel_separation}</wheelSeparation>
-      <wheelDiameter>${wheel_radius*2}</wheelDiameter>
-      <torque>${wheel_torque}</torque>
-      <commandTopic>/mobile_base_controller/cmd_vel</commandTopic>
-      <odometryTopic>odom</odometryTopic>
-      <odometryFrame>odom</odometryFrame>
-      <robotBaseFrame>base_footprint</robotBaseFrame>
-      <odometrySource>0</odometrySource>
-      <gravity>true</gravity>
-    </plugin-->
   </gazebo>
+  <xacro:macro name="ari_hand_gazebo_simulation" params="side">
+    <gazebo>
+      <plugin filename="libgazebo_underactuated_finger.so" name="gazebo_${side}_fingers">
+        <actuatedJoint>hand_${side}_fingers_joint</actuatedJoint>
+        <virtualJoint>
+          <name>hand_${side}_virtual_1_joint</name>
+          <scale_factor>1.0</scale_factor>
+        </virtualJoint>
+        <virtualJoint>
+          <name>hand_${side}_virtual_2_joint</name>
+          <scale_factor>1.0</scale_factor>
+        </virtualJoint>
+      </plugin>
+    </gazebo>
+  </xacro:macro>
   <!-- define global properties -->
   <xacro:property name="M_PI" value="3.1415926535897931" />

File: ari_description/urdf/arm/arm.urdf.xacro (robot description, xacro)
@@ -10,5 +10,5 @@
   <!--File includes-->
   <xacro:include filename="$(find ari_description)/urdf/deg_to_rad.xacro" />
-  <!--xacro:include filename="$(find ari_description)/urdf/arm/wrist.urdf.xacro" /-->
+  <xacro:include filename="$(find ari_description)/urdf/arm/actuators.urdf.xacro" />
   <xacro:include filename="$(find ari_description)/urdf/arm/arm.transmission.xacro" />
   <!--Constant parameters-->
@@ -214,4 +214,34 @@
                          soft_upper_limit="${135.0 * deg_to_rad - arm_eps}" />
     </joint>
+    <!-- Tool Link -->
+    <link name="${name}_${side}_tool_link">
+      <inertial>
+        <origin xyz="0 0 0" rpy="0 0 0" />
+        <mass value="0.0001" />
+        <inertia ixx="0.00001" ixy="0.0" ixz="0.0"
+                 iyy="0.00001" iyz="0.0"
+                 izz="0.00001" />
+      </inertial>
+    </link>
+    <joint name="${name}_${side}_tool_joint" type="fixed">
+      <origin xyz="0 ${-0.35231*reflect} 0.0011086"
+              rpy="${-1.5708*reflect} -0.2618 ${1.5708*reflect}" />
+      <parent link="${name}_${side}_4_link" />
+      <child link="${name}_${side}_tool_link" />
+       <axis xyz="0 0 0" />
+    </joint>
+   <!--Actuator-->
+    <xacro:finger_actuator parent="${name}_${side}_tool_link" name="hand_${side}_fingers">
+      <origin xyz="0 0 0.0"
+      rpy="${1.5708+1.5708*reflect} 0.0 0.0" />
+    </xacro:finger_actuator>
+    <link name="${name}_${side}_grasping_frame"/>
+    <joint name="${name}_${side}_grasping_fixed_joint" type="fixed">
+      <parent link="${name}_${side}_4_link" />/>
+      <child link="${name}_${side}_grasping_frame"/>
+      <axis xyz="0 0 1" />
+      <origin xyz="0 ${-0.35231*reflect} 0.0011086"
+              rpy="${-1.5708*reflect} -0.2618 ${1.5708*reflect}" />
+    </joint>
     <link
     name="hand_${side}_1_link">
@@ -255,5 +285,5 @@
   </link>
   <joint
-    name="hand_${side}_1_joint"
+    name="hand_${side}_virtual_1_joint"
     type="revolute">
     <origin
@@ -320,5 +350,5 @@
   </link>
   <joint
-    name="hand_${side}_2_joint"
+    name="hand_${side}_virtual_2_joint"
     type="revolute">
     <origin
@@ -386,8 +416,8 @@
       <implicitSpringDamper>1</implicitSpringDamper>
    </gazebo>
-   <gazebo reference="hand_${side}_1_joint">
-      <implicitSpringDamper>1</implicitSpringDamper>
-   </gazebo>
-   <gazebo reference="hand_${side}_2_joint">
+   <gazebo reference="hand_${side}_virtual_1_joint">
+      <implicitSpringDamper>1</implicitSpringDamper>
+   </gazebo>
+   <gazebo reference="hand_${side}_virtual_2_joint">
       <implicitSpringDamper>1</implicitSpringDamper>
    </gazebo>
@@ -396,6 +426,11 @@
     <xacro:arm_simple_transmission name="${name}" side="${side}" number="3" reduction="1.0" offset_value="0.0"/>
     <xacro:arm_simple_transmission name="${name}" side="${side}" number="4" reduction="1.0" offset_value="0.0"/>
-    <xacro:arm_simple_transmission name="hand" side="${side}" number="1" reduction="1.0" offset_value="0.0"/>
-    <xacro:arm_simple_transmission name="hand" side="${side}" number="2" reduction="1.0" offset_value="0.0"/>
+    <xacro:finger_transmissions finger_name="hand_${side}"
+                                act_name="hand_${side}_fingers_motor"
+                                start="0.0"
+                                reduction="1.0"
+    />
+    <!-- gazebo plugin -->
+    <xacro:ari_hand_gazebo_simulation side="${name}"/>
   </xacro:macro>
 </robot>
