Commit message: add hand joints and transmission for underactuation

File: ari_description/gazebo/gazebo.urdf.xacro (robot description, xacro)
@@ -38,19 +38,20 @@
       </xacro:if>
     </plugin>
-    <!--plugin name="gazebo_diff_drive" filename="libgazebo_diff_drive.so">
-      <legacyMode>false</legacyMode>
-      <alwaysOn>true</alwaysOn>
-      <updateRate>20</updateRate>
-      <wheelSeparation>${wheel_separation}</wheelSeparation>
-      <wheelDiameter>${wheel_radius*2}</wheelDiameter>
-      <torque>${wheel_torque}</torque>
-      <commandTopic>/mobile_base_controller/cmd_vel</commandTopic>
-      <odometryTopic>odom</odometryTopic>
-      <odometryFrame>odom</odometryFrame>
-      <robotBaseFrame>base_footprint</robotBaseFrame>
-      <odometrySource>0</odometrySource>
-      <gravity>true</gravity>
-    </plugin-->
   </gazebo>
+  <xacro:macro name="ari_hand_gazebo_simulation" params="side">
+    <gazebo>
+      <plugin filename="libgazebo_underactuated_finger.so" name="gazebo_${side}_fingers">
+        <actuatedJoint>hand_${side}_fingers_joint</actuatedJoint>
+        <virtualJoint>
+          <name>hand_${side}_virtual_1_joint</name>
+          <scale_factor>1.0</scale_factor>
+        </virtualJoint>
+        <virtualJoint>
+          <name>hand_${side}_virtual_2_joint</name>
+          <scale_factor>1.0</scale_factor>
+        </virtualJoint>
+      </plugin>
+    </gazebo>
+  </xacro:macro>
   <!-- define global properties -->
   <xacro:property name="M_PI" value="3.1415926535897931" />

File: ari_description/urdf/arm/arm.transmission.xacro (robot description, xacro)
@@ -22,3 +22,29 @@
     </transmission>
   </xacro:macro>
+  <xacro:macro name="finger_transmissions" params="finger_name act_name start reduction">
+    <!--First flexor-->
+    <transmission name="${finger_name}_virtual_1_trans">
+      <type>hey5_transmissions/Hey5Reducer</type>
+      <joint name="${finger_name}_virtual_1_joint">
+        <saturationLower>0.0</saturationLower>
+        <deadBandUpper>${start}</deadBandUpper>
+        <hardwareInterface>hardware_interface/JointStateInterface</hardwareInterface>
+      </joint>
+      <actuator name="${act_name}">
+        <mechanicalReduction>${reduction}</mechanicalReduction>
+      </actuator>
+    </transmission>
+    <!--Second flexor-->
+    <transmission name="${finger_name}_virtual_2_trans">
+      <type>hey5_transmissions/Hey5Reducer</type>
+      <joint name="${finger_name}_virtual_2_joint">
+        <saturationLower>0.0</saturationLower>
+        <deadBandUpper>${start}</deadBandUpper>
+        <hardwareInterface>hardware_interface/JointStateInterface</hardwareInterface>
+      </joint>
+      <actuator name="${act_name}">
+        <mechanicalReduction>${reduction}</mechanicalReduction>
+      </actuator>
+    </transmission>
+  </xacro:macro>
 </robot>

File: ari_description/urdf/arm/arm.urdf.xacro (robot description, xacro)
@@ -10,5 +10,5 @@
   <!--File includes-->
   <xacro:include filename="$(find ari_description)/urdf/deg_to_rad.xacro" />
-  <!--xacro:include filename="$(find ari_description)/urdf/arm/wrist.urdf.xacro" /-->
+  <xacro:include filename="$(find ari_description)/urdf/arm/actuators.urdf.xacro" />
   <xacro:include filename="$(find ari_description)/urdf/arm/arm.transmission.xacro" />
   <!--xacro:include filename="$(find ari_description_calibration)/urdf/calibration/calibration_constants.urdf.xacro" /-->
@@ -215,4 +215,34 @@
                          soft_upper_limit="${135.0 * deg_to_rad - arm_eps}" />
     </joint>
+    <!-- Tool Link -->
+    <link name="${name}_${side}_tool_link">
+      <inertial>
+        <origin xyz="0 0 0" rpy="0 0 0" />
+        <mass value="0.0001" />
+        <inertia ixx="0.00001" ixy="0.0" ixz="0.0"
+                 iyy="0.00001" iyz="0.0"
+                 izz="0.00001" />
+      </inertial>
+    </link>
+    <joint name="${name}_${side}_tool_joint" type="fixed">
+      <origin xyz="0 ${-0.35231*reflect} 0.0011086"
+              rpy="${-1.5708*reflect} -0.2618 ${1.5708*reflect}" />
+      <parent link="${name}_${side}_4_link" />
+      <child link="${name}_${side}_tool_link" />
+       <axis xyz="0 0 0" />
+    </joint>
+   <!--Actuator-->
+    <xacro:finger_actuator parent="${name}_${side}_tool_link" name="hand_${side}_fingers">
+      <origin xyz="0 0 0.0"
+      rpy="${1.5708+1.5708*reflect} 0.0 0.0" />
+    </xacro:finger_actuator>
+    <link name="${name}_${side}_grasping_frame"/>
+    <joint name="${name}_${side}_grasping_fixed_joint" type="fixed">
+      <parent link="${name}_${side}_4_link" />/>
+      <child link="${name}_${side}_grasping_frame"/>
+      <axis xyz="0 0 1" />
+      <origin xyz="0 ${-0.35231*reflect} 0.0011086"
+              rpy="${-1.5708*reflect} -0.2618 ${1.5708*reflect}" />
+    </joint>
     <link
     name="hand_${side}_1_link">
@@ -256,5 +286,5 @@
   </link>
   <joint
-    name="hand_${side}_1_joint"
+    name="hand_${side}_virtual_1_joint"
     type="revolute">
     <origin
@@ -321,5 +351,5 @@
   </link>
   <joint
-    name="hand_${side}_2_joint"
+    name="hand_${side}_virtual_2_joint"
     type="revolute">
     <origin
@@ -387,8 +417,8 @@
       <implicitSpringDamper>1</implicitSpringDamper>
    </gazebo>
-   <gazebo reference="hand_${side}_1_joint">
-      <implicitSpringDamper>1</implicitSpringDamper>
-   </gazebo>
-   <gazebo reference="hand_${side}_2_joint">
+   <gazebo reference="hand_${side}_virtual_1_joint">
+      <implicitSpringDamper>1</implicitSpringDamper>
+   </gazebo>
+   <gazebo reference="hand_${side}_virtual_2_joint">
       <implicitSpringDamper>1</implicitSpringDamper>
    </gazebo>
@@ -397,6 +427,11 @@
     <xacro:arm_simple_transmission name="${name}" side="${side}" number="3" reduction="1.0" offset_value="0.0"/>
     <xacro:arm_simple_transmission name="${name}" side="${side}" number="4" reduction="1.0" offset_value="0.0"/>
-    <xacro:arm_simple_transmission name="hand" side="${side}" number="1" reduction="1.0" offset_value="0.0"/>
-    <xacro:arm_simple_transmission name="hand" side="${side}" number="2" reduction="1.0" offset_value="0.0"/>
+    <xacro:finger_transmissions finger_name="hand_${side}"
+                                act_name="hand_${side}_fingers_motor"
+                                start="0.0"
+                                reduction="1.0"
+    />
+    <!-- gazebo plugin -->
+    <xacro:ari_hand_gazebo_simulation side="${name}"/>
   </xacro:macro>
 </robot>
