Commit message: port ari_description to ROS2

File: ari_description/gazebo/gazebo.urdf.xacro (robot description, xacro)
@@ -1,42 +1,83 @@
 <?xml version="1.0"?>
 <!--
-  Copyright (c) 2019, PAL Robotics, S.L.
-  All rights reserved.
-  This work is licensed under the Creative Commons Attribution-NonCommercial-NoDerivs 3.0 Unported License.
-  To view a copy of this license, visit http://creativecommons.org/licenses/by-nc-nd/3.0/ or send a letter to
-  Creative Commons, 444 Castro Street, Suite 900, Mountain View, California, 94041, USA.
--->
+  Copyright (c) 2023 PAL Robotics S.L. All rights reserved.
+  Licensed under the Apache License, Version 2.0 (the "License");
+  you may not use this file except in compliance with the License.
+  You may obtain a copy of the License at
+      http://www.apache.org/licenses/LICENSE-2.0
+  Unless required by applicable law or agreed to in writing, software
+  distributed under the License is distributed on an "AS IS" BASIS,
+  WITHOUT WARRANTIES OR CONDITIONS OF ANY KIND, either express or implied.
+  See the License for the specific language governing permissions and
+  limitations under the License.
+ -->
 <robot name="ari" xmlns:xacro="http://ros.org/wiki/xacro">
   <gazebo>
-    <plugin filename="libgazebo_ros_control.so" name="gazebo_ros_control">
-      <ns></ns>
-      <robotSimType>pal_hardware_gazebo/PalHardwareGazebo</robotSimType>
+    <plugin filename="libgazebo_ros2_control.so" name="gazebo_ros2_control">
+      <!-- in the future move this param file somewhere else -->
+      <parameters>$(find ari_controller_configuration)/config/gazebo_controller_manager_cfg.yaml</parameters>
       <xacro:if value="${is_multiple}">
-          <robotNamespace>/${nsp}</robotNamespace>
+        <!-- Do something about multirobot -->
       </xacro:if>
       <xacro:unless value="${is_multiple}">
-          <robotNamespace></robotNamespace>
+        <!-- Do something about multirobot -->
       </xacro:unless>
-      <controlPeriod>0.001</controlPeriod>
     </plugin>
     <plugin filename="libgazebo_ros_p3d.so" name="gazebo_ros_p3d">
-      <bodyName>base_footprint</bodyName>
-      <topicName>ground_truth_odom</topicName>
-      <alwaysOn>true</alwaysOn>
-      <updateRate>100.0</updateRate>
+      <body_name>base_footprint</body_name>
+      <always_on>true</always_on>
+      <update_rate>100.0</update_rate>
+      <ros>
+        <remapping>odom:=ground_truth_odom</remapping>
+      </ros>
       <xacro:if value="${is_multiple}">
-          <robotNamespace>/${nsp}</robotNamespace>
+	    <!--<robotNamespace>/${nsp}</robotNamespace>-->
       </xacro:if>
     </plugin>
   </gazebo>
   <gazebo>
-    <plugin filename="libgazebo_world_odometry.so" name="gazebo_ros_odometry">
-      <frameName>base_footprint</frameName>
-      <topicName>floating_base_pose_simulated</topicName>
+    <!--- backwards compatibility, used to be gazebo_world_odometry pal plugin-->
+    <plugin filename="libgazebo_ros_p3d.so" name="gazebo_ros_odometry">
+      <body_name>base_footprint</body_name>
+      <always_on>true</always_on>
+      <update_rate>1000.0</update_rate>
+      <ros>
+        <remapping>odom:=floating_base_pose_simulated</remapping>
+      </ros>
       <xacro:if value="${is_multiple}">
-          <robotNamespace>/${nsp}</robotNamespace>
+	    <!--<robotNamespace>/${nsp}</robotNamespace>-->
       </xacro:if>
     </plugin>
   </gazebo>
+  <gazebo reference="base_imu_link">
+    <sensor name="imu_sensor" type="imu">
+      <always_on>1</always_on>
+      <update_rate>10.0</update_rate>
+      <imu>
+        <noise>
+          <type>gaussian</type>
+          <rate>
+            <mean>0.0</mean>
+            <stddev>2e-4</stddev>
+            <bias_mean>0.0000075</bias_mean>
+            <bias_stddev>0.0000008</bias_stddev>
+          </rate>
+          <accel>
+            <mean>0.0</mean>
+            <stddev>1.7e-2</stddev>
+            <bias_mean>0.1</bias_mean>
+            <bias_stddev>0.001</bias_stddev>
+          </accel>
+        </noise>
+      </imu>
+      <plugin name="base_imu" filename="libgazebo_ros_imu_sensor.so">
+        <ros>
+          <!-- publish to /imu/data -->
+          <remapping>~/out:=base_imu</remapping>
+        </ros>
+      </plugin>
+    </sensor>
+  </gazebo>
+<!-- TODO ROS2
   <xacro:macro name="ari_hand_gazebo_simulation" params="side">
     <gazebo>
@@ -54,4 +95,5 @@
     </gazebo>
   </xacro:macro>
+-->
   <!-- define global properties -->
   <xacro:property name="M_PI" value="3.1415926535897931" />

File: ari_description/robots/ari.urdf.xacro (robot description, xacro)
@@ -1,20 +1,30 @@
 <?xml version="1.0"?>
 <!--
-  Copyright (c) 2019, PAL Robotics, S.L.
-  All rights reserved.
-  This work is licensed under the Creative Commons Attribution-NonCommercial-NoDerivs 3.0 Unported License.
-  To view a copy of this license, visit http://creativecommons.org/licenses/by-nc-nd/3.0/ or send a letter to
-  Creative Commons, 444 Castro Street, Suite 900, Mountain View, California, 94041, USA.
--->
+  Copyright (c) 2023 PAL Robotics S.L. All rights reserved.
+  Licensed under the Apache License, Version 2.0 (the "License");
+  you may not use this file except in compliance with the License.
+  You may obtain a copy of the License at
+      http://www.apache.org/licenses/LICENSE-2.0
+  Unless required by applicable law or agreed to in writing, software
+  distributed under the License is distributed on an "AS IS" BASIS,
+  WITHOUT WARRANTIES OR CONDITIONS OF ANY KIND, either express or implied.
+  See the License for the specific language governing permissions and
+  limitations under the License.
+ -->
 <robot  xmlns:xacro="http://ros.org/wiki/xacro"
         name="ari" >
-  <xacro:arg name="robot_model" default="v1"/>
-  <xacro:arg name="end_effector_right" default="ari-hand"/>
-  <xacro:arg name="end_effector_left" default="ari-hand"/>
+  <xacro:arg name="robot_model" default="v2"/>
+  <xacro:arg name="end_effector_right" default="no-hand"/>
+  <xacro:arg name="end_effector_left" default="no-hand"/>
   <xacro:arg name="front_fisheye_camera" default="false"/>
   <xacro:arg name="back_fisheye_camera" default="false"/>
+  <xacro:arg name="laser_model" default="ydlidar-tg15"/> <!-- false, hokuyo, sick-551, sick-561, sick-571, ydlidar-tg30, ydlidar-tg15 -->
   <xacro:arg name="camera_model_head" default="raspi"/>
+  <xacro:arg name="rgbd_sensors" default="false"/> <!-- false, true-->
   <xacro:arg name="has_thermal" default="false"/>
-  <xacro:arg name="simulation" default="false" />
+  <xacro:arg name="description_calibration_dir" default="$(find ari_description)/urdf/calibration"/>
+  <xacro:arg name="multiple" default="false"/>
+  <xacro:arg name="namespace" default=""/>
+  <xacro:arg name="use_sim" default="true"/>
   <xacro:property name="robot_model" value="$(arg robot_model)" />
   <xacro:property name="end_effector_right" value="$(arg end_effector_right)" />
@@ -22,18 +32,18 @@
   <xacro:property name="front_fisheye_camera" value="$(arg front_fisheye_camera)" />
   <xacro:property name="back_fisheye_camera" value="$(arg back_fisheye_camera)" />
+  <xacro:property name="laser_model" value="$(arg laser_model)" />
   <xacro:property name="camera_model_head" value="$(arg camera_model_head)"/>
+  <xacro:property name="rgbd_sensors" value="$(arg rgbd_sensors)"/>
   <xacro:property name="has_thermal" value="$(arg has_thermal)"/>
-  <xacro:arg name="multiple" default="false"/>
-  <xacro:arg name="namespace" default=""/>
   <xacro:property name="is_multiple" value="$(arg multiple)" />
   <xacro:property name="nsp" value="$(arg namespace)" />
-  <xacro:property name="use_nominal_extrinsics" value="$(arg simulation)"/>
+  <xacro:property name="use_nominal_extrinsics" value="$(arg use_sim)"/>
   <xacro:if value="${robot_model not in ['v1', 'v2']}">
     <xacro:wrong_ari_robot_model/>
   </xacro:if>
-  <xacro:if value="${end_effector_right not in ['ari-hand', 'false', False]}">
+  <xacro:if value="${end_effector_right not in ['ari-hand', 'no-hand', 'false', False]}">
     <xacro:wrong_end_effector/>
   </xacro:if>
-  <xacro:if value="${end_effector_left not in ['ari-hand', 'false', False]}">
+  <xacro:if value="${end_effector_left not in ['ari-hand', 'no-hand', 'false', False]}">
     <xacro:wrong_end_effector/>
   </xacro:if>
@@ -41,8 +51,13 @@
     <xacro:wrong_front_fisheye_camera/>
   </xacro:if>
+  <xacro:property name="has_front_fisheye_camera"           value="${front_fisheye_camera in ['Jetson', True, 'true', 'PC']}"/>
   <xacro:if value="${back_fisheye_camera not in ['true', True, 'false', False, 'Jetson', 'PC']}">
     <xacro:wrong_back_fisheye_camera/>
   </xacro:if>
-  <xacro:if value="${camera_model_head not in ['raspi', 'D435i']}">
+  <xacro:property name="has_back_fisheye_camera"           value="${back_fisheye_camera in ['Jetson', True, 'true', 'PC']}"/>
+  <xacro:if value="${laser_model not in ['No', 'false', False, 'sick-551', 'sick-561', 'sick-571', 'hokuyo', 'ydlidar-tg30', 'ydlidar-tg15']}">
+    <xacro:wrong_laser_model/>
+  </xacro:if>
+  <xacro:if value="${camera_model_head not in ['raspi', 'realsense-d435']}">
     <xacro:wrong_camera_model/>
   </xacro:if>
@@ -50,20 +65,15 @@
     <xacro:wrong_thermal_camera/>
   </xacro:if>
-  <xacro:arg name="laser_model" default="false"/> <!-- false, hokuyo, sick-551, sick-561, sick-571-->
-  <xacro:arg name="rgbd_sensors" default="false"/> <!-- false, true-->
-  <xacro:property name="laser_model" value="$(arg laser_model)" />
-  <xacro:property name="rgbd_sensors" value="$(arg rgbd_sensors)"/>
-  <xacro:property name="has_front_fisheye_camera"           value="${front_fisheye_camera in ['Jetson', True, 'true', 'PC']}"/>
-  <xacro:property name="has_back_fisheye_camera"           value="${back_fisheye_camera in ['Jetson', True, 'true', 'PC']}"/>
-  <xacro:if value="${laser_model not in ['No', 'false', False, 'sick-551', 'sick-561', 'sick-571', 'hokuyo', 'ydlidar-tg30', 'ydlidar-tg15']}">
-    <xacro:wrong_laser_model/>
-  </xacro:if>
   <!-- The properties below are modified using empy http://www.alcyone.com/software/empy/
        from the create_robot.py tool. Handle them with care -->
   <xacro:property name="head_link_name"          value="head_2_link"/>
   <!-- The following included files set up definitions of parts of the robot body -->
-  <xacro:include filename="$(find ari_description)/urdf/base/base.urdf.xacro" />   <!-- Base -->
-  <xacro:include filename="$(find ari_description)/urdf/head/head.urdf.xacro" /> <!-- head -->
-  <xacro:include filename="$(find ari_description)/urdf/torso/torso_sensors.urdf.xacro" /> <!-- Torso -->
+  <!-- Base -->
+  <xacro:include filename="$(find ari_description)/urdf/base/base.urdf.xacro" />
+  <!-- Torso -->
+  <xacro:include filename="$(find ari_description)/urdf/torso/torso_sensors.urdf.xacro" />
+  <!-- Head -->
+  <xacro:include filename="$(find ari_description)/urdf/head/head.urdf.xacro" />
+  <!-- Arms -->
   <xacro:if value="${robot_model == 'v1'}">
       <xacro:include filename="$(find ari_description)/urdf/arm/arm.urdf.xacro" />   <!-- Arms -->
@@ -74,4 +84,8 @@
   <!-- Generic simulator_gazebo plugins -->
   <xacro:include filename="$(find ari_description)/gazebo/gazebo.urdf.xacro" />
+  <!-- ros2_control -->
+  <xacro:include filename="$(find ari_description)/ros2_control/ros2_control.urdf.xacro" />
+  <xacro:ari_ros2_control
+    use_sim="$(arg use_sim)" />
   <!-- Materials for visualization -->
   <xacro:include filename="$(find ari_description)/urdf/materials.urdf.xacro" />
@@ -81,18 +95,18 @@
   <xacro:head name="head" parent="base_link" robot_model="${robot_model}"/>
   <xacro:if value="${robot_model == 'v1'}">
-  <xacro:ari_arm name="arm" parent="base_link" side="left" reflect="1" end_effector="${end_effector_left == 'ari-hand'}">
-    <origin xyz="-0.219 0.097624 1.1111" rpy="${105.0 * deg_to_rad} ${0.0 * deg_to_rad} ${-180.0 * deg_to_rad}" />
-  </xacro:ari_arm>
-  <xacro:ari_arm name="arm" parent="base_link" side="right" reflect="-1" end_effector="${end_effector_right == 'ari-hand'}">
-    <origin xyz="-0.219 -0.097624 1.1111" rpy="${-105.0 * deg_to_rad} ${0.0 * deg_to_rad} ${180.0 * deg_to_rad}" />
-  </xacro:ari_arm>
+    <xacro:ari_arm name="arm" parent="base_link" side="left" reflect="1" end_effector="${end_effector_left == 'ari-hand'}">
+      <origin xyz="-0.219 0.097624 1.1111" rpy="${105.0 * deg_to_rad} ${0.0 * deg_to_rad} ${-180.0 * deg_to_rad}" />
+    </xacro:ari_arm>
+    <xacro:ari_arm name="arm" parent="base_link" side="right" reflect="-1" end_effector="${end_effector_right == 'ari-hand'}">
+      <origin xyz="-0.219 -0.097624 1.1111" rpy="${-105.0 * deg_to_rad} ${0.0 * deg_to_rad} ${180.0 * deg_to_rad}" />
+    </xacro:ari_arm>
   </xacro:if>
   <xacro:if value="${robot_model == 'v2'}">
-  <xacro:ari_arm name="arm" parent="base_link" side="left" reflect="1" end_effector="false">
-    <origin xyz="-0.22 0.08146 1.153" rpy="${0* deg_to_rad} ${0 * deg_to_rad} ${0 * deg_to_rad}" />
-  </xacro:ari_arm>
-  <xacro:ari_arm name="arm" parent="base_link" side="right" reflect="-1" end_effector="false">
-    <origin xyz="-0.22 -0.08146 1.153" rpy="${0 * deg_to_rad} ${0* deg_to_rad} ${180 * deg_to_rad}" />
-  </xacro:ari_arm>
+    <xacro:ari_arm name="arm" parent="base_link" side="left" reflect="1" end_effector="false">
+      <origin xyz="-0.22 0.08146 1.153" rpy="${0* deg_to_rad} ${0 * deg_to_rad} ${0 * deg_to_rad}" />
+    </xacro:ari_arm>
+    <xacro:ari_arm name="arm" parent="base_link" side="right" reflect="-1" end_effector="false">
+      <origin xyz="-0.22 -0.08146 1.153" rpy="${0 * deg_to_rad} ${0* deg_to_rad} ${180 * deg_to_rad}" />
+    </xacro:ari_arm>
   </xacro:if>
 </robot>

File: ari_description/urdf/arm/arm.urdf.xacro (robot description, xacro)
@@ -11,5 +11,4 @@
   <xacro:include filename="$(find ari_description)/urdf/deg_to_rad.xacro" />
   <xacro:include filename="$(find ari_description)/urdf/arm/actuators.urdf.xacro" />
-  <xacro:include filename="$(find ari_description)/urdf/arm/arm.transmission.xacro" />
   <!--Constant parameters-->
   <xacro:property name="arm_friction"       value="1.0" />
@@ -459,8 +458,5 @@
      </gazebo>
    </xacro:if>
-    <xacro:arm_simple_transmission name="${name}" side="${side}" number="1" reduction="1.0" offset_value="0.0"/>
-    <xacro:arm_simple_transmission name="${name}" side="${side}" number="2" reduction="1.0" offset_value="0.0"/>
-    <xacro:arm_simple_transmission name="${name}" side="${side}" number="3" reduction="1.0" offset_value="0.0"/>
-    <xacro:arm_simple_transmission name="${name}" side="${side}" number="4" reduction="1.0" offset_value="0.0"/>
+   <!-- TODO ROS2 - support finger control on ARIv1
     <xacro:if value="${end_effector}">
       <xacro:finger_transmissions finger_name="hand_${side}"
@@ -468,8 +464,7 @@
                                   start="0.0"
                                   reduction="1.0"/>
-      <!-- <xacro:arm_simple_transmission name="${name}" side="${side}" number="4" reduction="1.0" offset_value="0.0"/> -->
-      <!-- gazebo plugin -->
       <xacro:ari_hand_gazebo_simulation side="${side}"/>
     </xacro:if>
+    -->
   </xacro:macro>
 </robot>

File: ari_description/urdf/arm/arm_v2.urdf.xacro (robot description, xacro)
@@ -11,5 +11,4 @@
   <xacro:include filename="$(find ari_description)/urdf/deg_to_rad.xacro" />
   <xacro:include filename="$(find ari_description)/urdf/arm/actuators.urdf.xacro" />
-  <xacro:include filename="$(find ari_description)/urdf/arm/arm.transmission.xacro" />
   <!--Constant parameters-->
   <xacro:property name="arm_friction"       value="1.0" />
@@ -311,9 +310,4 @@
       <implicitSpringDamper>1</implicitSpringDamper>
    </gazebo>
-    <xacro:arm_simple_transmission name="${name}" side="${side}" number="1" reduction="1.0" offset_value="0.0"/>
-    <xacro:arm_simple_transmission name="${name}" side="${side}" number="2" reduction="1.0" offset_value="0.0"/>
-    <xacro:arm_simple_transmission name="${name}" side="${side}" number="3" reduction="1.0" offset_value="0.0"/>
-    <xacro:arm_simple_transmission name="${name}" side="${side}" number="4" reduction="1.0" offset_value="0.0"/>
-    <xacro:arm_simple_transmission name="${name}" side="${side}" number="5" reduction="1.0" offset_value="0.0"/>
   </xacro:macro>
 </robot>

File: ari_description/urdf/head/head.ros2_control.xacro (robot description, xacro)
@@ -12,28 +12,14 @@
   limitations under the License.
  -->
-<robot>
-  <material name="Blue">
-    <color rgba="0.0 0.0 0.8 1.0"/>
-  </material>
-  <material name="Green">
-    <color rgba="0.0 0.8 0.0 1.0"/>
-  </material>
-  <material name="Grey">
-    <color rgba="0.75294 0.75294 0.75294 1.0"/>
-  </material>
-  <material name="LightGrey">
-    <color rgba="0.9 0.9 0.9 1.0"/>
-  </material>
- <material name="DarkGrey">
-   <color rgba="0.1 0.1 0.1 1.0"/>
- </material>
-  <material name="Red">
-    <color rgba="0.8 0.0 0.0 1.0"/>
-  </material>
-  <material name="White">
-    <color rgba="1.0 1.0 1.0 1.0"/>
-  </material>
-  <material name="Yellow">
-    <color rgba="0.96 0.88 0.14 1.0"/>
-  </material>
+<robot xmlns:xacro="http://ros.org/wiki/xacro">
+  <xacro:macro name="ros2_control_head" params="name reduction offset" >
+    <joint name="${name}_joint">
+      <command_interface name="position" />
+      <state_interface name="position" />
+      <state_interface name="velocity" />
+      <state_interface name="effort" />
+    </joint>
+    <xacro:include filename="$(find ari_description)/ros2_control/transmissions.urdf.xacro" />
+    <xacro:ari_simple_transmission name="${name}" reduction="${reduction}" offset_value="${offset}" />
+  </xacro:macro>
 </robot>

File: ari_description/urdf/head/head.urdf.xacro (robot description, xacro)
@@ -10,7 +10,8 @@
   <!--File includes-->
   <xacro:include filename="$(find ari_description)/urdf/deg_to_rad.xacro" />
-  <xacro:include filename="$(find ari_description)/urdf/head/head.transmission.xacro" />
   <xacro:include filename="$(find ari_description)/urdf/sensors/rpi_camera.gazebo.xacro" />
-  <xacro:include filename="$(find realsense2_description)/urdf/_d435.urdf.xacro" />
+<!-- TODO ROS2: disabled until realsense camera available
+    <xacro:include filename="$(find realsense2_description)/urdf/_d435.urdf.xacro" />
+-->
   <!--Constant parameters-->
   <xacro:property name="head_1_joint_offset" value="0.0" />
@@ -93,6 +94,4 @@
        <implicitSpringDamper>1</implicitSpringDamper>
     </gazebo>
-    <!-- extensions -->
-    <xacro:head_transmission name="${name}" reduction="1" offset_value="${head_1_joint_offset}"/>
   </xacro:macro>
   <!--************************-->
@@ -143,5 +142,4 @@
       <material>Gazebo/White</material>
     </gazebo>
-    <xacro:head_transmission name="${name}" reduction="1" offset_value="${head_2_joint_offset}"/>
   </xacro:macro>
   <!--************************-->

File: ari_description/urdf/torso/torso_sensors.urdf.xacro (robot description, xacro)
@@ -10,6 +10,8 @@
   <!--File includes-->
   <xacro:include filename="$(find ari_description)/urdf/deg_to_rad.xacro" />
+<!-- TODO ROS2: disabled until realsense camera available
   <xacro:include filename="$(find realsense2_description)/urdf/_d435.urdf.xacro" />
   <xacro:include filename="$(find realsense2_description)/urdf/_t265.urdf.xacro" />
+-->
   <xacro:include filename="$(find ari_description)/urdf/sensors/microphone.urdf.xacro"/>
   <xacro:include filename="$(find ari_description)/urdf/sensors/imx179_camera.gazebo.xacro"/>
@@ -65,13 +67,17 @@
   <!-- Torso sensors -->
   <!-- Torso front camera -->
+<!-- TODO ROS2: disabled until realsense camera available
   <xacro:sensor_d435 parent="${parent}" name="${name}_front_camera" topics_ns="${name}_front_camera" use_nominal_extrinsics="${use_nominal_extrinsics}">
     <origin xyz="${torso_front_camera_position_x} ${torso_front_camera_position_y} ${torso_front_camera_position_z}"
             rpy="${torso_front_camera_orientation_r} ${torso_front_camera_orientation_p} ${torso_front_camera_orientation_y}"/>
   </xacro:sensor_d435>
+-->
   <!-- Torso back camera -->
+<!-- TODO ROS2: disabled until realsense camera available
   <xacro:sensor_t265 parent="${parent}" name="${name}_back_camera" topics_ns="${name}_back_camera">
     <origin xyz="${torso_back_camera_position_x} ${torso_back_camera_position_y} ${torso_back_camera_position_z}"
             rpy="${torso_back_camera_orientation_r} ${torso_back_camera_orientation_p} ${torso_back_camera_orientation_y}"/>
   </xacro:sensor_t265>
+-->
   <!-- Optional SPRING cameras -->
   <xacro:if value="${has_front_fisheye_camera}">

File: ari_description/urdf/wheels/wheel.urdf.xacro (robot description, xacro)
@@ -1,13 +1,17 @@
 <?xml version="1.0"?>
 <!--
-Copyright (c) 2019, PAL Robotics, S.L.
-All rights reserved.
-This work is licensed under the Creative Commons Attribution-NonCommercial-NoDerivs 3.0 Unported License.
-To view a copy of this license, visit http://creativecommons.org/licenses/by-nc-nd/3.0/ or send a letter to
-Creative Commons, 444 Castro Street, Suite 900, Mountain View, California, 94041, USA.
--->
+  Copyright (c) 2023 PAL Robotics S.L. All rights reserved.
+  Licensed under the Apache License, Version 2.0 (the "License");
+  you may not use this file except in compliance with the License.
+  You may obtain a copy of the License at
+      http://www.apache.org/licenses/LICENSE-2.0
+  Unless required by applicable law or agreed to in writing, software
+  distributed under the License is distributed on an "AS IS" BASIS,
+  WITHOUT WARRANTIES OR CONDITIONS OF ANY KIND, either express or implied.
+  See the License for the specific language governing permissions and
+  limitations under the License.
+ -->
 <robot xmlns:xacro="http://ros.org/wiki/xacro">
-  <xacro:include filename="$(find ari_description)/urdf/wheels/wheel.transmission.xacro"/>
-  <xacro:include filename="$(find ari_description)/urdf/wheels/wheel.gazebo.xacro"/>
+  <xacro:include filename="$(find ari_description)/ros2_control/transmissions.urdf.xacro"/>
   <xacro:macro name="wheel" params="side reflect radius width torque velocity separation parent">
     <link name="wheel_${side}_link">
@@ -43,7 +47,5 @@
     </joint>
     <!-- Transmission -->
-    <xacro:wheel_transmission side="${side}"/>
-    <!-- Gazebo extensions -->
-    <xacro:wheel_gazebo side="${side}"/>
+    <xacro:ari_simple_transmission name="wheel_${side}"/>
   </xacro:macro>
 </robot>
