Commit message: port ari_description to ROS2

File: ari_description/urdf/wheels/wheel_v2.urdf.xacro (robot description, xacro)
@@ -1,13 +1,17 @@
 <?xml version="1.0"?>
 <!--
-Copyright (c) 2019, PAL Robotics, S.L.
-All rights reserved.
-This work is licensed under the Creative Commons Attribution-NonCommercial-NoDerivs 3.0 Unported License.
-To view a copy of this license, visit http://creativecommons.org/licenses/by-nc-nd/3.0/ or send a letter to
-Creative Commons, 444 Castro Street, Suite 900, Mountain View, California, 94041, USA.
--->
+  Copyright (c) 2023 PAL Robotics S.L. All rights reserved.
+  Licensed under the Apache License, Version 2.0 (the "License");
+  you may not use this file except in compliance with the License.
+  You may obtain a copy of the License at
+      http://www.apache.org/licenses/LICENSE-2.0
+  Unless required by applicable law or agreed to in writing, software
+  distributed under the License is distributed on an "AS IS" BASIS,
+  WITHOUT WARRANTIES OR CONDITIONS OF ANY KIND, either express or implied.
+  See the License for the specific language governing permissions and
+  limitations under the License.
+ -->
 <robot xmlns:xacro="http://ros.org/wiki/xacro">
-  <xacro:include filename="$(find ari_description)/urdf/wheels/wheel.transmission.xacro"/>
-  <xacro:include filename="$(find ari_description)/urdf/wheels/wheel.gazebo.xacro"/>
+  <xacro:include filename="$(find ari_description)/ros2_control/transmissions.urdf.xacro"/>
   <xacro:macro name="wheel" params="side reflect radius width torque velocity separation parent">
     <link name="wheel_${side}_link">
@@ -43,7 +47,5 @@
     </joint>
     <!-- Transmission -->
-    <xacro:wheel_transmission side="${side}"/>
-    <!-- Gazebo extensions -->
-    <xacro:wheel_gazebo side="${side}"/>
+    <xacro:ari_simple_transmission name="wheel_${side}"/>
   </xacro:macro>
 </robot>

Commit message: Modify ros2_control

File: ari_description/gazebo/gazebo.urdf.xacro (robot description, xacro)
@@ -36,65 +36,4 @@
     </plugin>
   </gazebo>
-  <gazebo>
-    <!--- backwards compatibility, used to be gazebo_world_odometry pal plugin-->
-    <plugin filename="libgazebo_ros_p3d.so" name="gazebo_ros_odometry">
-      <body_name>base_footprint</body_name>
-      <always_on>true</always_on>
-      <update_rate>1000.0</update_rate>
-      <ros>
-        <remapping>odom:=floating_base_pose_simulated</remapping>
-      </ros>
-      <xacro:if value="${is_multiple}">
-	    <!--<robotNamespace>/${nsp}</robotNamespace>-->
-      </xacro:if>
-    </plugin>
-  </gazebo>
-  <gazebo reference="base_imu_link">
-    <sensor name="imu_sensor" type="imu">
-      <always_on>1</always_on>
-      <update_rate>10.0</update_rate>
-      <imu>
-        <noise>
-          <type>gaussian</type>
-          <rate>
-            <mean>0.0</mean>
-            <stddev>2e-4</stddev>
-            <bias_mean>0.0000075</bias_mean>
-            <bias_stddev>0.0000008</bias_stddev>
-          </rate>
-          <accel>
-            <mean>0.0</mean>
-            <stddev>1.7e-2</stddev>
-            <bias_mean>0.1</bias_mean>
-            <bias_stddev>0.001</bias_stddev>
-          </accel>
-        </noise>
-      </imu>
-      <plugin name="base_imu" filename="libgazebo_ros_imu_sensor.so">
-        <ros>
-          <!-- publish to /imu/data -->
-          <remapping>~/out:=base_imu</remapping>
-        </ros>
-      </plugin>
-    </sensor>
-  </gazebo>
-<!-- TODO ROS2
-  <xacro:macro name="ari_hand_gazebo_simulation" params="side">
-    <gazebo>
-      <plugin filename="libgazebo_underactuated_finger.so" name="gazebo_${side}_fingers">
-        <actuatedJoint>hand_${side}_fingers_joint</actuatedJoint>
-        <virtualJoint>
-          <name>hand_${side}_virtual_1_joint</name>
-          <scale_factor>1.0</scale_factor>
-        </virtualJoint>
-        <virtualJoint>
-          <name>hand_${side}_virtual_2_joint</name>
-          <scale_factor>1.0</scale_factor>
-        </virtualJoint>
-      </plugin>
-    </gazebo>
-  </xacro:macro>
--->
-  <!-- define global properties -->
   <xacro:property name="M_PI" value="3.1415926535897931" />
 </robot>

File: ari_description/robots/ari.urdf.xacro (robot description, xacro)
@@ -78,5 +78,5 @@
   </xacro:if>
   <!-- Generic simulator_gazebo plugins -->
-  <xacro:include filename="$(find ari_description)/gazebo/gazebo.urdf.xacro" />
+  <!-- <xacro:include filename="$(find ari_description)/gazebo/gazebo.urdf.xacro" /> -->
   <!-- ros2_control -->
   <xacro:include filename="$(find ari_description)/ros2_control/ros2_control.urdf.xacro" />

File: ari_description/ros2_control/ros2_control.urdf.xacro (robot description, xacro)
@@ -23,9 +23,9 @@
     <xacro:if value="$(arg use_sim_time)">
       <!-- Init the ROS 2 control gazebo interface -->
-      <!-- <gazebo>
+      <gazebo>
         <plugin filename="libgazebo_ros2_control.so" name="gazebo_ros2_control">
           <parameters>$(find ari_description)/ros2_control/gazebo_controller_manager_cfg.yaml</parameters>
         </plugin>
-      </gazebo> -->
+      </gazebo>
       <ros2_control name="ros2_control_gazebo_system" type="system">
         <hardware>
