Commit message: Added the trasmission xacro files and the gazebo tags in the urdf files

File: ari_description/robots/ari.urdf.xacro (robot description, xacro)
@@ -41,5 +41,5 @@
   <xacro:include filename="$(find ari_description)/urdf/head/head.urdf.xacro" />
   <!-- Generic simulator_gazebo plugins -->
-  <!--xacro:include filename="$(find ari_description)/gazebo/gazebo.urdf.xacro" /-->
+  <xacro:include filename="$(find ari_description)/gazebo/gazebo.urdf.xacro" />
   <!-- Materials for visualization -->
   <xacro:include filename="$(find ari_description)/urdf/materials.urdf.xacro" />

File: ari_description/urdf/head/head.urdf.xacro (robot description, xacro)
@@ -10,6 +10,8 @@
   <!--File includes-->
   <xacro:include filename="$(find ari_description)/urdf/deg_to_rad.xacro" />
-  <!--xacro:include filename="$(find tiago_description)/urdf/head/head.transmission.xacro" /-->
+  <xacro:include filename="$(find tiago_description)/urdf/head/head.transmission.xacro" />
   <!--Constant parameters-->
+  <xacro:property name="head_1_joint_offset" value="0.0" />
+  <xacro:property name="head_2_joint_offset" value="0.0" />
   <!--xacro:property name="head_friction" value="1.0" />
   <xacro:property name="head_damping"  value="0.5" />
@@ -68,5 +70,5 @@
     </gazebo>
     <!-- extensions -->
-    <!--xacro:head_transmission name="${name}" reduction="1" offset_value="${head_1_joint_offset}"/-->
+    <xacro:head_transmission name="${name}" reduction="1" offset_value="${head_1_joint_offset}"/>
   </xacro:macro>
   <!--************************-->
@@ -87,5 +89,5 @@
           <mesh filename="package://ari_description/meshes/head/head_2.stl" scale="1 1 1"/>
         </geometry>
-        <material name="Yellow" />
+        <material name="White" />
       </visual>
       <collision>
@@ -94,4 +96,5 @@
           <mesh filename="package://ari_description/meshes/head/head_2.stl" scale="1 1 1"/>
         </geometry>
+        <material name="White" />
       </collision>
     </link>
@@ -109,5 +112,5 @@
                          soft_upper_limit="${head_2_upper_limit * deg_to_rad}" /-->
     </joint>
-    <!--xacro:head_transmission name="${name}" reduction="1" offset_value="${head_2_joint_offset}"/-->
+    <xacro:head_transmission name="${name}" reduction="1" offset_value="${head_2_joint_offset}"/>
   </xacro:macro>
   <xacro:macro name="head" params="name parent">

File: ari_description/urdf/wheels/wheel.urdf.xacro (robot description, xacro)
@@ -8,6 +8,6 @@
 -->
 <robot xmlns:xacro="http://ros.org/wiki/xacro">
-  <!--xacro:include filename="$(find ari_description)/urdf/wheels/wheel.transmission.xacro"/>
-  <xacro:include filename="$(find ari_description)/urdf/wheels/wheel.gazebo.xacro"/-->
+  <xacro:include filename="$(find ari_description)/urdf/wheels/wheel.transmission.xacro"/>
+  <xacro:include filename="$(find ari_description)/urdf/wheels/wheel.gazebo.xacro"/>
   <xacro:macro name="wheel" params="side reflect radius width torque velocity parent">
     <link name="wheel_${side}_link">
@@ -41,7 +41,7 @@
     </joint>
     <!-- Transmission -->
-    <!--xacro:wheel_transmission side="${side}"/-->
+    <xacro:wheel_transmission side="${side}"/>
     <!-- Gazebo extensions -->
-    <!--xacro:wheel_gazebo side="${side}"/-->
+    <xacro:wheel_gazebo side="${side}"/>
   </xacro:macro>
 </robot>

Commit message: Added the left arm

File: ari_description/robots/ari.urdf.xacro (robot description, xacro)
@@ -9,17 +9,10 @@
 <robot  xmlns:xacro="http://ros.org/wiki/xacro"
         name="ari" >
-  <!--xacro:arg name="arm" default="true"/--> <!-- true, false -->
-  <!--xacro:arg name="camera_model" default="orbbec-astra"/--> <!-- false, orbbec-astra, orbbec-astra-pro, asus-xtion -->
   <xacro:arg name="multiple" default="false"/>
   <xacro:arg name="namespace" default=""/>
-  <!--xacro:property name="camera_model" value="$(arg camera_model)" /-->
   <xacro:property name="is_multiple" value="$(arg multiple)" />
   <xacro:property name="nsp" value="$(arg namespace)" />
-  <!--xacro:if value="${camera_model not in ['false', False, 'orbbec-astra', 'orbbec-astra-pro', 'asus-xtion']}">
-    <xacro:wrong_camera_model/>
-  </xacro:if-->
   <!-- The properties below are modified using empy http://www.alcyone.com/software/empy/
        from the create_robot.py tool. Handle them with care -->
-  <!--xacro:property name="has_arm"                 value="$(arg arm)"/-->
   <xacro:property name="head_link_name"          value="head_2_link"/>
   <!-- The following included files set up definitions of parts of the robot base -->
@@ -28,9 +21,7 @@
   <!-- Torso -->
   <xacro:include filename="$(find ari_description)/urdf/torso/torso_sensors.urdf.xacro" />
-  <!--xacro:if value="${has_arm}"-->
-    <!-- Arm -->
-    <!--xacro:include filename="$(find tiago_description)/urdf/arm/arm.urdf.xacro" />
-    <xacro:include filename="$(find tiago_description)/urdf/end_effector/end_effector.urdf.xacro" />
-  </xacro:if-->
+  <!-- Arm -->
+  <xacro:include filename="$(find ari_description)/urdf/arm/arm.urdf.xacro" />
+  <!--xacro:include filename="$(find ari_description)/urdf/end_effector/end_effector.urdf.xacro" /-->
   <!-- Head -->
   <xacro:include filename="$(find ari_description)/urdf/head/head.urdf.xacro" />
@@ -41,12 +32,10 @@
   <!-- Now we can start using the macros included above to define the actual robot -->
   <xacro:base name="base"/>
-  <xacro:torso_sensors name="torso" parent="base_link"/> <!--camera_model="$(arg camera_model)"/-->
+  <xacro:torso_sensors name="torso" parent="base_link"/>
   <xacro:head name="head" parent="base_link"/>
-  <!--xacro:if value="${has_arm}">
-	  <xacro:tiago_arm name="arm" parent="torso_lift_link" wrist_6_range="${wrist_6_range}" reflect="1" tiago_dual="-1">
-        <origin xyz="0.15505 0.014 -0.151" rpy="0 0 ${-90 * deg_to_rad}" />
-      </xacro:tiago_arm>
-      <xacro:tiago_end_effector name="${end_effector_name}" parent="${end_effector_link}" type="${end_effector}" reflect="1"/>
-  </xacro:if-->
+  <xacro:ari_arm name="arm_left" parent="base_link" reflect="1">
+    <origin xyz="-0.219 0.097624 1.1111" rpy="${105.0 * deg_to_rad} ${0.0 * deg_to_rad} ${-180.0 * deg_to_rad}" />
+  </xacro:ari_arm>
+  <!--xacro:ari_end_effector name="${end_effector_name}" parent="${end_effector_link}" type="${end_effector}" reflect="1"/-->
   <!-- RGBD Laser Link -->
   <!--joint name="rgbd_laser_joint" type="fixed">
