Commit message: Add rgbd_laser_joint and rgbd_laser_link to ari.urdfx.xacrio

File: ari_description/robots/ari.urdf.xacro (robot description, xacro)
@@ -42,8 +42,8 @@
   </xacro:ari_arm>
   <!-- RGBD Laser Link -->
-  <!--joint name="rgbd_laser_joint" type="fixed">
-      <parent link="base_footprint"/>
+  <joint name="rgbd_laser_joint" type="fixed">
+      <parent link="base_link"/>
       <child link="rgbd_laser_link"/>
-      <origin xyz="-0.9 0 0" rpy="0 0 0" />
+      <origin xyz="-1 0 0" rpy="0 0 0" />
   </joint>
   <link name="rgbd_laser_link">
@@ -53,4 +53,4 @@
           <inertia ixx="0.0001"  ixy="0"  ixz="0" iyy="0.0001" iyz="0" izz="0.0001" />
       </inertial>
-  </link-->
+  </link>
 </robot>

File: ari_description/urdf/head/head.urdf.xacro (robot description, xacro)
@@ -120,5 +120,5 @@
   <!--      HEAD_CAMERA       -->
   <!--************************-->
-  <xacro:macro name="head_camera" params="name parent">
+  <xacro:macro name="head_front_camera" params="name parent">
   <link name="${name}_link">
     <inertial>
@@ -162,5 +162,5 @@
     <xacro:head_1 name="${name}_1" parent="${parent}" />
     <xacro:head_2 name="${name}_2" parent="${name}_1_link"/>
-    <xacro:head_camera name="${name}_front_camera" parent="${name}_2_link"/>
+    <xacro:head_front_camera name="${name}_front_camera" parent="${name}_2_link"/>
   </xacro:macro>
 </robot>

Commit message: changed rgbd link to base urdf

File: ari_description/robots/ari.urdf.xacro (robot description, xacro)
@@ -41,16 +41,3 @@
     <origin xyz="-0.219 -0.097624 1.1111" rpy="${-105.0 * deg_to_rad} ${0.0 * deg_to_rad} ${180.0 * deg_to_rad}" />
   </xacro:ari_arm>
-  <!-- RGBD Laser Link -->
-  <joint name="rgbd_laser_joint" type="fixed">
-      <parent link="base_link"/>
-      <child link="rgbd_laser_link"/>
-      <origin xyz="-1 0 0" rpy="0 0 0" />
-  </joint>
-  <link name="rgbd_laser_link">
-      <inertial>
-          <origin xyz="0 0 0" rpy="0 0 0"/>
-          <mass value="0.0001" />
-          <inertia ixx="0.0001"  ixy="0"  ixz="0" iyy="0.0001" iyz="0" izz="0.0001" />
-      </inertial>
-  </link>
 </robot>

File: ari_description/urdf/base/base.urdf.xacro (robot description, xacro)
@@ -79,3 +79,16 @@
                 offset_z="${caster_offset_z}" parent="${name}"/>
   </xacro:macro>
+  <!-- RGBD Laser Link -->
+  <joint name="rgbd_laser_joint" type="fixed">
+      <parent link="base_link"/>
+      <child link="rgbd_laser_link"/>
+      <origin xyz="-1 0 0" rpy="0 0 0" />
+  </joint>
+  <link name="rgbd_laser_link">
+      <inertial>
+          <origin xyz="0 0 0" rpy="0 0 0"/>
+          <mass value="0.0001" />
+          <inertia ixx="0.0001"  ixy="0"  ixz="0" iyy="0.0001" iyz="0" izz="0.0001" />
+      </inertial>
+  </link>
 </robot>

Commit message: Add parameter for end_effector

File: ari_description/robots/ari.urdf.xacro (robot description, xacro)
@@ -9,8 +9,13 @@
 <robot  xmlns:xacro="http://ros.org/wiki/xacro"
         name="ari" >
+  <xacro:arg name="ari_end_effector" default="ari_hand"/>
+  <xacro:property name="end_effector" value="$(arg ari_end_effector)" />
   <xacro:arg name="multiple" default="false"/>
   <xacro:arg name="namespace" default=""/>
   <xacro:property name="is_multiple" value="$(arg multiple)" />
   <xacro:property name="nsp" value="$(arg namespace)" />
+  <xacro:if value="${end_effector not in ['ari_hand', 'false', False]}">
+    <xacro:wrong_end_effector/>
+  </xacro:if>
   <!-- The properties below are modified using empy http://www.alcyone.com/software/empy/
        from the create_robot.py tool. Handle them with care -->
@@ -33,8 +38,8 @@
   <xacro:torso_sensors name="torso" parent="base_link"/>
   <xacro:head name="head" parent="base_link"/>
-  <xacro:ari_arm name="arm" parent="base_link" side="left" reflect="1">
+  <xacro:ari_arm name="arm" parent="base_link" side="left" reflect="1" end_effector="${end_effector == 'ari_hand'}">
     <origin xyz="-0.219 0.097624 1.1111" rpy="${105.0 * deg_to_rad} ${0.0 * deg_to_rad} ${-180.0 * deg_to_rad}" />
   </xacro:ari_arm>
-  <xacro:ari_arm name="arm" parent="base_link" side="right" reflect="-1">
+  <xacro:ari_arm name="arm" parent="base_link" side="right" reflect="-1" end_effector="${end_effector == 'ari_hand'}">
     <origin xyz="-0.219 -0.097624 1.1111" rpy="${-105.0 * deg_to_rad} ${0.0 * deg_to_rad} ${180.0 * deg_to_rad}" />
   </xacro:ari_arm>

File: ari_description/urdf/arm/arm.urdf.xacro (robot description, xacro)
@@ -24,5 +24,5 @@
   <xacro:property name="arm_4_max_effort"   value="5" />
   <xacro:property name="arm_eps"            value="0.07" />
-  <xacro:macro name="ari_arm" params="name parent side reflect *origin">
+  <xacro:macro name="ari_arm" params="name parent side reflect end_effector *origin">
     <!--************************-->
     <!--      ARM_BASE_LINK     -->
@@ -186,14 +186,45 @@
       </inertial>
       <visual>
-        <origin xyz="0 0 0" rpy="0 0 0" />
-        <geometry>
-          <mesh filename="package://ari_description/meshes/arm/${name}_4.stl" scale="1 ${reflect} 1"/>
+        <xacro:if value="${end_effector}">
+          <origin xyz="0 0 0" rpy="0 0 0" />
+        </xacro:if>
+        <xacro:unless value="${end_effector}">
+          <xacro:if value="${side == 'left'}">
+            <origin xyz="0 0 0" rpy="0 0 0" />
+          </xacro:if>
+          <xacro:if value="${side == 'right'}">
+            <origin xyz="0 0 0" rpy="0 0 ${-90 * deg_to_rad}" />
+          </xacro:if>
+        </xacro:unless>
+        <geometry>
+          <xacro:if value="${end_effector}">
+            <mesh filename="package://ari_description/meshes/arm/${name}_4.stl" scale="1 ${reflect} 1"/>
+          </xacro:if>
+          <xacro:unless value="${end_effector}">
+            <mesh filename="package://ari_description/meshes/arm/${name}_${side}_4.stl" scale="1 1 1"/>
+          </xacro:unless>
         </geometry>
         <material name="White" />
       </visual>
       <collision>
-        <origin xyz="0 0 0" rpy="0 0 0" />
-        <geometry>
-          <mesh filename="package://ari_description/meshes/arm/${name}_4.stl" scale="1 ${reflect} 1"/>
+        <xacro:if value="${end_effector}">
+          <origin xyz="0 0 0" rpy="0 0 0" />
+        </xacro:if>
+        <xacro:unless value="${end_effector}">
+          <xacro:if value="${side == 'left'}">
+            <origin xyz="0 0 0" rpy="0 0 0" />
+          </xacro:if>
+          <xacro:if value="${side == 'right'}">
+            <origin xyz="0 0 0" rpy="0 0 ${-90 * deg_to_rad}" />
+          </xacro:if>
+        </xacro:unless>
+        <origin xyz="0 0 0" rpy="0 0 0" />
+        <geometry>
+          <xacro:if value="${end_effector}">
+            <mesh filename="package://ari_description/meshes/arm/${name}_4.stl" scale="1 ${reflect} 1"/>
+          </xacro:if>
+          <xacro:unless value="${end_effector}">
+            <mesh filename="package://ari_description/meshes/arm/${name}_${side}_4.stl" scale="1 1 1"/>
+          </xacro:unless>
         </geometry>
       </collision>
@@ -214,164 +245,166 @@
                          soft_upper_limit="${135.0 * deg_to_rad - arm_eps}" />
     </joint>
-    <!-- Tool Link -->
-    <link name="${name}_${side}_tool_link">
-      <inertial>
-        <origin xyz="0 0 0" rpy="0 0 0" />
-        <mass value="0.0001" />
-        <inertia ixx="0.00001" ixy="0.0" ixz="0.0"
-                 iyy="0.00001" iyz="0.0"
-                 izz="0.00001" />
-      </inertial>
-    </link>
-    <joint name="${name}_${side}_tool_joint" type="fixed">
-      <origin xyz="0 ${-0.35231*reflect} 0.0011086"
-              rpy="${-1.5708*reflect} -0.2618 ${1.5708*reflect}" />
-      <parent link="${name}_${side}_4_link" />
-      <child link="${name}_${side}_tool_link" />
-       <axis xyz="0 0 0" />
-    </joint>
-   <!--Actuator-->
-    <xacro:finger_actuator parent="${name}_${side}_tool_link" name="hand_${side}_fingers">
-      <origin xyz="0 0 0.0"
-      rpy="${1.5708+1.5708*reflect} 0.0 0.0" />
-    </xacro:finger_actuator>
-    <link name="${name}_${side}_grasping_frame"/>
-    <joint name="${name}_${side}_grasping_fixed_joint" type="fixed">
-      <parent link="${name}_${side}_4_link" />
-      <child link="${name}_${side}_grasping_frame"/>
-      <axis xyz="0 0 1" />
-      <origin xyz="0 ${-0.35231*reflect} 0.0011086"
-              rpy="${-1.5708*reflect} -0.2618 ${1.5708*reflect}" />
+    <xacro:if value="${end_effector}">
+      <!-- Tool Link -->
+      <link name="${name}_${side}_tool_link">
+        <inertial>
+          <origin xyz="0 0 0" rpy="0 0 0" />
+          <mass value="0.0001" />
+          <inertia ixx="0.00001" ixy="0.0" ixz="0.0"
+                   iyy="0.00001" iyz="0.0"
+                   izz="0.00001" />
+        </inertial>
+      </link>
+      <joint name="${name}_${side}_tool_joint" type="fixed">
+        <origin xyz="0 ${-0.35231*reflect} 0.0011086"
+                rpy="${-1.5708*reflect} -0.2618 ${1.5708*reflect}" />
+        <parent link="${name}_${side}_4_link" />
+        <child link="${name}_${side}_tool_link" />
+         <axis xyz="0 0 0" />
+      </joint>
+     <!--Actuator-->
+      <xacro:finger_actuator parent="${name}_${side}_tool_link" name="hand_${side}_fingers">
+        <origin xyz="0 0 0.0"
+        rpy="${1.5708+1.5708*reflect} 0.0 0.0" />
+      </xacro:finger_actuator>
+      <link name="${name}_${side}_grasping_frame"/>
+      <joint name="${name}_${side}_grasping_fixed_joint" type="fixed">
+        <parent link="${name}_${side}_4_link" />
+        <child link="${name}_${side}_grasping_frame"/>
+        <axis xyz="0 0 1" />
+        <origin xyz="0 ${-0.35231*reflect} 0.0011086"
+                rpy="${-1.5708*reflect} -0.2618 ${1.5708*reflect}" />
+      </joint>
+      <link
+      name="hand_${side}_1_link">
+      <inertial>
+        <origin
+          xyz="-0.0194858087119051 -0.00284946290069976 -0.000289044791174375"
+          rpy="0 0 0" />
+        <mass
+          value="0.0400715645648009" />
+        <inertia
+          ixx="1.56769636746935E-06"
+          ixy="2.22831013516217E-08"
+          ixz="7.74537720537552E-09"
+          iyy="4.6054803967178E-06"
+          iyz="2.08251121489226E-10"
+          izz="4.01623373583446E-06" />
+      </inertial>
+      <visual>
+        <origin
+          xyz="0 0 0"
+          rpy="0 0 0" />
+        <geometry>
+          <mesh
+            filename="package://ari_description/meshes/arm/hand_1.stl" scale="1 ${reflect} 1"/>
+        </geometry>
+        <material
+          name="">
+          <color
+            rgba="0.752941176470588 0.752941176470588 0.752941176470588 1" />
+        </material>
+      </visual>
+      <collision>
+        <origin
+          xyz="0 0 0"
+          rpy="0 0 0" />
+        <geometry>
+          <mesh
+            filename="package://ari_description/meshes/arm/hand_1.stl" scale="1 ${reflect} 1"/>
+        </geometry>
+      </collision>
+    </link>
+    <joint
+      name="hand_${side}_virtual_1_joint"
+      type="revolute">
+      <origin
+        xyz="0 ${-0.35231*reflect} 0.0011086"
+        rpy="${-1.5708*reflect} -0.2618 ${1.5708*reflect}" />
+      <parent
+        link="${name}_${side}_4_link" />
+      <child
+        link="hand_${side}_1_link" />
+      <axis
+        xyz="0 0 ${-1*reflect}" />
+      <limit
+        lower="0"
+        upper="1.5708"
+        effort="1.0"
+        velocity="2.0" />
+  <!--
+      <dynamics friction="${arm_friction}" damping="${arm_damping}"/>
+      <safety_controller k_position="20"
+                           k_velocity="20"
+                           soft_lower_limit="${0.0 + arm_eps}"
+                           soft_upper_limit="${1.5708 - arm_eps}" />
+  -->
     </joint>
     <link
-    name="hand_${side}_1_link">
-    <inertial>
+      name="hand_${side}_2_link">
+      <inertial>
+        <origin
+          xyz="-0.0159508701186225 0.00214676466101674 0.000361575914240066"
+          rpy="0 0 0" />
+        <mass
+          value="0.0262043707272721" />
+        <inertia
+          ixx="9.15137557050205E-07"
+          ixy="5.3927377524493E-07"
+          ixz="-5.3325168061876E-09"
+          iyy="2.67374552400975E-06"
+          iyz="-6.4411286354103E-10"
+          izz="2.38630247657937E-06" />
+      </inertial>
+      <visual>
+        <origin
+          xyz="0 0 0"
+          rpy="0 0 0" />
+        <geometry>
+          <mesh
+            filename="package://ari_description/meshes/arm/hand_2.stl" scale="1 ${reflect} 1"/>
+        </geometry>
+        <material
+          name="">
+          <color
+            rgba="0.752941176470588 0.752941176470588 0.752941176470588 1" />
+        </material>
+      </visual>
+      <collision>
+        <origin
+          xyz="0 0 0"
+          rpy="0 0 0" />
+        <geometry>
+          <mesh
+            filename="package://ari_description/meshes/arm/hand_2.stl" scale="1 ${reflect} 1"/>
+        </geometry>
+      </collision>
+    </link>
+    <joint
+      name="hand_${side}_virtual_2_joint"
+      type="revolute">
       <origin
-        xyz="-0.0194858087119051 -0.00284946290069976 -0.000289044791174375"
+        xyz="-0.037185 0.0001459 0"
         rpy="0 0 0" />
-      <mass
-        value="0.0400715645648009" />
-      <inertia
-        ixx="1.56769636746935E-06"
-        ixy="2.22831013516217E-08"
-        ixz="7.74537720537552E-09"
-        iyy="4.6054803967178E-06"
-        iyz="2.08251121489226E-10"
-        izz="4.01623373583446E-06" />
-    </inertial>
-    <visual>
-      <origin
-        xyz="0 0 0"
-        rpy="0 0 0" />
-      <geometry>
-        <mesh
-          filename="package://ari_description/meshes/arm/hand_1.stl" scale="1 ${reflect} 1"/>
-      </geometry>
-      <material
-        name="">
-        <color
-          rgba="0.752941176470588 0.752941176470588 0.752941176470588 1" />
-      </material>
-    </visual>
-    <collision>
-      <origin
-        xyz="0 0 0"
-        rpy="0 0 0" />
-      <geometry>
-        <mesh
-          filename="package://ari_description/meshes/arm/hand_1.stl" scale="1 ${reflect} 1"/>
-      </geometry>
-    </collision>
-  </link>
-  <joint
-    name="hand_${side}_virtual_1_joint"
-    type="revolute">
-    <origin
-      xyz="0 ${-0.35231*reflect} 0.0011086"
-      rpy="${-1.5708*reflect} -0.2618 ${1.5708*reflect}" />
-    <parent
-      link="${name}_${side}_4_link" />
-    <child
-      link="hand_${side}_1_link" />
-    <axis
-      xyz="0 0 ${-1*reflect}" />
-    <limit
-      lower="0"
-      upper="1.5708"
-      effort="1.0"
-      velocity="2.0" />
-<!--
-    <dynamics friction="${arm_friction}" damping="${arm_damping}"/>
-    <safety_controller k_position="20"
-                         k_velocity="20"
-                         soft_lower_limit="${0.0 + arm_eps}"
-                         soft_upper_limit="${1.5708 - arm_eps}" />
--->
-  </joint>
-  <link
-    name="hand_${side}_2_link">
-    <inertial>
-      <origin
-        xyz="-0.0159508701186225 0.00214676466101674 0.000361575914240066"
-        rpy="0 0 0" />
-      <mass
-        value="0.0262043707272721" />
-      <inertia
-        ixx="9.15137557050205E-07"
-        ixy="5.3927377524493E-07"
-        ixz="-5.3325168061876E-09"
-        iyy="2.67374552400975E-06"
-        iyz="-6.4411286354103E-10"
-        izz="2.38630247657937E-06" />
-    </inertial>
-    <visual>
-      <origin
-        xyz="0 0 0"
-        rpy="0 0 0" />
-      <geometry>
-        <mesh
-          filename="package://ari_description/meshes/arm/hand_2.stl" scale="1 ${reflect} 1"/>
-      </geometry>
-      <material
-        name="">
-        <color
-          rgba="0.752941176470588 0.752941176470588 0.752941176470588 1" />
-      </material>
-    </visual>
-    <collision>
-      <origin
-        xyz="0 0 0"
-        rpy="0 0 0" />
-      <geometry>
-        <mesh
-          filename="package://ari_description/meshes/arm/hand_2.stl" scale="1 ${reflect} 1"/>
-      </geometry>
-    </collision>
-  </link>
-  <joint
-    name="hand_${side}_virtual_2_joint"
-    type="revolute">
-    <origin
-      xyz="-0.037185 0.0001459 0"
-      rpy="0 0 0" />
-    <parent
-      link="hand_${side}_1_link" />
-    <child
-      link="hand_${side}_2_link" />
-    <axis
-      xyz="0 0 ${-1*reflect}" />
-    <limit
-      lower="0"
-      upper="1.5708"
-      effort="1.0"
-      velocity="2.0" />
-<!--
-    <dynamics friction="${arm_friction}" damping="${arm_damping}"/>
-    <safety_controller k_position="20"
-                         k_velocity="20"
-                         soft_lower_limit="${0.0 + arm_eps}"
-                         soft_upper_limit="${1.5708 - arm_eps}" />
--->
-  </joint>
+      <parent
+        link="hand_${side}_1_link" />
+      <child
+        link="hand_${side}_2_link" />
+      <axis
+        xyz="0 0 ${-1*reflect}" />
+      <limit
+        lower="0"
+        upper="1.5708"
+        effort="1.0"
+        velocity="2.0" />
+  <!--
+      <dynamics friction="${arm_friction}" damping="${arm_damping}"/>
+      <safety_controller k_position="20"
+                           k_velocity="20"
+                           soft_lower_limit="${0.0 + arm_eps}"
+                           soft_upper_limit="${1.5708 - arm_eps}" />
+  -->
+    </joint>
+  </xacro:if>
    <gazebo reference="${name}_${side}_1_link">
      <mu1>0.9</mu1>
@@ -394,14 +427,16 @@
      <material>Gazebo/DarkGrey</material>
    </gazebo>
-   <gazebo reference="hand_${side}_1_link">
-     <mu1>0.9</mu1>
-     <mu2>0.9</mu2>
-     <material>Gazebo/DarkGrey</material>
-   </gazebo>
-   <gazebo reference="hand_${side}_2_link">
-     <mu1>0.9</mu1>
-     <mu2>0.9</mu2>
-     <material>Gazebo/DarkGrey</material>
-   </gazebo>
+   <xacro:if value="${end_effector}">
+     <gazebo reference="hand_${side}_1_link">
+       <mu1>0.9</mu1>
+       <mu2>0.9</mu2>
+       <material>Gazebo/DarkGrey</material>
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
Commit message: Separate both end effectors

File: ari_description/robots/ari.urdf.xacro (robot description, xacro)
@@ -9,11 +9,16 @@
 <robot  xmlns:xacro="http://ros.org/wiki/xacro"
         name="ari" >
-  <xacro:arg name="ari_end_effector" default="ari_hand"/>
-  <xacro:property name="end_effector" value="$(arg ari_end_effector)" />
+  <xacro:arg name="end_effector_right" default="ari-hand"/>
+  <xacro:arg name="end_effector_left" default="ari-hand"/>
+  <xacro:property name="end_effector_right" value="$(arg end_effector_right)" />
+  <xacro:property name="end_effector_left" value="$(arg end_effector_left)" />
   <xacro:arg name="multiple" default="false"/>
   <xacro:arg name="namespace" default=""/>
   <xacro:property name="is_multiple" value="$(arg multiple)" />
   <xacro:property name="nsp" value="$(arg namespace)" />
-  <xacro:if value="${end_effector not in ['ari_hand', 'false', False]}">
+  <xacro:if value="${end_effector_right not in ['ari-hand', 'false', False]}">
+    <xacro:wrong_end_effector/>
+  </xacro:if>
+  <xacro:if value="${end_effector_left not in ['ari-hand', 'false', False]}">
     <xacro:wrong_end_effector/>
   </xacro:if>
@@ -38,8 +43,8 @@
   <xacro:torso_sensors name="torso" parent="base_link"/>
   <xacro:head name="head" parent="base_link"/>
-  <xacro:ari_arm name="arm" parent="base_link" side="left" reflect="1" end_effector="${end_effector == 'ari_hand'}">
+  <xacro:ari_arm name="arm" parent="base_link" side="left" reflect="1" end_effector="${end_effector_left == 'ari-hand'}">
     <origin xyz="-0.219 0.097624 1.1111" rpy="${105.0 * deg_to_rad} ${0.0 * deg_to_rad} ${-180.0 * deg_to_rad}" />
   </xacro:ari_arm>
-  <xacro:ari_arm name="arm" parent="base_link" side="right" reflect="-1" end_effector="${end_effector == 'ari_hand'}">
+  <xacro:ari_arm name="arm" parent="base_link" side="right" reflect="-1" end_effector="${end_effector_right == 'ari-hand'}">
     <origin xyz="-0.219 -0.097624 1.1111" rpy="${-105.0 * deg_to_rad} ${0.0 * deg_to_rad} ${180.0 * deg_to_rad}" />
   </xacro:ari_arm>

File: ari_description/urdf/arm/arm.urdf.xacro (robot description, xacro)
@@ -330,5 +330,5 @@
       <limit
         lower="0"
-        upper="1.5708"
+        upper="1.35"
         effort="1.0"
         velocity="2.0" />
@@ -468,4 +468,5 @@
                                   start="0.0"
                                   reduction="1.0"/>
+      <!-- <xacro:arm_simple_transmission name="${name}" side="${side}" number="4" reduction="1.0" offset_value="0.0"/> -->
       <!-- gazebo plugin -->
       <xacro:ari_hand_gazebo_simulation side="${side}"/>
