Commit message: Add SPRING cameras

File: ari_description/robots/ari.urdf.xacro (robot description, xacro)
@@ -11,6 +11,8 @@
   <xacro:arg name="end_effector_right" default="ari-hand"/>
   <xacro:arg name="end_effector_left" default="ari-hand"/>
+  <xacro:arg name="spring_cameras" default="false"/>
   <xacro:property name="end_effector_right" value="$(arg end_effector_right)" />
   <xacro:property name="end_effector_left" value="$(arg end_effector_left)" />
+  <xacro:property name="spring_cameras" value="$(arg spring_cameras)" />
   <xacro:arg name="multiple" default="false"/>
   <xacro:arg name="namespace" default=""/>
@@ -22,4 +24,7 @@
   <xacro:if value="${end_effector_left not in ['ari-hand', 'false', False]}">
     <xacro:wrong_end_effector/>
+  </xacro:if>
+  <xacro:if value="${spring_cameras not in ['true', True, 'false', False]}">
+    <xacro:wrong_spring_cameras/>
   </xacro:if>
   <!-- The properties below are modified using empy http://www.alcyone.com/software/empy/

File: ari_description/urdf/torso/torso_sensors.urdf.xacro (robot description, xacro)
@@ -13,4 +13,5 @@
   <xacro:include filename="$(find realsense2_description)/urdf/_t265.urdf.xacro" />
   <xacro:include filename="$(find ari_description)/urdf/sensors/microphone.urdf.xacro"/>
+  <xacro:include filename="$(find ari_description)/urdf/sensors/imx179_camera.gazebo.xacro"/>
   <!--Constant parameters-->
   <xacro:property name="torso_front_camera_position_x" value="-0.11249" />
@@ -38,4 +39,55 @@
             rpy="${torso_back_camera_orientation_r} ${torso_back_camera_orientation_p} ${torso_back_camera_orientation_y}"/>
   </sensor_t265>
+  <!-- Optional SPRING cameras -->
+  <xacro:if value="${spring_cameras}">
+    <!-- Front IMX179 Camera -->
+    <link name="${name}_front_imx_link">
+      <inertial>
+        <origin xyz="0.0 0.0 0.0" rpy="0 0 0"/>
+        <mass value="0.00115745344894968"/>
+        <inertia ixx="6.76913771029748E-08" ixy="2.52492243040059E-13" ixz="-3.60412180500293E-11"
+                 iyy="2.88827920072855E-08" iyz="-1.65336506314803E-13"
+                 izz="3.97290092554434E-08"/>
+      </inertial>
+    </link>
+    <joint name="${name}_front_imx_joint" type="fixed">
+      <origin xyz="-0.1418 0.0 1.1956" rpy="0 ${-39 * deg_to_rad} 0"/>
+      <parent link="${parent}" />
+      <child link="${name}_front_imx_link" />
+      <axis xyz="0 0 0" />
+    </joint>
+    <joint name="${name}_front_imx_optical_joint" type="fixed">
+      <origin xyz="0.0 0.0 0.0" rpy="${-90 * deg_to_rad} 0 ${-90 * deg_to_rad}" />
+      <parent link="${name}_front_imx_link" />
+      <child link="${name}_front_imx_optical_frame" />
+      <axis xyz="0 0 0" />
+    </joint>
+    <link name="${name}_front_imx_optical_frame"/>
+    <xacro:imx179_camera_gazebo name="${name}_front_imx" topic="${name}_front_imx" frame="${name}_front_imx_optical_frame"/>
+    <!-- Back IMX179 Camera -->
+    <link name="${name}_back_imx_link">
+      <inertial>
+        <origin xyz="0.0 0.0 0.0" rpy="0 0 0"/>
+        <mass value="0.00115745344894968"/>
+        <inertia ixx="6.76913771029748E-08" ixy="2.52492243040059E-13" ixz="-3.60412180500293E-11"
+                 iyy="2.88827920072855E-08" iyz="-1.65336506314803E-13"
+                 izz="3.97290092554434E-08"/>
+      </inertial>
+    </link>
+    <joint name="${name}_back_imx_joint" type="fixed">
+      <origin xyz="-0.3209 0.0 1.1634" rpy="0 ${-25 * deg_to_rad} ${-180 * deg_to_rad}" />
+      <parent link="${parent}" />
+      <child link="${name}_back_imx_link" />
+      <axis xyz="0 0 0" />
+    </joint>
+    <joint name="${name}_back_imx_optical_joint" type="fixed">
+      <origin xyz="0.0 0.0 0.0" rpy="${-90 * deg_to_rad} 0 ${-90 * deg_to_rad}" />
+      <parent link="${name}_back_imx_link" />
+      <child link="${name}_back_imx_optical_frame" />
+      <axis xyz="0 0 0" />
+    </joint>
+    <link name="${name}_back_imx_optical_frame"/>
+    <xacro:imx179_camera_gazebo name="${name}_back_imx" topic="${name}_back_imx" frame="${name}_back_imx_optical_frame"/>
+  </xacro:if>
   <!-- Microphones -->
   <xacro:microphone name="${name}_mic_front" parent="${parent}">

Commit message: Change to support sick-571 laser in ari3

File: ari_description/robots/ari.urdf.xacro (robot description, xacro)
@@ -28,4 +28,14 @@
     <xacro:wrong_spring_cameras/>
   </xacro:if>
+  <xacro:arg name="laser_model" default="sick-571"/> <!-- false, hokuyo, sick-551, sick-561, sick-571-->
+  <xacro:arg name="rgbd_sensors" default="false"/> <!-- false, true-->
+  <xacro:property name="laser_model" value="$(arg laser_model)" />
+  <xacro:property name="rgbd_sensors" value="$(arg rgbd_sensors)"/>
+  <xacro:if value="${laser_model not in ['false', False, 'sick-551', 'sick-561', 'sick-571', 'hokuyo']}">
+    <xacro:wrong_laser_model/>
+  </xacro:if>
+  <!-- The following included files set up definitions of parts of the robot body -->
+  <!-- Base -->
+  <xacro:include filename="$(find ari_description)/urdf/base/base_sensors.urdf.xacro" />
   <!-- The properties below are modified using empy http://www.alcyone.com/software/empy/
        from the create_robot.py tool. Handle them with care -->
@@ -33,5 +43,5 @@
   <!-- The following included files set up definitions of parts of the robot base -->
   <!-- Base -->
-  <xacro:include filename="$(find ari_description)/urdf/base/base.urdf.xacro" />
+   <xacro:base_sensors name="base" laser_model="$(arg laser_model)" sonars="true"/>
   <!-- Torso -->
   <xacro:include filename="$(find ari_description)/urdf/torso/torso_sensors.urdf.xacro" />
@@ -45,5 +55,4 @@
   <xacro:include filename="$(find ari_description)/urdf/materials.urdf.xacro" />
   <!-- Now we can start using the macros included above to define the actual robot -->
-  <xacro:base name="base"/>
   <xacro:torso_sensors name="torso" parent="base_link"/>
   <xacro:head name="head" parent="base_link"/>

Commit message: Add camera model param and fix location

File: ari_description/robots/ari.urdf.xacro (robot description, xacro)
@@ -30,4 +30,7 @@
     <xacro:wrong_spring_cameras/>
   </xacro:if>
+  <xacro:if value="${camera_model not in ['head-rgb', 'head-rgbd']}">
+    <xacro:wrong_camera_model/>
+  </xacro:if>
   <xacro:arg name="laser_model" default="sick-571"/> <!-- false, hokuyo, sick-551, sick-561, sick-571-->
   <xacro:arg name="rgbd_sensors" default="false"/> <!-- false, true-->
@@ -37,10 +40,10 @@
     <xacro:wrong_laser_model/>
   </xacro:if>
+  <!-- The properties below are modified using empy http://www.alcyone.com/software/empy/
+       from the create_robot.py tool. Handle them with care -->
+  <xacro:property name="head_link_name"          value="head_2_link"/>
   <!-- The following included files set up definitions of parts of the robot body -->
   <!-- Base -->
   <xacro:include filename="$(find ari_description)/urdf/base/base.urdf.xacro" />
-  <!-- The properties below are modified using empy http://www.alcyone.com/software/empy/
-       from the create_robot.py tool. Handle them with care -->
-  <xacro:property name="head_link_name"          value="head_2_link"/>
   <!-- The following included files set up definitions of parts of the robot base -->
   <!-- Torso -->

Commit message: fixing stuff

File: ari_description/robots/ari.urdf.xacro (robot description, xacro)
@@ -37,11 +37,9 @@
   <!-- The following included files set up definitions of parts of the robot body -->
   <!-- Base -->
-  <xacro:include filename="$(find ari_description)/urdf/base/base_sensors.urdf.xacro" />
+  <xacro:include filename="$(find ari_description)/urdf/base/base.urdf.xacro" />
   <!-- The properties below are modified using empy http://www.alcyone.com/software/empy/
        from the create_robot.py tool. Handle them with care -->
   <xacro:property name="head_link_name"          value="head_2_link"/>
   <!-- The following included files set up definitions of parts of the robot base -->
-  <!-- Base -->
-   <xacro:base_sensors name="base" laser_model="$(arg laser_model)" sonars="true"/>
   <!-- Torso -->
   <xacro:include filename="$(find ari_description)/urdf/torso/torso_sensors.urdf.xacro" />
@@ -55,4 +53,5 @@
   <xacro:include filename="$(find ari_description)/urdf/materials.urdf.xacro" />
   <!-- Now we can start using the macros included above to define the actual robot -->
+  <xacro:base name="base"/>
   <xacro:torso_sensors name="torso" parent="base_link"/>
   <xacro:head name="head" parent="base_link"/>

File: ari_description/urdf/sensors/sick_tim571_laser.urdf.xacro (robot description, xacro)
@@ -29,5 +29,5 @@
       <axis xyz="0 1 0"/>
       <xacro:insert_block name="origin"/>
-      <parent link="${parent}_link"/>
+      <parent link="${parent}"/>
       <child  link="${name}_link"/>
     </joint>

File: ari_description/urdf/torso/torso_sensors.urdf.xacro (robot description, xacro)
@@ -14,4 +14,5 @@
   <xacro:include filename="$(find ari_description)/urdf/sensors/microphone.urdf.xacro"/>
   <xacro:include filename="$(find ari_description)/urdf/sensors/imx179_camera.gazebo.xacro"/>
+  <xacro:include filename="$(find ari_description)/urdf/sensors/sick_tim571_laser.urdf.xacro"/>
   <!--Constant parameters-->
   <xacro:property name="torso_front_camera_position_x" value="-0.11249" />
@@ -27,4 +28,8 @@
   <xacro:property name="torso_back_camera_orientation_p" value="${15 * deg_to_rad}" />
   <xacro:property name="torso_back_camera_orientation_y" value="${180 * deg_to_rad}" />
+  <!-- Laser characteristics -->
+  <xacro:property name="base_laser_x" value="-0.334"/>
+  <xacro:property name="base_laser_y" value="0.0"/>
+  <xacro:property name="base_laser_z" value="0.565"/>
   <xacro:macro name="torso_sensors" params="name parent">
   <!-- Torso sensors -->
@@ -94,4 +99,11 @@
     <origin xyz="-0.12173 -3.5497E-05 0.80332" rpy="${80 * deg_to_rad} 0 ${90 * deg_to_rad}"/>
   </xacro:microphone>
+  <xacro:if value="${laser_model == 'sick-571'}">
+    <!-- Laser -->
+    <!-- Theoretic FOV = 220 -->
+    <xacro:sick_tim571_laser name="${name}_laser" parent="${parent}" ros_topic="scan_raw" update_rate="10" min_angle="${-110 * deg_to_rad}" max_angle="${110 * deg_to_rad}" >
+      <origin xyz="${base_laser_x} ${base_laser_y} ${base_laser_z}" rpy="0 0 ${ 180 * deg_to_rad }" />
+    </xacro:sick_tim571_laser>
+  </xacro:if>
  </xacro:macro>
 </robot>

Commit message: Added laser_model dependencies

File: ari_description/robots/ari.urdf.xacro (robot description, xacro)
@@ -12,7 +12,9 @@
   <xacro:arg name="end_effector_left" default="ari-hand"/>
   <xacro:arg name="spring_cameras" default="false"/>
+  <xacro:arg name="camera_model" default="head-rgb"/>
   <xacro:property name="end_effector_right" value="$(arg end_effector_right)" />
   <xacro:property name="end_effector_left" value="$(arg end_effector_left)" />
   <xacro:property name="spring_cameras" value="$(arg spring_cameras)" />
+  <xacro:property name="camera_model" value="$(arg camera_model)"/>
   <xacro:arg name="multiple" default="false"/>
   <xacro:arg name="namespace" default=""/>
@@ -28,20 +30,18 @@
     <xacro:wrong_spring_cameras/>
   </xacro:if>
-  <xacro:arg name="laser_model" default="sick-571"/> <!-- false, hokuyo, sick-551, sick-561, sick-571-->
+  <xacro:arg name="laser_model" default="false"/> <!-- false, hokuyo, sick-551, sick-561, sick-571-->
   <xacro:arg name="rgbd_sensors" default="false"/> <!-- false, true-->
   <xacro:property name="laser_model" value="$(arg laser_model)" />
   <xacro:property name="rgbd_sensors" value="$(arg rgbd_sensors)"/>
-  <xacro:if value="${laser_model not in ['false', False, 'sick-551', 'sick-561', 'sick-571', 'hokuyo']}">
+  <xacro:if value="${laser_model not in ['No', 'false', False, 'sick-551', 'sick-561', 'sick-571', 'hokuyo']}">
     <xacro:wrong_laser_model/>
   </xacro:if>
-  <!-- The following included files set up definitions of parts of the robot body -->
-  <!-- Base -->
-  <xacro:include filename="$(find ari_description)/urdf/base/base_sensors.urdf.xacro" />
   <!-- The properties below are modified using empy http://www.alcyone.com/software/empy/
        from the create_robot.py tool. Handle them with care -->
   <xacro:property name="head_link_name"          value="head_2_link"/>
+  <!-- The following included files set up definitions of parts of the robot body -->
+  <!-- Base -->
+  <xacro:include filename="$(find ari_description)/urdf/base/base.urdf.xacro" />
   <!-- The following included files set up definitions of parts of the robot base -->
-  <!-- Base -->
-   <xacro:base_sensors name="base" laser_model="$(arg laser_model)" sonars="true"/>
   <!-- Torso -->
   <xacro:include filename="$(find ari_description)/urdf/torso/torso_sensors.urdf.xacro" />
@@ -55,4 +55,5 @@
   <xacro:include filename="$(find ari_description)/urdf/materials.urdf.xacro" />
   <!-- Now we can start using the macros included above to define the actual robot -->
+  <xacro:base name="base"/>
   <xacro:torso_sensors name="torso" parent="base_link"/>
   <xacro:head name="head" parent="base_link"/>

Commit message: Rename camera param and pass laser

File: ari_description/robots/ari.urdf.xacro (robot description, xacro)
@@ -12,9 +12,9 @@
   <xacro:arg name="end_effector_left" default="ari-hand"/>
   <xacro:arg name="spring_cameras" default="false"/>
-  <xacro:arg name="camera_model" default="head-rgb"/>
+  <xacro:arg name="camera_model_head" default="raspi"/>
   <xacro:property name="end_effector_right" value="$(arg end_effector_right)" />
   <xacro:property name="end_effector_left" value="$(arg end_effector_left)" />
   <xacro:property name="spring_cameras" value="$(arg spring_cameras)" />
-  <xacro:property name="camera_model" value="$(arg camera_model)"/>
+  <xacro:property name="camera_model_head" value="$(arg camera_model_head)"/>
   <xacro:arg name="multiple" default="false"/>
   <xacro:arg name="namespace" default=""/>
@@ -30,5 +30,5 @@
     <xacro:wrong_spring_cameras/>
   </xacro:if>
-  <xacro:if value="${camera_model not in ['head-rgb', 'head-rgbd']}">
+  <xacro:if value="${camera_model_head not in ['raspi', 'D435i']}">
     <xacro:wrong_camera_model/>
   </xacro:if>

File: ari_description/urdf/head/head.urdf.xacro (robot description, xacro)
@@ -206,8 +206,8 @@
     <xacro:head_1 name="${name}_1" parent="${parent}" />
     <xacro:head_2 name="${name}_2" parent="${name}_1_link"/>
-    <xacro:if value="${camera_model == 'head-rgb'}">
+    <xacro:if value="${camera_model_head == 'raspi'}">
       <xacro:head_front_camera name="${name}_front_camera" parent="${name}_2_link"/>
     </xacro:if>
-    <xacro:if value="${camera_model == 'head-rgbd'}">
+    <xacro:if value="${camera_model_head == 'D435i'}">
       <xacro:head_rgbd name="${name}_rgbd" parent="${name}_2_link"/>
     </xacro:if>

Commit message: Use separated fisheye params

File: ari_description/robots/ari.urdf.xacro (robot description, xacro)
@@ -11,9 +11,11 @@
   <xacro:arg name="end_effector_right" default="ari-hand"/>
   <xacro:arg name="end_effector_left" default="ari-hand"/>
-  <xacro:arg name="spring_cameras" default="false"/>
+  <xacro:arg name="front_fisheye_camera" default="false"/>
+  <xacro:arg name="back_fisheye_camera" default="false"/>
   <xacro:arg name="camera_model_head" default="raspi"/>
   <xacro:property name="end_effector_right" value="$(arg end_effector_right)" />
   <xacro:property name="end_effector_left" value="$(arg end_effector_left)" />
-  <xacro:property name="spring_cameras" value="$(arg spring_cameras)" />
+  <xacro:property name="front_fisheye_camera" value="$(arg front_fisheye_camera)" />
+  <xacro:property name="back_fisheye_camera" value="$(arg back_fisheye_camera)" />
   <xacro:property name="camera_model_head" value="$(arg camera_model_head)"/>
   <xacro:arg name="multiple" default="false"/>
@@ -27,6 +29,9 @@
     <xacro:wrong_end_effector/>
   </xacro:if>
-  <xacro:if value="${spring_cameras not in ['true', True, 'false', False]}">
-    <xacro:wrong_spring_cameras/>
+  <xacro:if value="${front_fisheye_camera not in ['true', True, 'false', False]}">
+    <xacro:wrong_front_fisheye_camera/>
+  </xacro:if>
+  <xacro:if value="${back_fisheye_camera not in ['true', True, 'false', False]}">
+    <xacro:wrong_back_fisheye_camera/>
   </xacro:if>
   <xacro:if value="${camera_model_head not in ['raspi', 'D435i']}">

File: ari_description/urdf/torso/torso_sensors.urdf.xacro (robot description, xacro)
@@ -45,7 +45,7 @@
   </sensor_t265>
   <!-- Optional SPRING cameras -->
-  <xacro:if value="${spring_cameras}">
+  <xacro:if value="${front_fisheye_camera}">
     <!-- Front IMX179 Camera -->
-    <link name="${name}_front_imx_link">
+    <link name="front_fisheye_camera_link">
       <inertial>
         <origin xyz="0.0 0.0 0.0" rpy="0 0 0"/>
@@ -56,20 +56,22 @@
       </inertial>
     </link>
-    <joint name="${name}_front_imx_joint" type="fixed">
+    <joint name="front_fisheye_camera_joint" type="fixed">
       <origin xyz="-0.1418 0.0 1.1956" rpy="0 ${-39 * deg_to_rad} 0"/>
       <parent link="${parent}" />
-      <child link="${name}_front_imx_link" />
+      <child link="front_fisheye_camera_link" />
       <axis xyz="0 0 0" />
     </joint>
-    <joint name="${name}_front_imx_optical_joint" type="fixed">
+    <joint name="front_fisheye_camera_optical_joint" type="fixed">
       <origin xyz="0.0 0.0 0.0" rpy="${-90 * deg_to_rad} 0 ${-90 * deg_to_rad}" />
-      <parent link="${name}_front_imx_link" />
-      <child link="${name}_front_imx_optical_frame" />
+      <parent link="front_fisheye_camera_link" />
+      <child link="front_fisheye_camera_optical_frame" />
       <axis xyz="0 0 0" />
     </joint>
-    <link name="${name}_front_imx_optical_frame"/>
-    <xacro:imx179_camera_gazebo name="${name}_front_imx" topic="${name}_front_imx" frame="${name}_front_imx_optical_frame"/>
+    <link name="front_fisheye_camera_optical_frame"/>
+    <xacro:imx179_camera_gazebo name="front_fisheye_camera" topic="front_fisheye_camera" frame="front_fisheye_camera_optical_frame"/>
+  </xacro:if>
+  <xacro:if value="${back_fisheye_camera}">
     <!-- Back IMX179 Camera -->
-    <link name="${name}_back_imx_link">
+    <link name="rear_fisheye_camera_link">
       <inertial>
         <origin xyz="0.0 0.0 0.0" rpy="0 0 0"/>
@@ -80,18 +82,18 @@
       </inertial>
     </link>
-    <joint name="${name}_back_imx_joint" type="fixed">
+    <joint name="rear_fisheye_camera_joint" type="fixed">
       <origin xyz="-0.3209 0.0 1.1634" rpy="0 ${-25 * deg_to_rad} ${-180 * deg_to_rad}" />
       <parent link="${parent}" />
-      <child link="${name}_back_imx_link" />
+      <child link="rear_fisheye_camera_link" />
       <axis xyz="0 0 0" />
     </joint>
-    <joint name="${name}_back_imx_optical_joint" type="fixed">
+    <joint name="rear_fisheye_camera_optical_joint" type="fixed">
       <origin xyz="0.0 0.0 0.0" rpy="${-90 * deg_to_rad} 0 ${-90 * deg_to_rad}" />
-      <parent link="${name}_back_imx_link" />
-      <child link="${name}_back_imx_optical_frame" />
+      <parent link="rear_fisheye_camera_link" />
+      <child link="rear_fisheye_camera_optical_frame" />
       <axis xyz="0 0 0" />
     </joint>
-    <link name="${name}_back_imx_optical_frame"/>
-    <xacro:imx179_camera_gazebo name="${name}_back_imx" topic="${name}_back_imx" frame="${name}_back_imx_optical_frame"/>
+    <link name="rear_fisheye_camera_optical_frame"/>
+    <xacro:imx179_camera_gazebo name="rear_fisheye_camera" topic="rear_fisheye_camera" frame="rear_fisheye_camera_optical_frame"/>
   </xacro:if>
   <!-- Microphones -->

Commit message: Proper handling of string parameters for fisheye camera

File: ari_description/robots/ari.urdf.xacro (robot description, xacro)
@@ -29,8 +29,8 @@
     <xacro:wrong_end_effector/>
   </xacro:if>
-  <xacro:if value="${front_fisheye_camera not in ['true', True, 'false', False]}">
+  <xacro:if value="${front_fisheye_camera not in ['true', True, 'false', False, 'Jetson']}">
     <xacro:wrong_front_fisheye_camera/>
   </xacro:if>
-  <xacro:if value="${back_fisheye_camera not in ['true', True, 'false', False]}">
+  <xacro:if value="${back_fisheye_camera not in ['true', True, 'false', False, 'Jetson']}">
     <xacro:wrong_back_fisheye_camera/>
   </xacro:if>
@@ -42,4 +42,6 @@
   <xacro:property name="laser_model" value="$(arg laser_model)" />
   <xacro:property name="rgbd_sensors" value="$(arg rgbd_sensors)"/>
+  <xacro:property name="has_front_fisheye_camera"           value="${front_fisheye_camera in ['Jetson', True, 'true', 'PC']}"/>
+  <xacro:property name="has_back_fisheye_camera"           value="${back_fisheye_camera in ['Jetson', True, 'true', 'PC']}"/>
   <xacro:if value="${laser_model not in ['No', 'false', False, 'sick-551', 'sick-561', 'sick-571', 'hokuyo']}">
     <xacro:wrong_laser_model/>

File: ari_description/urdf/torso/torso_sensors.urdf.xacro (robot description, xacro)
@@ -45,5 +45,5 @@
   </sensor_t265>
   <!-- Optional SPRING cameras -->
-  <xacro:if value="${front_fisheye_camera}">
+  <xacro:if value="${has_front_fisheye_camera}">
     <!-- Front IMX179 Camera -->
     <link name="front_fisheye_camera_link">
@@ -71,5 +71,5 @@
     <xacro:imx179_camera_gazebo name="front_fisheye_camera" topic="front_fisheye_camera" frame="front_fisheye_camera_optical_frame"/>
   </xacro:if>
-  <xacro:if value="${back_fisheye_camera}">
+  <xacro:if value="${has_back_fisheye_camera}">
     <!-- Back IMX179 Camera -->
     <link name="rear_fisheye_camera_link">
