Commit message: add has thermal parameter and tf link

File: ari_description/robots/ari.urdf.xacro (robot description, xacro)
@@ -14,4 +14,5 @@
   <xacro:arg name="back_fisheye_camera" default="false"/>
   <xacro:arg name="camera_model_head" default="raspi"/>
+  <xacro:arg name="has_thermal" default="false"/>
   <xacro:property name="end_effector_right" value="$(arg end_effector_right)" />
   <xacro:property name="end_effector_left" value="$(arg end_effector_left)" />
@@ -19,4 +20,5 @@
   <xacro:property name="back_fisheye_camera" value="$(arg back_fisheye_camera)" />
   <xacro:property name="camera_model_head" value="$(arg camera_model_head)"/>
+  <xacro:property name="has_thermal" value="$(arg has_thermal)"/>
   <xacro:arg name="multiple" default="false"/>
   <xacro:arg name="namespace" default=""/>
@@ -37,4 +39,7 @@
   <xacro:if value="${camera_model_head not in ['raspi', 'D435i']}">
     <xacro:wrong_camera_model/>
+  </xacro:if>
+  <xacro:if value="${has_thermal not in ['true', True, 'false', False]}">
+    <xacro:wrong_thermal_camera/>
   </xacro:if>
   <xacro:arg name="laser_model" default="false"/> <!-- false, hokuyo, sick-551, sick-561, sick-571-->

File: ari_description/urdf/head/head.urdf.xacro (robot description, xacro)
@@ -175,4 +175,19 @@
   <xacro:rpi_camera_gazebo name="${name}" topic="${name}/color" frame="${name}_color_optical_frame"/>
   </xacro:macro>
+  <!-- Optional thermal camera -->
+  <xacro:macro name="thermal_camera" params="name parent">
+    <joint name="thermal_camera_joint" type="fixed">
+        <parent link="${parent}"/>
+        <child link="thermal_camera"/>
+        <origin xyz="0.05 0.15 0" rpy="${0*deg_to_rad} ${-90*deg_to_rad} ${-180*deg_to_rad}" />
+    </joint>
+    <link name="thermal_camera">
+        <inertial>
+            <origin xyz="0 0 0" rpy="0 0 0"/>
+            <mass value="0.0001" />
+            <inertia ixx="0.0001"  ixy="0"  ixz="0" iyy="0.0001" iyz="0" izz="0.0001" />
+        </inertial>
+    </link>
+  </xacro:macro>
   <joint name="ear_led_left_link" type="fixed">
     <origin xyz="0.021 0.095 0.192" rpy="-0.1 0 0.0" />
@@ -212,4 +227,7 @@
       <xacro:head_rgbd name="${name}_rgbd" parent="${name}_2_link"/>
     </xacro:if>
+    <xacro:if value="${(has_thermal == 'true') or (has_thermal == True) }">
+      <xacro:thermal_camera name="thermal_camera" parent="${name}_2_link"/>
+    </xacro:if>
  </xacro:macro>
 </robot>

Commit message: include urdf for ari_v2

File: ari_description/robots/ari.urdf.xacro (robot description, xacro)
@@ -9,4 +9,5 @@
 <robot  xmlns:xacro="http://ros.org/wiki/xacro"
         name="ari" >
+  <xacro:arg name="version" default="v1"/>
   <xacro:arg name="end_effector_right" default="ari-hand"/>
   <xacro:arg name="end_effector_left" default="ari-hand"/>
@@ -15,4 +16,5 @@
   <xacro:arg name="camera_model_head" default="raspi"/>
   <xacro:arg name="has_thermal" default="false"/>
+  <xacro:property name="version" value="$(arg version)" />
   <xacro:property name="end_effector_right" value="$(arg end_effector_right)" />
   <xacro:property name="end_effector_left" value="$(arg end_effector_left)" />
@@ -25,4 +27,7 @@
   <xacro:property name="is_multiple" value="$(arg multiple)" />
   <xacro:property name="nsp" value="$(arg namespace)" />
+  <xacro:if value="${version not in ['v1', 'v2']}">
+    <xacro:wrong_ari_version/>
+  </xacro:if>
   <xacro:if value="${end_effector_right not in ['ari-hand', 'false', False]}">
     <xacro:wrong_end_effector/>
@@ -56,13 +61,16 @@
   <xacro:property name="head_link_name"          value="head_2_link"/>
   <!-- The following included files set up definitions of parts of the robot body -->
-  <!-- Base -->
-  <xacro:include filename="$(find ari_description)/urdf/base/base.urdf.xacro" />
-  <!-- The following included files set up definitions of parts of the robot base -->
-  <!-- Torso -->
-  <xacro:include filename="$(find ari_description)/urdf/torso/torso_sensors.urdf.xacro" />
-  <!-- Arm -->
-  <xacro:include filename="$(find ari_description)/urdf/arm/arm.urdf.xacro" />
-  <!-- Head -->
-  <xacro:include filename="$(find ari_description)/urdf/head/head.urdf.xacro" />
+  <xacro:if value="${version == 'v1'}">
+      <xacro:include filename="$(find ari_description)/urdf/base/base.urdf.xacro" />   <!-- Base -->
+      <xacro:include filename="$(find ari_description)/urdf/torso/torso_sensors.urdf.xacro" /> <!-- Torso -->
+      <xacro:include filename="$(find ari_description)/urdf/arm/arm.urdf.xacro" />   <!-- Arms -->
+      <xacro:include filename="$(find ari_description)/urdf/head/head.urdf.xacro" /> <!-- head -->
+  </xacro:if>
+  <xacro:if value="${version == 'v2'}">
+      <xacro:include filename="$(find ari_description)/urdf/base/base_v2.urdf.xacro" />   <!-- Base -->
+      <xacro:include filename="$(find ari_description)/urdf/torso/torso_sensors_v2.urdf.xacro" /> <!-- Torso -->
+      <xacro:include filename="$(find ari_description)/urdf/arm/arm_v2.urdf.xacro" />   <!-- Arms -->
+      <xacro:include filename="$(find ari_description)/urdf/head/head_v2.urdf.xacro" /> <!-- head -->
+  </xacro:if>
   <!-- Generic simulator_gazebo plugins -->
   <xacro:include filename="$(find ari_description)/gazebo/gazebo.urdf.xacro" />
@@ -73,4 +81,5 @@
   <xacro:torso_sensors name="torso" parent="base_link"/>
   <xacro:head name="head" parent="base_link"/>
+  <xacro:if value="${version == 'v1'}">
   <xacro:ari_arm name="arm" parent="base_link" side="left" reflect="1" end_effector="${end_effector_left == 'ari-hand'}">
     <origin xyz="-0.219 0.097624 1.1111" rpy="${105.0 * deg_to_rad} ${0.0 * deg_to_rad} ${-180.0 * deg_to_rad}" />
@@ -79,3 +88,12 @@
     <origin xyz="-0.219 -0.097624 1.1111" rpy="${-105.0 * deg_to_rad} ${0.0 * deg_to_rad} ${180.0 * deg_to_rad}" />
   </xacro:ari_arm>
+  </xacro:if>
+  <xacro:if value="${version == 'v2'}">
+  <xacro:ari_arm name="arm" parent="base_link" side="left" reflect="1" end_effector="${end_effector_left == 'ari-hand'}">
+    <origin xyz="-0.22 0.08146 1.153" rpy="${170.0 * deg_to_rad} ${180 * deg_to_rad} ${-180.0 * deg_to_rad}" />
+  </xacro:ari_arm>
+  <xacro:ari_arm name="arm" parent="base_link" side="right" reflect="-1" end_effector="${end_effector_right == 'ari-hand'}">
+    <origin xyz="-0.22 -0.08146 1.153" rpy="${20.0 * deg_to_rad} ${180 * deg_to_rad} ${180.0 * deg_to_rad}" />
+  </xacro:ari_arm>
+  </xacro:if>
 </robot>

Commit message: reflect arm_base_link in z-axis

File: ari_description/robots/ari.urdf.xacro (robot description, xacro)
@@ -66,4 +66,5 @@
       <xacro:include filename="$(find ari_description)/urdf/arm/arm.urdf.xacro" />   <!-- Arms -->
       <xacro:include filename="$(find ari_description)/urdf/head/head.urdf.xacro" /> <!-- head -->
+      <xacro:include filename="$(find ari_description)/urdf/arm/arm_v2.urdf.xacro" />   <!-- Arms -->
   </xacro:if>
   <xacro:if value="${version == 'v2'}">
@@ -89,11 +90,11 @@
   </xacro:ari_arm>
   </xacro:if>
-  <xacro:if value="${version == 'v2'}">
-  <xacro:ari_arm name="arm" parent="base_link" side="left" reflect="1" end_effector="${end_effector_left == 'ari-hand'}">
-    <origin xyz="-0.22 0.08146 1.153" rpy="${170.0 * deg_to_rad} ${180 * deg_to_rad} ${-180.0 * deg_to_rad}" />
-  </xacro:ari_arm>
-  <xacro:ari_arm name="arm" parent="base_link" side="right" reflect="-1" end_effector="${end_effector_right == 'ari-hand'}">
-    <origin xyz="-0.22 -0.08146 1.153" rpy="${20.0 * deg_to_rad} ${180 * deg_to_rad} ${180.0 * deg_to_rad}" />
-  </xacro:ari_arm>
+  <xacro:if value="${version == 'v1'}">
+  <xacro:ari_arm_v2 name="arm_2" parent="base_link" side="left" reflect="1" end_effector="${end_effector_left == 'ari-hand'}">
+    <origin xyz="-0.22 0.08146 1.153" rpy="${-10 * deg_to_rad} ${0 * deg_to_rad} ${0.0 * deg_to_rad}" />
+  </xacro:ari_arm_v2>
+  <xacro:ari_arm_v2 name="arm_2" parent="base_link" side="right" reflect="-1" end_effector="${end_effector_right == 'ari-hand'}">
+    <origin xyz="-0.22 -0.08146 1.153" rpy="${-200 * deg_to_rad} ${00 * deg_to_rad} ${0.0 * deg_to_rad}" />
+  </xacro:ari_arm_v2>
   </xacro:if>
 </robot>

File: ari_description/urdf/arm/arm_v2.urdf.xacro (robot description, xacro)
@@ -10,6 +10,6 @@
   <!--File includes-->
   <xacro:include filename="$(find ari_description)/urdf/deg_to_rad.xacro" />
-  <xacro:include filename="$(find ari_description)/urdf/arm/actuators_v2.urdf.xacro" />
-  <xacro:include filename="$(find ari_description)/urdf/arm/arm_v2.transmission.xacro" />
+  <xacro:include filename="$(find ari_description)/urdf/arm/actuators.urdf.xacro" />
+  <xacro:include filename="$(find ari_description)/urdf/arm/arm.transmission.xacro" />
   <!--Constant parameters-->
   <xacro:property name="arm_friction"       value="1.0" />
@@ -24,5 +24,5 @@
   <xacro:property name="arm_4_max_effort"   value="5" />
   <xacro:property name="arm_eps"            value="0.07" />
-  <xacro:macro name="ari_arm" params="name parent side reflect end_effector *origin">
+  <xacro:macro name="ari_arm_v2" params="name parent side reflect end_effector *origin">
     <!--************************-->
     <!--      ARM_BASE_LINK     -->
@@ -46,8 +46,8 @@
       <origin
         xyz="0 0 0"
-        rpy="0 0 0" />
+        rpy="${0 * deg_to_rad * reflect} ${0 * deg_to_rad} 0" />
       <geometry>
         <mesh
-          filename="package://ari_left_arm/meshes/arm_left_base_link.STL" />
+          filename="package://ari_left_arm/meshes/arm_left_base_link.STL" scale="1 1 ${reflect} "/>
       </geometry>
       <material
@@ -63,5 +63,5 @@
       <geometry>
         <mesh
-          filename="package://ari_left_arm/meshes/arm_left_base_link.STL" />
+          filename="package://ari_left_arm/meshes/arm_left_base_link.STL" scale="1 1 ${reflect}"/>
       </geometry>
     </collision>
@@ -78,5 +78,5 @@
 <inertial>
       <origin
-        xyz="-0.00734678702660377 -2.69505911157866E-06 0.0810729999795757"
+        xyz="-0.00734678702660377 ${-2.69505911157866E-06 * reflect} 0.0810729999795757"
         rpy="0 0 0" />
       <mass
@@ -109,5 +109,5 @@
     <origin
       xyz="0 0.0047319 -0.00041399"
-      rpy="-1.6581 0 0" />
+      rpy="${(-95.002132011 + 0) * deg_to_rad * reflect} 0 0" />
        <axis xyz="0 0 ${-1*reflect}" />
       <limit lower="-2.09" upper="2.09" effort="0" velocity="0" />
@@ -196,5 +196,5 @@
       xyz="-0.023833 ${0.1003 * reflect} -0.008"
       rpy="${1.4835 * reflect} 1.5708 0" />
-      <axis xyz="0 0 ${-1*reflect}" />
+      <axis xyz="0 0 ${1*reflect}" />
       <limit lower="-2.09" upper="2.09" effort="${arm_3_max_effort}" velocity="${arm_3_max_vel}" />
       <dynamics friction="${arm_friction}" damping="${arm_damping}"/>
@@ -272,6 +272,6 @@
     <origin
       xyz="0 ${0.00049107 * reflect} -0.1001"
-      rpy="1.5708 -1.5708 0" />
-      <axis xyz="0 0 ${-1*reflect}" />
+      rpy="${1.5708 * reflect} ${-1.5708 * reflect} 0" />
+      <axis xyz="0 0 ${1*reflect}" />
       <xacro:property name="arm_4_upper_limit"       value="135.0"/>
       <xacro:property name="arm_4_lower_limit"       value="-5.0"/>
@@ -318,5 +318,5 @@
       xyz="-0.106 ${0 * reflect} 0.0010076"
       rpy="-1.5708 0 -1.5708" />
-      <axis xyz="0 0 ${-1*reflect}" />
+      <axis xyz="0 0 ${1*reflect}" />
       <xacro:property name="arm_5_upper_limit"       value="135.0"/>
       <xacro:property name="arm_5_lower_limit"       value="-5.0"/>
