Commit message: new_arm direct copy of left-arm.urdf

File: ari_description/robots/ari.urdf.xacro (robot description, xacro)
@@ -92,8 +92,8 @@
   <xacro:if value="${version == 'v1'}">
   <xacro:ari_arm_v2 name="arm_2" parent="base_link" side="left" reflect="1" end_effector="${end_effector_left == 'ari-hand'}">
-    <origin xyz="-0.22 0.08146 1.153" rpy="${-10 * deg_to_rad} ${0 * deg_to_rad} ${0.0 * deg_to_rad}" />
+    <origin xyz="-0.22 0.08146 1.153" rpy="${105 * deg_to_rad} ${0 * deg_to_rad} ${180 * deg_to_rad}" />
   </xacro:ari_arm_v2>
   <xacro:ari_arm_v2 name="arm_2" parent="base_link" side="right" reflect="-1" end_effector="${end_effector_right == 'ari-hand'}">
-    <origin xyz="-0.22 -0.08146 1.153" rpy="${-200 * deg_to_rad} ${00 * deg_to_rad} ${0.0 * deg_to_rad}" />
+    <origin xyz="-0.22 -0.08146 1.153" rpy="${105 * deg_to_rad} ${0 * deg_to_rad} ${-180 * deg_to_rad}" />
   </xacro:ari_arm_v2>
   </xacro:if>

File: ari_description/urdf/arm/arm_v2.urdf.xacro (robot description, xacro)
@@ -29,41 +29,27 @@
     <!--************************-->
     <link name="${name}_${side}_base_link">
-    <inertial>
-      <origin
-        xyz="0.00705797129984277 -0.0045072380254732 0.000352877816427871"
-        rpy="0 0 0" />
-      <mass
-        value="0.481395506498302" />
-      <inertia
-        ixx="0.00022416049267238"
-        ixy="-4.61763481387137E-07"
-        ixz="3.15922577645587E-08"
-        iyy="0.000454778831736013"
-        iyz="-1.22837579712493E-05"
-        izz="0.000315397102146471" />
-    </inertial>
-    <visual>
-      <origin
-        xyz="0 0 0"
-        rpy="${0 * deg_to_rad * reflect} ${0 * deg_to_rad} 0" />
-      <geometry>
-        <mesh
-          filename="package://ari_left_arm/meshes/arm_left_base_link.STL" scale="1 1 ${reflect} "/>
-      </geometry>
-      <material
-        name="">
-        <color
-          rgba="0.250980392156863 0.250980392156863 0.250980392156863 1" />
-      </material>
-    </visual>
-    <collision>
-      <origin
-        xyz="0 0 0"
-        rpy="0 0 0" />
-      <geometry>
-        <mesh
-          filename="package://ari_left_arm/meshes/arm_left_base_link.STL" scale="1 1 ${reflect}"/>
-      </geometry>
-    </collision>
+      <inertial>
+        <origin xyz="0.00705797129984277 -0.0045072380254732 0.000352877816427871" rpy="0 0 0" />
+        <mass value="0.481395506498302" />
+        <inertia
+          ixx="0.00022416049267238" ixy="-4.61763481387137E-07" ixz="3.15922577645587E-08"
+          iyy="0.000454778831736013" iyz="-1.22837579712493E-05"
+          izz="0.000315397102146471" />
+      </inertial>
+      <visual>
+        <origin xyz="0 0 0" rpy="0 0 0" />
+        <geometry>
+          <mesh filename="package://ari_left_arm/meshes/arm_left_base_link.STL" />
+        </geometry>
+        <material name="">
+          <color rgba="0.250980392156863 0.250980392156863 0.250980392156863 1" />
+        </material>
+      </visual>
+      <collision>
+        <origin xyz="0 0 0" rpy="0 0 0" />
+        <geometry>
+          <mesh filename="package://ari_left_arm/meshes/arm_left_base_link.STL" />
+        </geometry>
+      </collision>
     </link>
     <joint name="${name}_${side}_base_joint" type="fixed">
@@ -76,22 +62,19 @@
     <!--************************-->
     <link name="${name}_${side}_1_link">
-<inertial>
-      <origin
-        xyz="-0.00734678702660377 ${-2.69505911157866E-06 * reflect} 0.0810729999795757"
-        rpy="0 0 0" />
-      <mass
-        value="0.626384555512818" />
-      <inertia
-        ixx="0.000821053471340784"
-        ixy="${1.33625825269483E-09 * reflect}"
-        ixz="5.75448054528536E-05"
-        iyy="0.000645070570600376"
-        iyz="${1.29840357496973E-08 * reflect}"
-        izz="0.00042489826130461" />
-    </inertial>
-      <visual>
-        <origin xyz="0 0 0" rpy="0 0 0" />
-        <geometry>
-          <mesh filename="package://ari_left_arm/meshes/arm_left_1_link.STL" scale="1 ${reflect} 1"/>
+      <inertial>
+        <origin xyz="-0.00734678702660377 -2.69505911157866E-06 0.0810729999795757" rpy="0 0 0" />
+        <mass value="0.626384555512818" />
+        <inertia
+          ixx="0.000821053471340784"
+          ixy="1.33625825269483E-09"
+          ixz="5.75448054528536E-05"
+          iyy="0.000645070570600376"
+          iyz="1.29840357496973E-08"
+          izz="0.00042489826130461" />
+      </inertial>
+      <visual>
+        <origin xyz="0 0 0" rpy="0 0 0" />
+        <geometry>
+          <mesh filename="package://ari_left_arm/meshes/arm_left_1_link.STL" />
         </geometry>
         <material name="White"/>
@@ -100,5 +83,5 @@
         <origin xyz="0 0 0" rpy="0 0 0" />
         <geometry>
-          <mesh filename="package://ari_left_arm/meshes/arm_left_1_link.STL" scale="1 ${reflect} 1"/>
+          <mesh filename="package://ari_left_arm/meshes/arm_left_1_link.STL" />
         </geometry>
       </collision>
@@ -107,8 +90,6 @@
       <parent link="${name}_${side}_base_link" />
       <child link="${name}_${side}_1_link" />
-    <origin
-      xyz="0 0.0047319 -0.00041399"
-      rpy="${(-95.002132011 + 0) * deg_to_rad * reflect} 0 0" />
-       <axis xyz="0 0 ${-1*reflect}" />
+      <origin xyz="0 0.0047319 -0.00041399" rpy="-1.6581 0 0" />
+      <axis xyz="0 0 ${1*reflect}" />
       <limit lower="-2.09" upper="2.09" effort="0" velocity="0" />
       <dynamics friction="${arm_friction}" damping="${arm_damping}"/>
@@ -119,22 +100,15 @@
     </joint>
    <link name="${name}_${side}_2_link">
-    <inertial>
-      <origin
-        xyz="-0.0161127523661181 0.0616543232748495 0.00107974895632202"
-        rpy="0 0 0" />
-      <mass
-        value="0.596237000710046" />
-      <inertia
-        ixx="0.000605516102063168"
-        ixy="${-6.92656946627981E-05 * reflect}"
-        ixz="-3.00910746627475E-05"
-        iyy="0.00052936125812993"
-        iyz="${8.82594522397616E-05* reflect}"
-        izz="0.00076716727169814" />
-    </inertial>
-      <visual>
-        <origin xyz="0 0 0" rpy="0 0 0" />
-        <geometry>
-          <mesh filename="package://ari_left_arm/meshes/arm_left_2_link.STL" scale="1 ${reflect} 1"/>
+      <inertial>
+        <origin xyz="-0.0161127523661181 0.0616543232748495 0.00107974895632202" rpy="0 0 0" />
+        <mass value="0.596237000710046" />
+        <inertia ixx="0.000605516102063168" ixy="6.92656946627981E-05" ixz="-3.00910746627475E-05"
+                 iyy="0.00052936125812993" iyz="8.82594522397616E-05"
+                 izz="0.00076716727169814" />
+      </inertial>
+      <visual>
+        <origin xyz="0 0 0" rpy="0 0 0" />
+        <geometry>
+          <mesh filename="package://ari_left_arm/meshes/arm_left_2_link.STL" />
         </geometry>
         <material name="White" />
@@ -143,5 +117,5 @@
         <origin xyz="0 0 0" rpy="0 0 0" />
         <geometry>
-          <mesh filename="package://ari_left_arm/meshes/arm_left_2_link.STL" scale="1 ${reflect} 1"/>
+          <mesh filename="package://ari_left_arm/meshes/arm_left_2_link.STL" />
         </geometry>
       </collision>
@@ -150,8 +124,7 @@
       <parent link="${name}_${side}_1_link" />
       <child link="${name}_${side}_2_link" />
-    <origin
-      xyz="0.008 0 0.1022"
-      rpy="0 ${1.5708 * reflect} 0" />
-      <axis xyz="0 0 ${-1*reflect}" />
+      <origin xyz="0.008 0 0.1022"
+              rpy="0 1.5708 0" />
+      <axis xyz="0 0 ${1*reflect}" />
       <limit lower="0" upper="1.74" effort="${arm_2_max_effort}" velocity="${arm_2_max_vel}" />
       <dynamics friction="${arm_friction}" damping="${arm_damping}"/>
@@ -163,16 +136,9 @@
     <link name="${name}_${side}_3_link">
       <inertial>
-      <origin
-        xyz="0.00261891635576198 ${0.00556893374970152 * reflect} -0.0736249834385048"
-        rpy="0 0 0" />
-      <mass
-        value="0.466609845797877" />
-      <inertia
-        ixx="0.000392473879065454"
-        ixy="${-2.37021311492145E-06 * reflect}"
-        ixz="-2.32964689257321E-06"
-        iyy="0.000496851819658831"
-        iyz="${3.53479285950679E-05 * reflect}"
-        izz="0.000300396202339632" />
+        <origin xyz="0.00261891635576198 0.00556893374970152 -0.0736249834385048" rpy="0 0 0" />
+        <mass value="0.466609845797877" />
+        <inertia ixx="0.000392473879065454" ixy="-2.37021311492145E-06" ixz="-2.32964689257321E-06"
+                 iyy="0.000496851819658831" iyz="3.53479285950679E-05"
+                 izz="0.000300396202339632" />
       </inertial>
       <visual>
@@ -193,7 +159,6 @@
       <parent link="${name}_${side}_2_link" />
       <child link="${name}_${side}_3_link" />
-    <origin
-      xyz="-0.023833 ${0.1003 * reflect} -0.008"
-      rpy="${1.4835 * reflect} 1.5708 0" />
+      <origin xyz="-0.023833 0.1003 -0.008"
+              rpy="1.4835 1.5708 0" />
       <axis xyz="0 0 ${1*reflect}" />
       <limit lower="-2.09" upper="2.09" effort="${arm_3_max_effort}" velocity="${arm_3_max_vel}" />
@@ -209,16 +174,13 @@
     <link name="${name}_${side}_4_link">
       <inertial>
-      <origin
-        xyz="-0.0608591897788406 -0.00187833296903389 0.00810641294898702"
-        rpy="0 0 0" />
-      <mass
-        value="0.46859967403181" />
-      <inertia
-        ixx="0.000324797037287554"
-        ixy="4.43054498245902E-06"
-        ixz="-8.74108555513621E-05"
-        iyy="0.000476423112694781"
-        iyz="3.90099985090552E-06"
-        izz="0.000496361891301139" />
+        <origin xyz="-0.0608591897788406 -0.00187833296903389 0.00810641294898702" rpy="0 0 0" />
+        <mass value="0.46859967403181" />
+        <inertia
+          ixx="0.000324797037287554"
+          ixy="4.43054498245902E-06"
+          ixz="-8.74108555513621E-05"
+          iyy="0.000476423112694781"
+          iyz="3.90099985090552E-06"
+          izz="0.000496361891301139" />
       </inertial>
       <visual>
@@ -270,7 +232,6 @@
       <parent link="${name}_${side}_3_link" />
       <child link="${name}_${side}_4_link" />
-    <origin
-      xyz="0 ${0.00049107 * reflect} -0.1001"
-      rpy="${1.5708 * reflect} ${-1.5708 * reflect} 0" />
+      <origin xyz="0 0.00049107 -0.1001"
+              rpy="1.5708 -1.5708 0" />
       <axis xyz="0 0 ${1*reflect}" />
       <xacro:property name="arm_4_upper_limit"       value="135.0"/>
@@ -283,43 +244,52 @@
                          soft_upper_limit="${0.0 * deg_to_rad - arm_eps}" />
     </joint>
-    <link name="${name}_${side}_5_link">
-      <inertial>
+      <link name="${name}_${side}_5_link">
+        <inertial>
+          <origin xyz="-0.00291138214248795 0.00734841390123893 -0.143226648424061"  rpy="0 0 0" />
+          <mass value="0.350866984764556" />
+          <inertia ixx="0.00107915836241808" ixy="9.10002640587304E-06" ixz="-6.79108896259101E-05"
+                   iyy="0.00113810193294057" iyz="2.83986806757018E-06"
+                   izz="0.000200374211782208" />
+      </inertial>
+      <visual>
+        <origin
+          xyz="0 0 0"
+          rpy="0 0 0" />
+        <geometry>
+          <mesh
+            filename="package://ari_left_arm/meshes/arm_left_5_link.STL"/>
+        </geometry>
+        <material
+          name="White" />
+      </visual>
+      <collision>
+        <origin
+          xyz="0 0 0"
+          rpy="0 0 0" />
+        <geometry>
+          <mesh
+            filename="package://ari_left_arm/meshes/arm_left_5_link.STL"/>
+        </geometry>
+      </collision>
+    </link>
+    <joint
+      name="${name}_${side}_5_joint"
+      type="revolute">
       <origin
-        xyz="-0.00291138214248795 0.00734841390123893 -0.143226648424061"
-        rpy="0 0 0" />
-      <mass
-        value="0.350866984764556" />
-      <inertia
-        ixx="0.00107915836241808"
-        ixy="9.10002640587304E-06"
-        ixz="-6.79108896259101E-05"
-        iyy="0.00113810193294057"
-        iyz="2.83986806757018E-06"
-        izz="0.000200374211782208" />
-      </inertial>
-      <visual>
-          <origin xyz="0 0 0" rpy="0 0 0" />
-        <geometry>
-          <mesh filename="package://ari_left_arm/meshes/arm_left_5_link.STL" scale="1 ${reflect} 1"/>
-        </geometry>
-        <material name="White" />
-      </visual>
-      <collision>
-        <origin xyz="0 0 0" rpy="0 0 0" />
-        <geometry>
-            <mesh filename="package://ari_left_arm/meshes/arm_left_4_link.STL" scale="1 ${reflect} 1"/>
-        </geometry>
-      </collision>
-    </link>
-    <joint name="${name}_${side}_5_joint" type="revolute">
-      <parent link="${name}_${side}_4_link" />
-      <child link="${name}_${side}_5_link" />
-    <origin
-      xyz="-0.106 ${0 * reflect} 0.0010076"
-      rpy="-1.5708 0 -1.5708" />
-      <axis xyz="0 0 ${1*reflect}" />
+        xyz="-0.106 0 0.0010076"
+        rpy="-1.5708 0 -1.5708" />
+      <parent
+        link="${name}_${side}_4_link" />
+      <child
+        link="${name}_${side}_5_link" />
+      <axis
+        xyz="0 0 1" />
       <xacro:property name="arm_5_upper_limit"       value="135.0"/>
       <xacro:property name="arm_5_lower_limit"       value="-5.0"/>
-      <limit lower="-2.09" upper="2.09" effort="${arm_4_max_effort}" velocity="${arm_4_max_vel}" />
+      <limit
+        lower="-2.09"
+        upper="2.09"
+        effort="${arm_4_max_effort}"
+        velocity="${arm_4_max_vel}" />
       <dynamics friction="${arm_friction}" damping="${arm_damping}"/>
       <safety_controller k_position="20"

Commit message: Left arm_v2 correct

File: ari_description/robots/ari.urdf.xacro (robot description, xacro)
@@ -92,8 +92,8 @@
   <xacro:if value="${version == 'v1'}">
   <xacro:ari_arm_v2 name="arm_2" parent="base_link" side="left" reflect="1" end_effector="${end_effector_left == 'ari-hand'}">
-    <origin xyz="-0.22 0.08146 1.153" rpy="${105 * deg_to_rad} ${0 * deg_to_rad} ${180 * deg_to_rad}" />
+    <origin xyz="-0.22 0.08146 1.153" rpy="${-15* deg_to_rad} ${0 * deg_to_rad} ${0 * deg_to_rad}" />
   </xacro:ari_arm_v2>
   <xacro:ari_arm_v2 name="arm_2" parent="base_link" side="right" reflect="-1" end_effector="${end_effector_right == 'ari-hand'}">
-    <origin xyz="-0.22 -0.08146 1.153" rpy="${105 * deg_to_rad} ${0 * deg_to_rad} ${-180 * deg_to_rad}" />
+    <origin xyz="-0.22 -0.08146 1.153" rpy="${105 * deg_to_rad} ${0 * deg_to_rad} ${0 * deg_to_rad}" />
   </xacro:ari_arm_v2>
   </xacro:if>
