Commit message: Mirror arms succeeded

File: ari_description/robots/ari.urdf.xacro (robot description, xacro)
@@ -73,4 +73,5 @@
       <xacro:include filename="$(find ari_description)/urdf/arm/arm_v2.urdf.xacro" />   <!-- Arms -->
       <xacro:include filename="$(find ari_description)/urdf/head/head_v2.urdf.xacro" /> <!-- head -->
+      <xacro:include filename="$(find ari_description)/urdf/arm/arm.urdf.xacro" />   <!-- Arms -->
   </xacro:if>
   <!-- Generic simulator_gazebo plugins -->
@@ -84,16 +85,16 @@
   <xacro:if value="${version == 'v1'}">
   <xacro:ari_arm name="arm" parent="base_link" side="left" reflect="1" end_effector="${end_effector_left == 'ari-hand'}">
-    <origin xyz="-0.219 0.097624 1.1111" rpy="${105.0 * deg_to_rad} ${0.0 * deg_to_rad} ${-180.0 * deg_to_rad}" />
+    <origin xyz="-0.219 0.097624 1.1111" rpy="${105.0 * deg_to_rad} ${0.0 * deg_to_rad} ${180* deg_to_rad}" />
   </xacro:ari_arm>
   <xacro:ari_arm name="arm" parent="base_link" side="right" reflect="-1" end_effector="${end_effector_right == 'ari-hand'}">
-    <origin xyz="-0.219 -0.097624 1.1111" rpy="${-105.0 * deg_to_rad} ${0.0 * deg_to_rad} ${180.0 * deg_to_rad}" />
+    <origin xyz="-0.219 -0.097624 1.1111" rpy="${-105.0 * deg_to_rad} ${0.0 * deg_to_rad} ${-180* deg_to_rad}" />
   </xacro:ari_arm>
   </xacro:if>
-  <xacro:if value="${version == 'v1'}">
+  <xacro:if value="${version == 'v2'}">
   <xacro:ari_arm_v2 name="arm_2" parent="base_link" side="left" reflect="1" end_effector="${end_effector_left == 'ari-hand'}">
-    <origin xyz="-0.22 0.08146 1.153" rpy="${-15* deg_to_rad} ${0 * deg_to_rad} ${0 * deg_to_rad}" />
+    <origin xyz="-0.22 0.08146 1.153" rpy="${0* deg_to_rad} ${0 * deg_to_rad} ${0 * deg_to_rad}" />
   </xacro:ari_arm_v2>
   <xacro:ari_arm_v2 name="arm_2" parent="base_link" side="right" reflect="-1" end_effector="${end_effector_right == 'ari-hand'}">
-    <origin xyz="-0.22 -0.08146 1.153" rpy="${105 * deg_to_rad} ${0 * deg_to_rad} ${0 * deg_to_rad}" />
+    <origin xyz="-0.22 -0.08146 1.153" rpy="${180* deg_to_rad} ${0* deg_to_rad} ${0 * deg_to_rad}" />
   </xacro:ari_arm_v2>
   </xacro:if>

File: ari_description/urdf/arm/arm_v2.urdf.xacro (robot description, xacro)
@@ -40,5 +40,5 @@
         <origin xyz="0 0 0" rpy="0 0 0" />
         <geometry>
-          <mesh filename="package://ari_left_arm/meshes/arm_left_base_link.STL" />
+          <mesh filename="package://ari_left_arm/meshes/arm_left_base_link.STL" scale="1 1 ${reflect}"/>
         </geometry>
         <material name="">
@@ -49,5 +49,5 @@
         <origin xyz="0 0 0" rpy="0 0 0" />
         <geometry>
-          <mesh filename="package://ari_left_arm/meshes/arm_left_base_link.STL" />
+          <mesh filename="package://ari_left_arm/meshes/arm_left_base_link.STL" scale="1 1 ${reflect}"/>
         </geometry>
       </collision>
@@ -63,12 +63,12 @@
     <link name="${name}_${side}_1_link">
       <inertial>
-        <origin xyz="-0.00734678702660377 -2.69505911157866E-06 0.0810729999795757" rpy="0 0 0" />
+        <origin xyz="-0.00734678702660377 ${-2.69505911157866E-06 * reflect} 0.0810729999795757" rpy="0.0 0.0 0.0"/>
         <mass value="0.626384555512818" />
         <inertia
           ixx="0.000821053471340784"
-          ixy="1.33625825269483E-09"
+          ixy="${1.33625825269483E-09 * reflect}"
           ixz="5.75448054528536E-05"
           iyy="0.000645070570600376"
-          iyz="1.29840357496973E-08"
+          iyz="${1.29840357496973E-08 * reflect}"
           izz="0.00042489826130461" />
       </inertial>
@@ -76,5 +76,5 @@
         <origin xyz="0 0 0" rpy="0 0 0" />
         <geometry>
-          <mesh filename="package://ari_left_arm/meshes/arm_left_1_link.STL" />
+          <mesh filename="package://ari_left_arm/meshes/arm_left_1_link.STL" scale="1 ${reflect} 1"/>
         </geometry>
         <material name="White"/>
@@ -83,5 +83,5 @@
         <origin xyz="0 0 0" rpy="0 0 0" />
         <geometry>
-          <mesh filename="package://ari_left_arm/meshes/arm_left_1_link.STL" />
+          <mesh filename="package://ari_left_arm/meshes/arm_left_1_link.STL" scale="1 ${reflect} 1"/>
         </geometry>
       </collision>
@@ -90,6 +90,6 @@
       <parent link="${name}_${side}_base_link" />
       <child link="${name}_${side}_1_link" />
-      <origin xyz="0 0.0047319 -0.00041399" rpy="-1.6581 0 0" />
-      <axis xyz="0 0 ${1*reflect}" />
+      <origin xyz="0.0 0.0047319 -0.00041399" rpy="${(-90 - 5.002132011 * reflect) * deg_to_rad} 0.0 0.0"/>
+      <axis xyz="0 0 ${-reflect}" />
       <limit lower="-2.09" upper="2.09" effort="0" velocity="0" />
       <dynamics friction="${arm_friction}" damping="${arm_damping}"/>
@@ -110,5 +110,5 @@
         <origin xyz="0 0 0" rpy="0 0 0" />
         <geometry>
-          <mesh filename="package://ari_left_arm/meshes/arm_left_2_link.STL" />
+          <mesh filename="package://ari_left_arm/meshes/arm_left_2_link.STL" scale="1 ${reflect} 1" />
         </geometry>
         <material name="White" />
@@ -117,5 +117,5 @@
         <origin xyz="0 0 0" rpy="0 0 0" />
         <geometry>
-          <mesh filename="package://ari_left_arm/meshes/arm_left_2_link.STL" />
+          <mesh filename="package://ari_left_arm/meshes/arm_left_2_link.STL" scale="1 ${reflect} 1"/>
         </geometry>
       </collision>
@@ -125,6 +125,6 @@
       <child link="${name}_${side}_2_link" />
       <origin xyz="0.008 0 0.1022"
-              rpy="0 1.5708 0" />
-      <axis xyz="0 0 ${1*reflect}" />
+              rpy="0 ${1.5708} 0" />
+      <axis xyz="0 0 ${reflect}" />
       <limit lower="0" upper="1.74" effort="${arm_2_max_effort}" velocity="${arm_2_max_vel}" />
       <dynamics friction="${arm_friction}" damping="${arm_damping}"/>
@@ -145,5 +145,5 @@
         <origin xyz="0 0 0" rpy="0 0 0" />
         <geometry>
-          <mesh filename="package://ari_left_arm/meshes/arm_left_3_link.STL" scale="1 ${reflect} 1"/>
+          <mesh filename="package://ari_left_arm/meshes/arm_left_3_link.STL" scale="1 1 ${reflect}"/>
         </geometry>
         <material name="White" />
@@ -152,5 +152,5 @@
         <origin xyz="0 0 0" rpy="0 0 0" />
         <geometry>
-          <mesh filename="package://ari_left_arm/meshes/arm_left_3_link.STL" scale="1 ${reflect} 1"/>
+          <mesh filename="package://ari_left_arm/meshes/arm_left_3_link.STL" scale="1 1 ${reflect}"/>
         </geometry>
       </collision>
@@ -159,6 +159,6 @@
       <parent link="${name}_${side}_2_link" />
       <child link="${name}_${side}_3_link" />
-      <origin xyz="-0.023833 0.1003 -0.008"
-              rpy="1.4835 1.5708 0" />
+      <origin xyz="-0.023833 ${0.1003 * reflect} -0.008"
+              rpy="${(90 - 5.00192155 * reflect) * deg_to_rad} ${90 * deg_to_rad} 0" />
       <axis xyz="0 0 ${1*reflect}" />
       <limit lower="-2.09" upper="2.09" effort="${arm_3_max_effort}" velocity="${arm_3_max_vel}" />
@@ -198,8 +198,8 @@
         <geometry>
           <xacro:if value="${end_effector}">
-            <mesh filename="package://ari_left_arm/meshes/arm_left_4_link.STL" scale="1 ${reflect} 1"/>
+            <mesh filename="package://ari_left_arm/meshes/arm_left_4_link.STL" scale="${reflect} 1 1"/>
           </xacro:if>
           <xacro:unless value="${end_effector}">
-            <mesh filename="package://ari_left_arm/meshes/arm_left_4_link.STL" scale="1 1 1"/>
+            <mesh filename="package://ari_left_arm/meshes/arm_left_4_link.STL" scale="${reflect} 1 1"/>
           </xacro:unless>
         </geometry>
@@ -224,5 +224,5 @@
           </xacro:if>
           <xacro:unless value="${end_effector}">
-            <mesh filename="package://ari_left_arm/meshes/arm_left_4_link.STL" scale="1 1 1"/>
+            <mesh filename="package://ari_left_arm/meshes/arm_left_4_link.STL" scale="1 ${reflect} 1"/>
           </xacro:unless>
         </geometry>
@@ -232,6 +232,6 @@
       <parent link="${name}_${side}_3_link" />
       <child link="${name}_${side}_4_link" />
-      <origin xyz="0 0.00049107 -0.1001"
-              rpy="1.5708 -1.5708 0" />
+      <origin xyz="0 0.00049107 ${-0.1001 * reflect}"
+              rpy="${90 * deg_to_rad} ${-90 * deg_to_rad} 0" />
       <axis xyz="0 0 ${1*reflect}" />
       <xacro:property name="arm_4_upper_limit"       value="135.0"/>
@@ -244,5 +244,5 @@
                          soft_upper_limit="${0.0 * deg_to_rad - arm_eps}" />
     </joint>
-      <link name="${name}_${side}_5_link">
+    <link name="${name}_${side}_5_link">
         <inertial>
           <origin xyz="-0.00291138214248795 0.00734841390123893 -0.143226648424061"  rpy="0 0 0" />
@@ -251,5 +251,5 @@
                    iyy="0.00113810193294057" iyz="2.83986806757018E-06"
                    izz="0.000200374211782208" />
-      </inertial>
+        </inertial>
       <visual>
         <origin
@@ -258,5 +258,5 @@
         <geometry>
           <mesh
-            filename="package://ari_left_arm/meshes/arm_left_5_link.STL"/>
+            filename="package://ari_left_arm/meshes/arm_left_5_link.STL" scale="1 1 ${reflect}"/>
         </geometry>
         <material
@@ -269,5 +269,5 @@
         <geometry>
           <mesh
-            filename="package://ari_left_arm/meshes/arm_left_5_link.STL"/>
+            filename="package://ari_left_arm/meshes/arm_left_5_link.STL" scale="1 1 ${reflect}"/>
         </geometry>
       </collision>
@@ -277,5 +277,5 @@
       type="revolute">
       <origin
-        xyz="-0.106 0 0.0010076"
+        xyz="${-0.106 * reflect} 0 0.0010076"
         rpy="-1.5708 0 -1.5708" />
       <parent
