Commit message: update stl and urdf for sensor and wheels

File: ari_description/robots/ari.urdf.xacro (robot description, xacro)
@@ -66,5 +66,4 @@
       <xacro:include filename="$(find ari_description)/urdf/arm/arm.urdf.xacro" />   <!-- Arms -->
       <xacro:include filename="$(find ari_description)/urdf/head/head.urdf.xacro" /> <!-- head -->
-      <xacro:include filename="$(find ari_description)/urdf/arm/arm_v2.urdf.xacro" />   <!-- Arms -->
   </xacro:if>
   <xacro:if value="${version == 'v2'}">
@@ -73,5 +72,4 @@
       <xacro:include filename="$(find ari_description)/urdf/arm/arm_v2.urdf.xacro" />   <!-- Arms -->
       <xacro:include filename="$(find ari_description)/urdf/head/head_v2.urdf.xacro" /> <!-- head -->
-      <xacro:include filename="$(find ari_description)/urdf/arm/arm.urdf.xacro" />   <!-- Arms -->
   </xacro:if>
   <!-- Generic simulator_gazebo plugins -->
@@ -92,10 +90,10 @@
   </xacro:if>
   <xacro:if value="${version == 'v2'}">
-  <xacro:ari_arm_v2 name="arm_2" parent="base_link" side="left" reflect="1" end_effector="${end_effector_left == 'ari-hand'}">
+  <xacro:ari_arm name="arm" parent="base_link" side="left" reflect="1" end_effector="${end_effector_left == 'ari-hand'}">
     <origin xyz="-0.22 0.08146 1.153" rpy="${0* deg_to_rad} ${0 * deg_to_rad} ${0 * deg_to_rad}" />
-  </xacro:ari_arm_v2>
-  <xacro:ari_arm_v2 name="arm_2" parent="base_link" side="right" reflect="-1" end_effector="${end_effector_right == 'ari-hand'}">
-    <origin xyz="-0.22 -0.08146 1.153" rpy="${180* deg_to_rad} ${0* deg_to_rad} ${0 * deg_to_rad}" />
-  </xacro:ari_arm_v2>
+  </xacro:ari_arm>
+  <xacro:ari_arm name="arm" parent="base_link" side="right" reflect="-1" end_effector="${end_effector_right == 'ari-hand'}">
+    <origin xyz="-0.22 -0.08146 1.153" rpy="${0 * deg_to_rad} ${0* deg_to_rad} ${180 * deg_to_rad}" />
+  </xacro:ari_arm>
   </xacro:if>
 </robot>

File: ari_description/urdf/arm/arm_v2.urdf.xacro (robot description, xacro)
@@ -24,5 +24,5 @@
   <xacro:property name="arm_4_max_effort"   value="5" />
   <xacro:property name="arm_eps"            value="0.07" />
-  <xacro:macro name="ari_arm_v2" params="name parent side reflect end_effector *origin">
+  <xacro:macro name="ari_arm" params="name parent side reflect end_effector *origin">
     <!--************************-->
     <!--      ARM_BASE_LINK     -->
@@ -40,5 +40,5 @@
         <origin xyz="0 0 0" rpy="0 0 0" />
         <geometry>
-          <mesh filename="package://ari_left_arm/meshes/arm_left_base_link.STL" scale="1 1 ${reflect}"/>
+          <mesh filename="package://ari_description/meshes/arm/arm_base_v2.stl" scale="${reflect} 1 1"/>
         </geometry>
         <material name="">
@@ -49,5 +49,5 @@
         <origin xyz="0 0 0" rpy="0 0 0" />
         <geometry>
-          <mesh filename="package://ari_left_arm/meshes/arm_left_base_link.STL" scale="1 1 ${reflect}"/>
+          <mesh filename="package://ari_description/meshes/arm/arm_base_v2.stl" scale="${reflect} 1 1"/>
         </geometry>
       </collision>
@@ -76,5 +76,5 @@
         <origin xyz="0 0 0" rpy="0 0 0" />
         <geometry>
-          <mesh filename="package://ari_left_arm/meshes/arm_left_1_link.STL" scale="1 ${reflect} 1"/>
+          <mesh filename="package://ari_description/meshes/arm/arm_1_v2.stl" scale=" ${reflect} 1 1"/>
         </geometry>
         <material name="White"/>
@@ -83,5 +83,5 @@
         <origin xyz="0 0 0" rpy="0 0 0" />
         <geometry>
-          <mesh filename="package://ari_left_arm/meshes/arm_left_1_link.STL" scale="1 ${reflect} 1"/>
+          <mesh filename="package://ari_description/meshes/arm/arm_1_v2.stl" scale="${reflect} 1 1"/>
         </geometry>
       </collision>
@@ -90,7 +90,7 @@
       <parent link="${name}_${side}_base_link" />
       <child link="${name}_${side}_1_link" />
-      <origin xyz="0.0 0.0047319 -0.00041399" rpy="${(-90 - 5.002132011 * reflect) * deg_to_rad} 0.0 0.0"/>
-      <axis xyz="0 0 ${-reflect}" />
-      <limit lower="-2.09" upper="2.09" effort="0" velocity="0" />
+      <origin xyz="0.0 0.0047319 -0.00041399" rpy="${(-90 - 5.0) * deg_to_rad} 0.0 0.0"/>
+      <axis xyz="0 0 ${-1 * reflect}" />
+      <limit lower="${-120.0 * deg_to_rad}" upper="${120.0 * deg_to_rad}" effort="0" velocity="0" />
       <dynamics friction="${arm_friction}" damping="${arm_damping}"/>
       <safety_controller k_position="20"
@@ -110,5 +110,5 @@
         <origin xyz="0 0 0" rpy="0 0 0" />
         <geometry>
-          <mesh filename="package://ari_left_arm/meshes/arm_left_2_link.STL" scale="1 ${reflect} 1" />
+          <mesh filename="package://ari_description/meshes/arm/arm_2_v2.stl" scale="1 1 ${reflect}" />
         </geometry>
         <material name="White" />
@@ -117,5 +117,5 @@
         <origin xyz="0 0 0" rpy="0 0 0" />
         <geometry>
-          <mesh filename="package://ari_left_arm/meshes/arm_left_2_link.STL" scale="1 ${reflect} 1"/>
+          <mesh filename="package://ari_description/meshes/arm/arm_2_v2.stl" scale="1 1 ${reflect}"/>
         </geometry>
       </collision>
@@ -124,13 +124,13 @@
       <parent link="${name}_${side}_1_link" />
       <child link="${name}_${side}_2_link" />
-      <origin xyz="0.008 0 0.1022"
-              rpy="0 ${1.5708} 0" />
-      <axis xyz="0 0 ${reflect}" />
-      <limit lower="0" upper="1.74" effort="${arm_2_max_effort}" velocity="${arm_2_max_vel}" />
-      <dynamics friction="${arm_friction}" damping="${arm_damping}"/>
-      <safety_controller k_position="20"
-                         k_velocity="20"
-                         soft_lower_limit="${0.0 * deg_to_rad  + arm_eps}"
-                         soft_upper_limit="${99.0 * deg_to_rad - arm_eps}" />
+      <origin xyz="${0.008 * reflect} 0 0.1022"
+              rpy="0 ${1.5708 * 1} 0" />
+      <axis xyz="0 0 1" />
+      <limit lower="${-24 * deg_to_rad}" upper="${70 * deg_to_rad}" effort="${arm_2_max_effort}" velocity="${arm_2_max_vel}" />
+      <dynamics friction="${arm_friction}" damping="${arm_damping}"/>
+      <safety_controller k_position="20"
+                         k_velocity="20"
+                         soft_lower_limit="${-24 * deg_to_rad  + arm_eps}"
+                         soft_upper_limit="${70 * deg_to_rad - arm_eps}" />
     </joint>
     <link name="${name}_${side}_3_link">
@@ -145,5 +145,5 @@
         <origin xyz="0 0 0" rpy="0 0 0" />
         <geometry>
-          <mesh filename="package://ari_left_arm/meshes/arm_left_3_link.STL" scale="1 1 ${reflect}"/>
+          <mesh filename="package://ari_description/meshes/arm/arm_3_v2.stl" scale="${reflect} 1 1"/>
         </geometry>
         <material name="White" />
@@ -152,5 +152,5 @@
         <origin xyz="0 0 0" rpy="0 0 0" />
         <geometry>
-          <mesh filename="package://ari_left_arm/meshes/arm_left_3_link.STL" scale="1 1 ${reflect}"/>
+          <mesh filename="package://ari_description/meshes/arm/arm_3_v2.stl" scale="${reflect} 1 1"/>
         </geometry>
       </collision>
@@ -159,13 +159,13 @@
       <parent link="${name}_${side}_2_link" />
       <child link="${name}_${side}_3_link" />
-      <origin xyz="-0.023833 ${0.1003 * reflect} -0.008"
-              rpy="${(90 - 5.00192155 * reflect) * deg_to_rad} ${90 * deg_to_rad} 0" />
-      <axis xyz="0 0 1" />
-      <limit lower="-2.09" upper="2.09" effort="${arm_3_max_effort}" velocity="${arm_3_max_vel}" />
-      <dynamics friction="${arm_friction}" damping="${arm_damping}"/>
-      <safety_controller k_position="20"
-                         k_velocity="20"
-                         soft_lower_limit="${-120.0 * deg_to_rad + arm_eps}"
-                         soft_upper_limit="${120.0 * deg_to_rad - arm_eps}" />
+      <origin xyz="${-0.023833 * 1} ${0.1003 * 1} ${-0.008 * reflect}"
+              rpy="${(90 - 5.0) * deg_to_rad} ${90 * deg_to_rad} 0" />
+      <axis xyz="0 0 ${reflect}" />
+      <limit lower="${-45 * deg_to_rad}" upper="${195.0 * deg_to_rad}" effort="${arm_3_max_effort}" velocity="${arm_3_max_vel}" />
+      <dynamics friction="${arm_friction}" damping="${arm_damping}"/>
+      <safety_controller k_position="20"
+                         k_velocity="20"
+                         soft_lower_limit="${-45 * deg_to_rad + arm_eps}"
+                         soft_upper_limit="${195 * deg_to_rad - arm_eps}" />
     </joint>
     <!--************************-->
@@ -198,8 +198,8 @@
         <geometry>
           <xacro:if value="${end_effector}">
-            <mesh filename="package://ari_left_arm/meshes/arm_left_4_link.STL" scale="${reflect} 1 1"/>
+            <mesh filename="package://ari_description/meshes/arm/arm_4_v2.stl" scale="1 ${reflect} 1"/>
           </xacro:if>
           <xacro:unless value="${end_effector}">
-            <mesh filename="package://ari_left_arm/meshes/arm_left_4_link.STL" scale="${reflect} 1 1"/>
+            <mesh filename="package://ari_description/meshes/arm/arm_4_v2.stl" scale="1 ${reflect} 1"/>
           </xacro:unless>
         </geometry>
@@ -221,8 +221,8 @@
         <geometry>
           <xacro:if value="${end_effector}">
-            <mesh filename="package://ari_left_arm/meshes/arm_left_4_link.STL" scale="${reflect} 1 1"/>
+            <mesh filename="package://ari_description/meshes/arm/arm_4_v2.stl" scale="1 ${reflect} 1"/>
           </xacro:if>
           <xacro:unless value="${end_effector}">
-            <mesh filename="package://ari_left_arm/meshes/arm_left_4_link.STL" scale="${reflect} 1 1"/>
+            <mesh filename="package://ari_description/meshes/arm/arm_4_v2.stl" scale="1 ${reflect} 1"/>
           </xacro:unless>
         </geometry>
@@ -232,15 +232,15 @@
       <parent link="${name}_${side}_3_link" />
       <child link="${name}_${side}_4_link" />
-      <origin xyz="0 0.00049107 ${-0.1001 * reflect}"
+      <origin xyz="0 0.00049107 -0.1001"
               rpy="${90 * deg_to_rad} ${-90 * deg_to_rad} 0" />
-      <axis xyz="0 0 ${1*reflect}" />
+      <axis xyz="0 0 ${-1*reflect}" />
       <xacro:property name="arm_4_upper_limit"       value="135.0"/>
       <xacro:property name="arm_4_lower_limit"       value="-5.0"/>
-      <limit lower="-1.74" upper="0" effort="${arm_4_max_effort}" velocity="${arm_4_max_vel}" />
-      <dynamics friction="${arm_friction}" damping="${arm_damping}"/>
-      <safety_controller k_position="20"
-                         k_velocity="20"
-                         soft_lower_limit="${-99.0 * deg_to_rad + arm_eps}"
-                         soft_upper_limit="${0.0 * deg_to_rad - arm_eps}" />
+      <limit lower="${0 * deg_to_rad}" upper="${100 * deg_to_rad}" effort="${arm_4_max_effort}" velocity="${arm_4_max_vel}" />
+      <dynamics friction="${arm_friction}" damping="${arm_damping}"/>
+      <safety_controller k_position="20"
+                         k_velocity="20"
+                         soft_lower_limit="${0 * deg_to_rad + arm_eps}"
+                         soft_upper_limit="${100 * deg_to_rad - arm_eps}" />
     </joint>
     <link name="${name}_${side}_5_link">
@@ -258,5 +258,5 @@
         <geometry>
           <mesh
-            filename="package://ari_left_arm/meshes/arm_left_5_link.STL" scale="1 1 ${reflect}"/>
+            filename="package://ari_description/meshes/arm/arm_5_v2.stl" scale="${reflect} 1 1"/>
         </geometry>
         <material
@@ -269,5 +269,5 @@
         <geometry>
           <mesh
-            filename="package://ari_left_arm/meshes/arm_left_5_link.STL" scale="1 1 ${reflect}"/>
+            filename="package://ari_description/meshes/arm/arm_5_v2.stl" scale="${reflect} 1 1"/>
         </geometry>
       </collision>
@@ -277,6 +277,6 @@
       type="revolute">
       <origin
-        xyz="${-0.106 * reflect} 0 0.0010076"
-        rpy="-1.5708 0 -1.5708" />
+        xyz="-0.106 0 0.0010076"
+        rpy="${-90 * deg_to_rad} 0 ${-90 * deg_to_rad}" />
       <parent
         link="${name}_${side}_4_link" />
@@ -284,5 +284,5 @@
         link="${name}_${side}_5_link" />
       <axis
-        xyz="0 0 1" />
+        xyz="0 0 ${reflect}" />
       <xacro:property name="arm_5_upper_limit"       value="135.0"/>
       <xacro:property name="arm_5_lower_limit"       value="-5.0"/>

File: ari_description/urdf/base/base_v2.urdf.xacro (robot description, xacro)
@@ -12,8 +12,11 @@
   <xacro:include filename="$(find ari_description)/urdf/wheels/wheel_v2.urdf.xacro"/>
   <xacro:include filename="$(find ari_description)/urdf/wheels/caster_v2.urdf.xacro"/>
+  <xacro:include filename="$(find ari_description)/urdf/base/docking_link_v2.urdf.xacro"/>
+  <xacro:include filename="$(find ari_description)/urdf/sensors/torso_v2_rgbd.urdf.xacro"/>
+  <xacro:include filename="$(find ari_description)/urdf/sensors/torso_v2_265.urdf.xacro"/>
   <!-- Wheel characteristics -->
   <xacro:property name="wheel_radius"     value="0.125"/>
   <xacro:property name="wheel_width"      value="0.075"/>
-  <xacro:property name="wheel_separation" value="0.44"/>
+  <xacro:property name="wheel_separation" value="0.4668"/>
   <xacro:property name="wheel_torque"     value="6.0"/>
   <xacro:property name="wheel_velocity"   value="1.0"/>
@@ -22,6 +25,6 @@
   <xacro:property name="caster_width"        value="0.055"/>
   <xacro:property name="caster_separation_x" value="0.91"/>
-  <xacro:property name="caster_offset_y"     value="0.1025"/>
-  <xacro:property name="caster_offset_z"     value="-0.08"/>
+  <xacro:property name="caster_offset_y"     value="0.0875"/>
+  <xacro:property name="caster_offset_z"     value="-0.0305"/>
   <xacro:macro name="base" params="name">
   <!-- Base -->
@@ -45,5 +48,5 @@
       <geometry>
         <mesh
-          filename="package://ari_base/meshes/base_link.STL" />
+          filename="package://ari_description/meshes/base/base_v2.stl" />
       </geometry>
       <material name="Grey" />
@@ -53,5 +56,5 @@
       <geometry>
         <mesh
-          filename="package://ari_base/meshes/base_link.STL" />
+          filename="package://ari_description/meshes/base/base_v2.stl" />
       </geometry>
       <material name="Grey" />
@@ -115,16 +118,13 @@
     </inertial>
   </link>
-  <!-- Docking Link -->
-  <joint name="docking_joint" type="fixed">
-      <parent link="base_link"/>
-      <child link="docking_link"/>
-      <origin xyz="-0.602 0 0" rpy="0 0 0" />
-  </joint>
-  <link name="docking_link">
-      <inertial>
-          <origin xyz="0 0 0" rpy="0 0 0"/>
-          <mass value="0.0001" />
-          <inertia ixx="0.0001"  ixy="0"  ixz="0" iyy="0.0001" iyz="0" izz="0.0001" />
-      </inertial>
-  </link>
+  <xacro:docking_link name="docking">
+    <origin xyz="-0.600830 0 0.039" rpy="0 0 0" />
+  </xacro:docking_link>
+<!--   <xacro:torso_rgbd name="torso_rgbd">
+    <origin xyz="-0.13799 -0.00034911 1.0305" rpy="0 0.75049 0" />
+  </xacro:torso_rgbd>
+  <xacro:torso_265 name="torso_265">
+    <origin xyz="-0.31955 0.009 1.0599" rpy="0 0.2618 3.1416" />
+  </xacro:torso_265>
+ -->
 </robot>

File: ari_description/urdf/head/head_v2.urdf.xacro (robot description, xacro)
@@ -37,22 +37,14 @@
     <link name="${name}_link">
     <inertial>
-      <origin
-        xyz="0.0108359726631008 0.000718390176517933 0.0855378659235452"
-        rpy="0 0 0" />
-      <mass
-        value="0.412082934872394" />
-      <inertia
-        ixx="0.000403841240088291"
-        ixy="-2.50683274214796E-07"
-        ixz="-1.29761673527528E-05"
-        iyy="0.000282783550645599"
-        iyz="-1.48768048583041E-09"
-        izz="0.000403570643105203" />
-    </inertial>
+      <origin xyz="0.0108359726631008 0.000718390176517933 0.0855378659235452" rpy="0 0 0"/>
+      <mass value="0.412082934872394" />
+      <inertia ixx="0.000403841240088291" ixy="-2.50683274214796E-07" ixz="-1.29761673527528E-05"
+               iyy="0.000282783550645599" iyz="-1.48768048583041E-09"
+               izz="0.000403570643105203" />
+      </inertial>
       <visual>
         <origin xyz="0 0 0" rpy="0 0 0"/>
         <geometry>
-        <mesh
-          filename="package://ari_head/meshes/head_1_link.STL" />
+          <mesh filename="package://ari_description/meshes/head/head_1_v2.stl" scale="1 1 1"/>
         </geometry>
         <material name="White" />
@@ -61,5 +53,5 @@
         <origin xyz="0.0 0 0" rpy="0 0 0.0" />
         <geometry>
-          <mesh filename="package://ari_head/meshes/head_1_link.STL" scale="1 1 1"/>
+          <mesh filename="package://ari_description/meshes/head/head_1_v2.stl" scale="1 1 1"/>
         </geometry>
         <material name="White" />
@@ -94,22 +86,15 @@
   <xacro:macro name="head_2" params="name parent">
     <link name="${name}_link">
-    <inertial>
-      <origin
-        xyz="0.00794853114293399 0.10682927811673 -0.0216446425740413"
-        rpy="0 0 0" />
-      <mass
-        value="0.943484631730919" />
-      <inertia
-        ixx="0.00356848001507154"
-        ixy="0.000577244872529115"
-        ixz="2.42088792789485E-08"
-        iyy="0.00239180242384949"
-        iyz="-6.2275127757022E-07"
-        izz="0.00306783859370423" />
-    </inertial>
+      <inertial>
+        <origin xyz="0.00794853114293399 0.10682927811673 -0.0216446425740413" rpy="0 0 0"/>
+        <mass value="0.943484631730919"/>
+        <inertia ixx="0.00356848001507154" ixy="0.000577244872529115" ixz="2.42088792789485E-08"
+                 iyy="0.00239180242384949" iyz="-6.2275127757022E-07"
+                 izz="0.00306783859370423" />
+      </inertial>
       <visual>
         <origin xyz="0 0 0" rpy="0 0 0" />
         <geometry>
-          <mesh filename="package://ari_head/meshes/head_2_link.STL" scale="1 1 1"/>
+          <mesh filename="package://ari_description/meshes/head/head_2_v2.stl" scale="1 1 1"/>
         </geometry>
         <material name="White" />
@@ -118,5 +103,5 @@
         <origin xyz="0 0 0" rpy="0 0 0" />
         <geometry>
-          <mesh filename="package://ari_head/meshes/head_2_link.STL" scale="1 1 1"/>
+          <mesh filename="package://ari_description/meshes/head/head_2_v2.stl" scale="1 1 1"/>
         </geometry>
         <material name="White" />
@@ -126,7 +111,5 @@
       <parent link="${parent}"/>
       <child link="${name}_link"/>
-      <origin
-      xyz="0.0425 0.022 0.1011"
-      rpy="1.5708 0 -3.1416" />
+      <origin xyz="0.0425 0.022 0.1011" rpy="1.5708 0 -3.1416" />
       <axis xyz="0 0 -1" />
       <limit lower="-0.261" upper="0.436" effort="3.26" velocity="${head_max_vel}" />

File: ari_description/urdf/torso/torso_sensors_v2.urdf.xacro (robot description, xacro)
@@ -16,13 +16,13 @@
   <xacro:include filename="$(find ari_description)/urdf/sensors/sick_tim571_laser.urdf.xacro"/>
   <!--Constant parameters-->
-  <xacro:property name="torso_front_camera_position_x" value="-0.11249" />
-  <xacro:property name="torso_front_camera_position_y" value="0.0" />
-  <xacro:property name="torso_front_camera_position_z" value="0.97052" />
+  <xacro:property name="torso_front_camera_position_x" value="-0.13799" />
+  <xacro:property name="torso_front_camera_position_y" value="-0.00034911" />
+  <xacro:property name="torso_front_camera_position_z" value="1.0305" />
   <xacro:property name="torso_front_camera_orientation_r" value="0.0" />
-  <xacro:property name="torso_front_camera_orientation_p" value="${42.5 * deg_to_rad}" />
+  <xacro:property name="torso_front_camera_orientation_p" value="${43 * deg_to_rad}" />
   <xacro:property name="torso_front_camera_orientation_y" value="0.0" />
-  <xacro:property name="torso_back_camera_position_x" value="-0.3275" />
+  <xacro:property name="torso_back_camera_position_x" value="-0.31955" />
   <xacro:property name="torso_back_camera_position_y" value="0.009" />
-  <xacro:property name="torso_back_camera_position_z" value="1.0337" />
+  <xacro:property name="torso_back_camera_position_z" value="1.0599" />
   <xacro:property name="torso_back_camera_orientation_r" value="0.0" />
   <xacro:property name="torso_back_camera_orientation_p" value="${15 * deg_to_rad}" />
