Commit message: typo in test

File: ari_description/robots/ari.urdf.xacro (robot description, xacro)
@@ -83,8 +83,8 @@
   <xacro:if value="${version == 'v1'}">
   <xacro:ari_arm name="arm" parent="base_link" side="left" reflect="1" end_effector="${end_effector_left == 'ari-hand'}">
-    <origin xyz="-0.219 0.097624 1.1111" rpy="${105.0 * deg_to_rad} ${0.0 * deg_to_rad} ${180* deg_to_rad}" />
+    <origin xyz="-0.219 0.097624 1.1111" rpy="${105.0 * deg_to_rad} ${0.0 * deg_to_rad} ${-180.0 * deg_to_rad}" />
   </xacro:ari_arm>
   <xacro:ari_arm name="arm" parent="base_link" side="right" reflect="-1" end_effector="${end_effector_right == 'ari-hand'}">
-    <origin xyz="-0.219 -0.097624 1.1111" rpy="${-105.0 * deg_to_rad} ${0.0 * deg_to_rad} ${-180* deg_to_rad}" />
+    <origin xyz="-0.219 -0.097624 1.1111" rpy="${-105.0 * deg_to_rad} ${0.0 * deg_to_rad} ${180.0 * deg_to_rad}" />
   </xacro:ari_arm>
   </xacro:if>

File: ari_description/urdf/wheels/caster_v2.urdf.xacro (robot description, xacro)
@@ -7,20 +7,19 @@
   Creative Commons, 444 Castro Street, Suite 900, Mountain View, California, 94041, USA.
 -->
-    <!--  CHECK PARAMETERS FROM BASE_V2 FILE -->
 <robot xmlns:xacro="http://ros.org/wiki/xacro">
-  <xacro:include filename="$(find ari_description)/urdf/wheels/caster.gazebo.xacro"/>
+  <xacro:include filename="$(find ari_description)/urdf/wheels/caster_v2.gazebo.xacro"/>
   <xacro:macro name="caster" params="side reflect radius width separation_x offset_y offset_z parent">
     <link name="caster_${side}_link">
       <inertial>
-        <origin xyz="${1.4445E-06 * reflect} 0.016213 ${-0.00019766 * reflect}" rpy="0 0 0"/>
-        <mass value="0.24242"/>
-        <inertia  ixx="0.0002099" ixy="${-5.5806E-09 * reflect}" ixz="-6.9375E-11"
-                  iyy="0.00020239" iyz="${-2.6771E-09 * reflect}"
-                  izz="0.00025496"/>
+        <origin xyz="${-0.016512 * reflect} 0.17601 ${-0.029897 * reflect}" rpy="0 0 0"/>
+        <mass value="0.046595"/>
+        <inertia  ixx="7.5074E-06" ixy="${-5.6754E-07 * reflect}" ixz="-2.3436E-07"
+                  iyy="1.6751E-05" iyz="${-1.435E-08 * reflect}"
+                  izz="1.1856E-05"/>
       </inertial>
       <visual>
         <origin xyz="0 0 0" rpy="0 0 0"/>
         <geometry>
-          <mesh filename="package://ari_description/meshes/wheels/caster_${side}.stl"/>
+          <mesh filename="package://ari_description/meshes/wheels/caster_v2.stl" scale="1 ${reflect} 1"/>
         </geometry>
         <material name="Grey"/>
@@ -36,6 +35,6 @@
       <parent link="${parent}_link"/>
       <child link="caster_${side}_link"/>
-      <origin xyz="${-separation_x / 2} ${-offset_y * reflect} ${offset_z}" rpy="${90.0 * deg_to_rad} 0 0"/>
-      <axis xyz="0 0 -1"/>
+      <origin xyz="${-separation_x / 2} ${-offset_y * reflect} ${offset_z}" rpy="${0.0 * deg_to_rad} 0 0"/>
+      <axis xyz="0 0 1"/>
     </joint>
     <!-- Gazebo extensions -->

File: ari_description/urdf/wheels/wheel_v2.urdf.xacro (robot description, xacro)
@@ -7,5 +7,4 @@
 Creative Commons, 444 Castro Street, Suite 900, Mountain View, California, 94041, USA.
 -->
-<!--  CHECK PARAMETERS FROM BASE_V2 FILE -->
 <robot xmlns:xacro="http://ros.org/wiki/xacro">
   <xacro:include filename="$(find ari_description)/urdf/wheels/wheel_v2.transmission.xacro"/>
@@ -14,22 +13,14 @@
     <link name="wheel_${side}_link">
     <inertial>
-      <origin
-        xyz="-6.7466E-06 0.00019427 -1.3878E-17"
-        rpy="0 0 0" />
-      <mass
-        value="2.0456" />
-      <inertia
-        ixx="0.0052532"
-        ixy="-2.566E-08"
-        ixz="${1.1121E-18 * reflect}"
-        iyy="0.009772"
-        iyz="${2.3459E-17 * reflect}"
-        izz="0.0052531" />
+      <origin xyz="-6.7466E-06 0.00019427 -1.3878E-17" rpy="0 0 0"/>
+      <mass value="2.0456" />
+      <inertia ixx="0.0052532" ixy="-2.566E-08" ixz="${1.1121E-18 * reflect}"
+               iyy="0.009772" iyz="${2.3459E-17 * reflect}"
+               izz="0.0052531" />
     </inertial>
       <visual>
         <origin xyz="0 0 0" rpy="0 0 0"/>
         <geometry>
-        <mesh
-          filename="package://ari_base/meshes/wheel_left_link.STL" />
+        <mesh filename="package://ari_description/meshes/wheels/wheel_${side}_v2.stl"/>
         </geometry>
         <material name="White"/>
@@ -47,5 +38,5 @@
       <parent link="${parent}_link"/>
       <child link="wheel_${side}_link"/>
-      <origin xyz="0 ${-separation / 2 * reflect} 0" rpy="${90.0 * deg_to_rad} 0 0"/>
+      <origin xyz="0 ${ -separation / 2 * reflect} 0" rpy="${0 * deg_to_rad} 0 0"/>
       <axis xyz="0 0 -1"/>
       <limit effort="${torque}" velocity="${velocity / radius}"/>

Commit message: replace version with robot_model

File: ari_description/robots/ari.urdf.xacro (robot description, xacro)
@@ -9,5 +9,5 @@
 <robot  xmlns:xacro="http://ros.org/wiki/xacro"
         name="ari" >
-  <xacro:arg name="version" default="v1"/>
+  <xacro:arg name="robot_model" default="v1"/>
   <xacro:arg name="end_effector_right" default="ari-hand"/>
   <xacro:arg name="end_effector_left" default="ari-hand"/>
@@ -16,5 +16,5 @@
   <xacro:arg name="camera_model_head" default="raspi"/>
   <xacro:arg name="has_thermal" default="false"/>
-  <xacro:property name="version" value="$(arg version)" />
+  <xacro:property name="robot_model" value="$(arg robot_model)" />
   <xacro:property name="end_effector_right" value="$(arg end_effector_right)" />
   <xacro:property name="end_effector_left" value="$(arg end_effector_left)" />
@@ -27,6 +27,6 @@
   <xacro:property name="is_multiple" value="$(arg multiple)" />
   <xacro:property name="nsp" value="$(arg namespace)" />
-  <xacro:if value="${version not in ['v1', 'v2']}">
-    <xacro:wrong_ari_version/>
+  <xacro:if value="${robot_model not in ['v1', 'v2']}">
+    <xacro:wrong_ari_robot_model/>
   </xacro:if>
   <xacro:if value="${end_effector_right not in ['ari-hand', 'false', False]}">
@@ -61,5 +61,5 @@
   <xacro:property name="head_link_name"          value="head_2_link"/>
   <!-- The following included files set up definitions of parts of the robot body -->
-  <xacro:if value="${version == 'v1'}">
+  <xacro:if value="${robot_model == 'v1'}">
       <xacro:include filename="$(find ari_description)/urdf/base/base.urdf.xacro" />   <!-- Base -->
       <xacro:include filename="$(find ari_description)/urdf/torso/torso_sensors.urdf.xacro" /> <!-- Torso -->
@@ -67,5 +67,5 @@
       <xacro:include filename="$(find ari_description)/urdf/head/head.urdf.xacro" /> <!-- head -->
   </xacro:if>
-  <xacro:if value="${version == 'v2'}">
+  <xacro:if value="${robot_model == 'v2'}">
       <xacro:include filename="$(find ari_description)/urdf/base/base_v2.urdf.xacro" />   <!-- Base -->
       <xacro:include filename="$(find ari_description)/urdf/torso/torso_sensors_v2.urdf.xacro" /> <!-- Torso -->
@@ -81,5 +81,5 @@
   <xacro:torso_sensors name="torso" parent="base_link"/>
   <xacro:head name="head" parent="base_link"/>
-  <xacro:if value="${version == 'v1'}">
+  <xacro:if value="${robot_model == 'v1'}">
   <xacro:ari_arm name="arm" parent="base_link" side="left" reflect="1" end_effector="${end_effector_left == 'ari-hand'}">
     <origin xyz="-0.219 0.097624 1.1111" rpy="${105.0 * deg_to_rad} ${0.0 * deg_to_rad} ${-180.0 * deg_to_rad}" />
@@ -89,5 +89,5 @@
   </xacro:ari_arm>
   </xacro:if>
-  <xacro:if value="${version == 'v2'}">
+  <xacro:if value="${robot_model == 'v2'}">
   <xacro:ari_arm name="arm" parent="base_link" side="left" reflect="1" end_effector="${end_effector_left == 'ari-hand'}">
     <origin xyz="-0.22 0.08146 1.153" rpy="${0* deg_to_rad} ${0 * deg_to_rad} ${0 * deg_to_rad}" />

File: ari_description/urdf/arm/arm_v2.urdf.xacro (robot description, xacro)
@@ -19,8 +19,10 @@
   <xacro:property name="arm_3_max_vel"      value="2.35" />
   <xacro:property name="arm_4_max_vel"      value="2.35" />
+  <xacro:property name="arm_5_max_vel"      value="2.35" />
   <xacro:property name="arm_1_max_effort"   value="10.0" />
   <xacro:property name="arm_2_max_effort"   value="10.0" />
   <xacro:property name="arm_3_max_effort"   value="5" />
   <xacro:property name="arm_4_max_effort"   value="5" />
+  <xacro:property name="arm_5_max_effort"   value="5" />
   <xacro:property name="arm_eps"            value="0.07" />
   <xacro:macro name="ari_arm" params="name parent side reflect end_effector *origin">
@@ -76,5 +78,5 @@
         <origin xyz="0 0 0" rpy="0 0 0" />
         <geometry>
-          <mesh filename="package://ari_description/meshes/arm/arm_1_v2.stl" scale=" ${reflect} 1 1"/>
+          <mesh filename="package://ari_description/meshes/arm/arm_1_v2.stl" scale="${reflect} 1 1"/>
         </geometry>
         <material name="White"/>
@@ -92,5 +94,5 @@
       <origin xyz="0.0 0.0047319 -0.00041399" rpy="${(-90 - 5.0) * deg_to_rad} 0.0 0.0"/>
       <axis xyz="0 0 ${-1 * reflect}" />
-      <limit lower="${-120.0 * deg_to_rad}" upper="${120.0 * deg_to_rad}" effort="0" velocity="0" />
+      <limit lower="${-120.0 * deg_to_rad}" upper="${120.0 * deg_to_rad}" effort="${arm_1_max_effort}" velocity="${arm_1_max_vel}" />
       <dynamics friction="${arm_friction}" damping="${arm_damping}"/>
       <safety_controller k_position="20"
@@ -243,5 +245,5 @@
       <xacro:property name="arm_5_lower_limit"       value="-5.0"/>
       <limit lower="${-120 * deg_to_rad}" upper="${120 * deg_to_rad}"
-        effort="${arm_4_max_effort}" velocity="${arm_4_max_vel}" />
+        effort="${arm_5_max_effort}" velocity="${arm_5_max_vel}" />
       <dynamics friction="${arm_friction}" damping="${arm_damping}"/>
       <safety_controller k_position="20"
@@ -270,21 +272,9 @@
      <material>Gazebo/DarkGrey</material>
    </gazebo>
-      <gazebo reference="${name}_${side}_5 _link">
-     <mu1>0.9</mu1>
-     <mu2>0.9</mu2>
-     <material>Gazebo/DarkGrey</material>
-   </gazebo>
-   <xacro:if value="${end_effector}">
-     <gazebo reference="hand_${side}_1_link">
-       <mu1>0.9</mu1>
-       <mu2>0.9</mu2>
-       <material>Gazebo/DarkGrey</material>
-     </gazebo>
-     <gazebo reference="hand_${side}_2_link">
-       <mu1>0.9</mu1>
-       <mu2>0.9</mu2>
-       <material>Gazebo/DarkGrey</material>
-     </gazebo>
-   </xacro:if>
+   <gazebo reference="${name}_${side}_5_link">
+     <mu1>0.9</mu1>
+     <mu2>0.9</mu2>
+     <material>Gazebo/DarkGrey</material>
+   </gazebo>
    <gazebo reference="${name}_${side}_1_joint">
       <implicitSpringDamper>1</implicitSpringDamper>
@@ -299,28 +289,12 @@
       <implicitSpringDamper>1</implicitSpringDamper>
    </gazebo>
-      <gazebo reference="${name}_${side}_5_joint">
-      <implicitSpringDamper>1</implicitSpringDamper>
-   </gazebo>
-   <xacro:if value="${end_effector}">
-     <gazebo reference="hand_${side}_virtual_1_joint">
-        <implicitSpringDamper>1</implicitSpringDamper>
-     </gazebo>
-     <gazebo reference="hand_${side}_virtual_2_joint">
-        <implicitSpringDamper>1</implicitSpringDamper>
-     </gazebo>
-   </xacro:if>
+   <gazebo reference="${name}_${side}_5_joint">
+      <implicitSpringDamper>1</implicitSpringDamper>
+   </gazebo>
     <xacro:arm_simple_transmission name="${name}" side="${side}" number="1" reduction="1.0" offset_value="0.0"/>
     <xacro:arm_simple_transmission name="${name}" side="${side}" number="2" reduction="1.0" offset_value="0.0"/>
     <xacro:arm_simple_transmission name="${name}" side="${side}" number="3" reduction="1.0" offset_value="0.0"/>
     <xacro:arm_simple_transmission name="${name}" side="${side}" number="4" reduction="1.0" offset_value="0.0"/>
-    <xacro:if value="${end_effector}">
-      <xacro:finger_transmissions finger_name="hand_${side}"
-                                  act_name="hand_${side}_fingers_motor"
-                                  start="0.0"
-                                  reduction="1.0"/>
-      <!-- <xacro:arm_simple_transmission name="${name}" side="${side}" number="4" reduction="1.0" offset_value="0.0"/> -->
-      <!-- gazebo plugin -->
-      <xacro:ari_hand_gazebo_simulation side="${side}"/>
-    </xacro:if>
+    <xacro:arm_simple_transmission name="${name}" side="${side}" number="5" reduction="1.0" offset_value="0.0"/>
   </xacro:macro>
 </robot>

Commit message: Update launch files and add meshes

File: ari_description/robots/ari.urdf.xacro (robot description, xacro)
@@ -90,8 +90,8 @@
   </xacro:if>
   <xacro:if value="${robot_model == 'v2'}">
-  <xacro:ari_arm name="arm" parent="base_link" side="left" reflect="1" end_effector="${end_effector_left == 'ari-hand'}">
+  <xacro:ari_arm name="arm" parent="base_link" side="left" reflect="1" end_effector="false">
     <origin xyz="-0.22 0.08146 1.153" rpy="${0* deg_to_rad} ${0 * deg_to_rad} ${0 * deg_to_rad}" />
   </xacro:ari_arm>
-  <xacro:ari_arm name="arm" parent="base_link" side="right" reflect="-1" end_effector="${end_effector_right == 'ari-hand'}">
+  <xacro:ari_arm name="arm" parent="base_link" side="right" reflect="-1" end_effector="false">
     <origin xyz="-0.22 -0.08146 1.153" rpy="${0 * deg_to_rad} ${0* deg_to_rad} ${180 * deg_to_rad}" />
   </xacro:ari_arm>

File: ari_description/urdf/arm/arm_v2.urdf.xacro (robot description, xacro)
@@ -119,5 +119,5 @@
         <origin xyz="0 0 0" rpy="0 0 0" />
         <geometry>
-          <mesh filename="package://ari_description/meshes/arm/arm_2_v2.stl" scale="1 1 ${reflect}"/>
+          <mesh filename="package://ari_description/meshes/arm/arm_2_v2.stl" scale="1 1 ${reflect}" />
         </geometry>
       </collision>
@@ -205,13 +205,13 @@
       <origin xyz="0 0.00049107 -0.1001"
               rpy="${90 * deg_to_rad} ${-90 * deg_to_rad} 0" />
-      <axis xyz="0 0 ${1*reflect}" />
+      <axis xyz="0 0 ${-1 * reflect}" />
       <xacro:property name="arm_4_upper_limit"       value="135.0"/>
       <xacro:property name="arm_4_lower_limit"       value="-5.0"/>
-      <limit lower="${-100 * deg_to_rad}" upper="${0 * deg_to_rad}" effort="${arm_4_max_effort}" velocity="${arm_4_max_vel}" />
-      <dynamics friction="${arm_friction}" damping="${arm_damping}"/>
-      <safety_controller k_position="20"
-                         k_velocity="20"
-                         soft_lower_limit="${-100 * deg_to_rad + arm_eps}"
-                         soft_upper_limit="${0 * deg_to_rad - arm_eps}" />
+      <limit lower="${0 * deg_to_rad}" upper="${135 * deg_to_rad}" effort="${arm_4_max_effort}" velocity="${arm_4_max_vel}" />
+      <dynamics friction="${arm_friction}" damping="${arm_damping}"/>
+      <safety_controller k_position="20"
+                         k_velocity="20"
+                         soft_lower_limit="${0 * deg_to_rad + arm_eps}"
+                         soft_upper_limit="${135 * deg_to_rad - arm_eps}" />
     </joint>
     <link name="${name}_${side}_5_link">

File: ari_description/urdf/base/base_v2.urdf.xacro (robot description, xacro)
@@ -14,12 +14,12 @@
   <xacro:include filename="$(find ari_description)/urdf/base/docking_link_v2.urdf.xacro"/>
   <!-- Wheel characteristics -->
-  <xacro:property name="wheel_radius"     value="0.125"/>
-  <xacro:property name="wheel_width"      value="0.075"/>
+  <xacro:property name="wheel_radius"     value="0.11"/>
+  <xacro:property name="wheel_width"      value="0.06"/>
   <xacro:property name="wheel_separation" value="0.4668"/>
   <xacro:property name="wheel_torque"     value="6.0"/>
   <xacro:property name="wheel_velocity"   value="1.0"/>
   <!-- Caster wheel characteristics -->
-  <xacro:property name="caster_radius"       value="0.045"/>
-  <xacro:property name="caster_width"        value="0.055"/>
+  <xacro:property name="caster_radius"       value="0.040"/>
+  <xacro:property name="caster_width"        value="0.045"/>
   <xacro:property name="caster_separation_x" value="0.91"/>
   <xacro:property name="caster_offset_y"     value="0.0875"/>

File: ari_description/urdf/head/head_v2.urdf.xacro (robot description, xacro)
@@ -55,5 +55,5 @@
       <origin xyz="0 0 0" rpy="0 0 0" />
       <geometry>
-        <mesh filename="package://ari_description/meshes/head/head_base_v2.stl" scale="1 1 1"/>
+          <mesh filename="package://ari_description/meshes/head/head_base_v2.stl" scale="1 1 1"/>
       </geometry>
     </collision>

File: ari_description/urdf/wheels/caster_v2.urdf.xacro (robot description, xacro)
@@ -19,14 +19,14 @@
       </inertial>
       <visual>
-        <origin xyz="0 0 0" rpy="0 0 0"/>
+        <origin xyz="0.0 0.0 0.0" rpy="0 0 0"/>
         <geometry>
-          <mesh filename="package://ari_description/meshes/wheels/caster_v2.stl" scale="1 ${reflect} 1"/>
+          <mesh filename="package://ari_description/meshes/wheels/caster_v2.stl" scale="1 1 1"/>
         </geometry>
         <material name="Grey"/>
       </visual>
       <collision>
-        <origin xyz="0 0 0" rpy="0 0 0"/>
+        <origin xyz="-0.02 0 -0.023" rpy="${90 * deg_to_rad} 0 0"/>
         <geometry>
-          <mesh filename="package://ari_description/meshes/wheels/caster_v2.stl" scale="1 ${reflect} 1"/>
+          <cylinder radius="${radius}" length="${width}"/>
         </geometry>
       </collision>

File: ari_description/urdf/wheels/wheel_v2.urdf.xacro (robot description, xacro)
@@ -8,6 +8,6 @@
 -->
 <robot xmlns:xacro="http://ros.org/wiki/xacro">
-  <xacro:include filename="$(find ari_description)/urdf/wheels/wheel_v2.transmission.xacro"/>
-  <xacro:include filename="$(find ari_description)/urdf/wheels/wheel_v2.gazebo.xacro"/>
+  <xacro:include filename="$(find ari_description)/urdf/wheels/wheel.transmission.xacro"/>
+  <xacro:include filename="$(find ari_description)/urdf/wheels/wheel.gazebo.xacro"/>
   <xacro:macro name="wheel" params="side reflect radius width torque velocity separation parent">
     <link name="wheel_${side}_link">
@@ -20,5 +20,5 @@
     </inertial>
       <visual>
-        <origin xyz="0 0 0" rpy="0 0 0"/>
+        <origin xyz="0 0 0" rpy="${-90 * deg_to_rad}  0 0"/>
         <geometry>
           <mesh filename="package://ari_description/meshes/wheels/wheel_${side}_v2.stl"/>
@@ -29,5 +29,5 @@
         <origin xyz="0 0 0" rpy="0 0 0"/>
         <geometry>
-          <mesh filename="package://ari_description/meshes/wheels/wheel_${side}_v2.stl"/>
+          <cylinder radius="${radius}" length="${width}"/>
         </geometry>
       </collision>
@@ -38,5 +38,5 @@
       <parent link="${parent}_link"/>
       <child link="wheel_${side}_link"/>
-      <origin xyz="0 ${ -separation / 2 * reflect} 0" rpy="${0 * deg_to_rad} 0 0"/>
+      <origin xyz="0 ${ -separation / 2 * reflect} 0" rpy="${90 * deg_to_rad} 0 0"/>
       <axis xyz="0 0 -1"/>
       <limit effort="${torque}" velocity="${velocity / radius}"/>
