Commit message: Combine base torso and head urdf files for v1 and v2

File: ari_description/robots/ari.urdf.xacro (robot description, xacro)
@@ -61,15 +61,12 @@
   <xacro:property name="head_link_name"          value="head_2_link"/>
   <!-- The following included files set up definitions of parts of the robot body -->
+  <xacro:include filename="$(find ari_description)/urdf/base/base.urdf.xacro" />   <!-- Base -->
+  <xacro:include filename="$(find ari_description)/urdf/head/head.urdf.xacro" /> <!-- head -->
+  <xacro:include filename="$(find ari_description)/urdf/torso/torso_sensors.urdf.xacro" /> <!-- Torso -->
   <xacro:if value="${robot_model == 'v1'}">
-      <xacro:include filename="$(find ari_description)/urdf/base/base.urdf.xacro" />   <!-- Base -->
-      <xacro:include filename="$(find ari_description)/urdf/torso/torso_sensors.urdf.xacro" /> <!-- Torso -->
       <xacro:include filename="$(find ari_description)/urdf/arm/arm.urdf.xacro" />   <!-- Arms -->
-      <xacro:include filename="$(find ari_description)/urdf/head/head.urdf.xacro" /> <!-- head -->
   </xacro:if>
   <xacro:if value="${robot_model == 'v2'}">
-      <xacro:include filename="$(find ari_description)/urdf/base/base_v2.urdf.xacro" />   <!-- Base -->
-      <xacro:include filename="$(find ari_description)/urdf/torso/torso_sensors_v2.urdf.xacro" /> <!-- Torso -->
       <xacro:include filename="$(find ari_description)/urdf/arm/arm_v2.urdf.xacro" />   <!-- Arms -->
-      <xacro:include filename="$(find ari_description)/urdf/head/head_v2.urdf.xacro" /> <!-- head -->
   </xacro:if>
   <!-- Generic simulator_gazebo plugins -->
@@ -78,7 +75,7 @@
   <xacro:include filename="$(find ari_description)/urdf/materials.urdf.xacro" />
   <!-- Now we can start using the macros included above to define the actual robot -->
-  <xacro:base name="base"/>
-  <xacro:torso_sensors name="torso" parent="base_link"/>
-  <xacro:head name="head" parent="base_link"/>
+  <xacro:base name="base" robot_model="${robot_model}"/>
+  <xacro:torso_sensors name="torso" parent="base_link" robot_model="${robot_model}"/>
+  <xacro:head name="head" parent="base_link" robot_model="${robot_model}"/>
   <xacro:if value="${robot_model == 'v1'}">
   <xacro:ari_arm name="arm" parent="base_link" side="left" reflect="1" end_effector="${end_effector_left == 'ari-hand'}">

File: ari_description/urdf/base/base.urdf.xacro (robot description, xacro)
@@ -8,21 +8,40 @@
 -->
 <robot xmlns:xacro="http://ros.org/wiki/xacro">
-  <!--File includes-->
   <xacro:include filename="$(find ari_description)/urdf/deg_to_rad.xacro" />
-  <xacro:include filename="$(find ari_description)/urdf/wheels/wheel.urdf.xacro"/>
-  <xacro:include filename="$(find ari_description)/urdf/wheels/caster.urdf.xacro"/>
-  <!-- Wheel characteristics -->
-  <xacro:property name="wheel_radius"     value="0.125"/>
-  <xacro:property name="wheel_width"      value="0.075"/>
-  <xacro:property name="wheel_separation" value="0.44"/>
+  <xacro:macro name="base" params="name robot_model">
+    <xacro:if value="${robot_model == 'v1'}">
+    <!--File includes-->
+      <xacro:include filename="$(find ari_description)/urdf/wheels/wheel.urdf.xacro"/>
+      <xacro:include filename="$(find ari_description)/urdf/wheels/caster.urdf.xacro"/>
+      <!-- Wheel characteristics -->
+      <xacro:property name="wheel_radius"     value="0.125"/>
+      <xacro:property name="wheel_width"      value="0.075"/>
+      <xacro:property name="wheel_separation" value="0.44"/>
+      <xacro:property name="wheel_torque"     value="6.0"/>
+      <xacro:property name="wheel_velocity"   value="1.0"/>
+          <!-- Caster wheel characteristics -->
+      <xacro:property name="caster_radius"       value="0.045"/>
+      <xacro:property name="caster_width"        value="0.055"/>
+      <xacro:property name="caster_separation_x" value="0.91"/>
+      <xacro:property name="caster_offset_y"     value="0.1025"/>
+      <xacro:property name="caster_offset_z"     value="-0.08"/>
+    </xacro:if>
+    <xacro:if value="${robot_model == 'v2'}">
+      <!--File includes-->
+      <xacro:include filename="$(find ari_description)/urdf/wheels/wheel_v2.urdf.xacro"/>
+      <xacro:include filename="$(find ari_description)/urdf/wheels/caster_v2.urdf.xacro"/>
+      <!-- Wheel characteristics -->
+  <xacro:property name="wheel_radius"     value="0.1"/>
+  <xacro:property name="wheel_width"      value="0.06"/>
+  <xacro:property name="wheel_separation" value="0.4668"/>
   <xacro:property name="wheel_torque"     value="6.0"/>
   <xacro:property name="wheel_velocity"   value="1.0"/>
   <!-- Caster wheel characteristics -->
-  <xacro:property name="caster_radius"       value="0.045"/>
-  <xacro:property name="caster_width"        value="0.055"/>
+  <xacro:property name="caster_radius"       value="0.040"/>
+  <xacro:property name="caster_width"        value="0.045"/>
   <xacro:property name="caster_separation_x" value="0.91"/>
-  <xacro:property name="caster_offset_y"     value="0.1025"/>
-  <xacro:property name="caster_offset_z"     value="-0.08"/>
-  <xacro:macro name="base" params="name">
+  <xacro:property name="caster_offset_y"     value="0.0875"/>
+  <xacro:property name="caster_offset_z"     value="-0.0305"/>
+    </xacro:if>
   <!-- Base -->
   <link name="${name}_link">
@@ -37,5 +56,10 @@
       <origin xyz="0 0 0" rpy="0 0 0" />
       <geometry>
-        <mesh filename="package://ari_description/meshes/base/base.stl" />
+        <xacro:if value="${robot_model == 'v1'}">
+          <mesh filename="package://ari_description/meshes/base/base.stl" />
+        </xacro:if>
+        <xacro:if value="${robot_model == 'v2'}">
+          <mesh filename="package://ari_description/meshes/base/base_v2.stl" />
+        </xacro:if>
       </geometry>
       <material name="Grey" />
@@ -44,5 +68,10 @@
       <origin xyz="0 0 0" rpy="0 0 0" />
       <geometry>
-        <mesh filename="package://ari_description/meshes/base/base_collision.stl" />
+        <xacro:if value="${robot_model == 'v1'}">
+          <mesh filename="package://ari_description/meshes/base/base_collision.stl" />
+        </xacro:if>
+        <xacro:if value="${robot_model == 'v2'}">
+          <mesh filename="package://ari_description/meshes/base/base_v2.stl" />
+        </xacro:if>
       </geometry>
       <material name="Grey" />
@@ -78,4 +107,22 @@
   <xacro:caster side="left"  reflect="-1.0" radius="${caster_radius}" width="${caster_width}" separation_x="${caster_separation_x}" offset_y="${caster_offset_y}"
                 offset_z="${caster_offset_z}" parent="${name}"/>
+  <!-- Docking Link -->
+  <joint name="docking_joint" type="fixed">
+      <parent link="base_link"/>
+      <child link="docking_link"/>
+      <xacro:if value="${robot_model == 'v1'}">
+        <origin xyz="-0.602 0 0" rpy="0 0 0" />
+      </xacro:if>
+      <xacro:if value="${robot_model == 'v2'}">
+        <origin xyz="-0.600830 0 0.039" rpy="0 0 0" />
+      </xacro:if>
+  </joint>
+  <link name="docking_link">
+      <inertial>
+          <origin xyz="0 0 0" rpy="0 0 0"/>
+          <mass value="0.0001" />
+          <inertia ixx="0.0001"  ixy="0"  ixz="0" iyy="0.0001" iyz="0" izz="0.0001" />
+      </inertial>
+  </link>
   </xacro:macro>
   <!-- RGBD Laser Link -->
@@ -106,16 +153,3 @@
     </inertial>
   </link>
-  <!-- Docking Link -->
-  <joint name="docking_joint" type="fixed">
-      <parent link="base_link"/>
-      <child link="docking_link"/>
-      <origin xyz="-0.602 0 0" rpy="0 0 0" />
-  </joint>
-  <link name="docking_link">
-      <inertial>
-          <origin xyz="0 0 0" rpy="0 0 0"/>
-          <mass value="0.0001" />
-          <inertia ixx="0.0001"  ixy="0"  ixz="0" iyy="0.0001" iyz="0" izz="0.0001" />
-      </inertial>
-  </link>
 </robot>

File: ari_description/urdf/head/head.urdf.xacro (robot description, xacro)
@@ -34,5 +34,5 @@
   <!--     HEAD_1 (PAN)       -->
   <!--************************-->
-  <xacro:macro name="head_1" params="name parent">
+  <xacro:macro name="head_1" params="name parent robot_model">
     <link name="${name}_link">
       <inertial>
@@ -46,5 +46,10 @@
         <origin xyz="0 0 0" rpy="0 0 0"/>
         <geometry>
-          <mesh filename="package://ari_description/meshes/head/head_1.stl" scale="1 1 1"/>
+          <xacro:if value="${robot_model == 'v1'}">
+            <mesh filename="package://ari_description/meshes/head/head_1.stl" scale="1 1 1"/>
+          </xacro:if>
+          <xacro:if value="${robot_model == 'v2'}">
+            <mesh filename="package://ari_description/meshes/head/head_1_v2.stl" scale="1 1 1"/>
+          </xacro:if>
         </geometry>
         <material name="White" />
@@ -53,5 +58,10 @@
         <origin xyz="0.0 0 0" rpy="0 0 0.0" />
         <geometry>
-          <mesh filename="package://ari_description/meshes/head/head_1_collision.stl" scale="1 1 1"/>
+          <xacro:if value="${robot_model == 'v1'}">
+            <mesh filename="package://ari_description/meshes/head/head_1_collision.stl" scale="1 1 1"/>
+          </xacro:if>
+          <xacro:if value="${robot_model == 'v2'}">
+            <mesh filename="package://ari_description/meshes/head/head_1_v2.stl" scale="1 1 1"/>
+          </xacro:if>
         </geometry>
         <material name="White" />
@@ -61,5 +71,10 @@
       <parent link="${parent}"/>
       <child link="${name}_link"/>
-      <origin xyz="-0.2255 0 1.1915"  rpy="0 0 0" />
+      <xacro:if value="${robot_model == 'v1'}">
+        <origin xyz="-0.2255 0 1.1915"  rpy="0 0 0" />
+      </xacro:if>
+      <xacro:if value="${robot_model == 'v2'}">
+        <origin xyz="-0.22 0.0 1.207"  rpy="0 0 0" />
+      </xacro:if>
       <axis xyz="0 0 1" />
       <limit lower="${head_1_lower_limit * deg_to_rad}" upper="${head_1_upper_limit * deg_to_rad}" effort="3.4" velocity="${head_max_vel}" />
@@ -84,5 +99,5 @@
   <!--      HEAD_2 (TILT)     -->
   <!--************************-->
-  <xacro:macro name="head_2" params="name parent">
+  <xacro:macro name="head_2" params="name parent robot_model">
     <link name="${name}_link">
       <inertial>
@@ -111,5 +126,10 @@
       <parent link="${parent}"/>
       <child link="${name}_link"/>
-      <origin xyz="0.0425000000000001 0 0.093"  rpy="${90.0 * deg_to_rad} 0 0" />
+      <xacro:if value="${robot_model == 'v1'}">
+        <origin xyz="0.0425000000000001 0 0.093"  rpy="${90.0 * deg_to_rad} 0 0" />
+      </xacro:if>
+      <xacro:if value="${robot_model == 'v2'}">
+        <origin xyz="0.0425 0.0 0.1011"  rpy="${90.0 * deg_to_rad} 0 0" />
+      </xacro:if>
       <axis xyz="0 0 -1" />
       <limit lower="${head_2_lower_limit * deg_to_rad}" upper="${head_2_upper_limit * deg_to_rad}" effort="3.26" velocity="${head_max_vel}" />
@@ -218,7 +238,7 @@
     </inertial>
   </link>
-  <xacro:macro name="head" params="name parent">
-    <xacro:head_1 name="${name}_1" parent="${parent}" />
-    <xacro:head_2 name="${name}_2" parent="${name}_1_link"/>
+  <xacro:macro name="head" params="name parent robot_model">
+    <xacro:head_1 name="${name}_1" parent="${parent}" robot_model="${robot_model}" />
+    <xacro:head_2 name="${name}_2" parent="${name}_1_link" robot_model="${robot_model}"/>
     <xacro:if value="${camera_model_head == 'raspi'}">
       <xacro:head_front_camera name="${name}_front_camera" parent="${name}_2_link"/>

File: ari_description/urdf/torso/torso_sensors.urdf.xacro (robot description, xacro)
@@ -15,22 +15,39 @@
   <xacro:include filename="$(find ari_description)/urdf/sensors/imx179_camera.gazebo.xacro"/>
   <xacro:include filename="$(find ari_description)/urdf/sensors/sick_tim571_laser.urdf.xacro"/>
-  <!--Constant parameters-->
-  <xacro:property name="torso_front_camera_position_x" value="-0.11249" />
-  <xacro:property name="torso_front_camera_position_y" value="0.0" />
-  <xacro:property name="torso_front_camera_position_z" value="0.97052" />
-  <xacro:property name="torso_front_camera_orientation_r" value="0.0" />
-  <xacro:property name="torso_front_camera_orientation_p" value="${42.5 * deg_to_rad}" />
-  <xacro:property name="torso_front_camera_orientation_y" value="0.0" />
-  <xacro:property name="torso_back_camera_position_x" value="-0.3275" />
-  <xacro:property name="torso_back_camera_position_y" value="0.009" />
-  <xacro:property name="torso_back_camera_position_z" value="1.0337" />
-  <xacro:property name="torso_back_camera_orientation_r" value="0.0" />
-  <xacro:property name="torso_back_camera_orientation_p" value="${15 * deg_to_rad}" />
-  <xacro:property name="torso_back_camera_orientation_y" value="${180 * deg_to_rad}" />
   <!-- Laser characteristics -->
   <xacro:property name="base_laser_x" value="-0.34"/>
   <xacro:property name="base_laser_y" value="0.0"/>
   <xacro:property name="base_laser_z" value="0.564"/>
-  <xacro:macro name="torso_sensors" params="name parent">
+  <xacro:macro name="torso_sensors" params="name parent robot_model">
+    <xacro:if value="${robot_model == 'v1'}">
+      <!--Constant parameters-->
+      <xacro:property name="torso_front_camera_position_x" value="-0.11249" />
+      <xacro:property name="torso_front_camera_position_y" value="0.0" />
+      <xacro:property name="torso_front_camera_position_z" value="0.97052" />
+      <xacro:property name="torso_front_camera_orientation_r" value="0.0" />
+      <xacro:property name="torso_front_camera_orientation_p" value="${42.5 * deg_to_rad}" />
+      <xacro:property name="torso_front_camera_orientation_y" value="0.0" />
+      <xacro:property name="torso_back_camera_position_x" value="-0.3275" />
+      <xacro:property name="torso_back_camera_position_y" value="0.009" />
+      <xacro:property name="torso_back_camera_position_z" value="1.0337" />
+      <xacro:property name="torso_back_camera_orientation_r" value="0.0" />
+      <xacro:property name="torso_back_camera_orientation_p" value="${15 * deg_to_rad}" />
+      <xacro:property name="torso_back_camera_orientation_y" value="${180 * deg_to_rad}" />
+    </xacro:if>
+    <xacro:if value="${robot_model == 'v2'}">
+      <!--Constant parameters-->
+      <xacro:property name="torso_front_camera_position_x" value="-0.13799" />
+      <xacro:property name="torso_front_camera_position_y" value="-0.00034911" />
+      <xacro:property name="torso_front_camera_position_z" value="1.0305" />
+      <xacro:property name="torso_front_camera_orientation_r" value="0.0" />
+      <xacro:property name="torso_front_camera_orientation_p" value="${43 * deg_to_rad}" />
+      <xacro:property name="torso_front_camera_orientation_y" value="0.0" />
+      <xacro:property name="torso_back_camera_position_x" value="-0.31955" />
+      <xacro:property name="torso_back_camera_position_y" value="0.009" />
+      <xacro:property name="torso_back_camera_position_z" value="1.0599" />
+      <xacro:property name="torso_back_camera_orientation_r" value="0.0" />
+      <xacro:property name="torso_back_camera_orientation_p" value="${15 * deg_to_rad}" />
+      <xacro:property name="torso_back_camera_orientation_y" value="${180 * deg_to_rad}" />
+    </xacro:if>
   <!-- Torso sensors -->
   <!-- Torso front camera -->

Commit message: set nominal extrinsics as param

File: ari_description/robots/ari.urdf.xacro (robot description, xacro)
@@ -16,4 +16,5 @@
   <xacro:arg name="camera_model_head" default="raspi"/>
   <xacro:arg name="has_thermal" default="false"/>
+  <xacro:arg name="use_nominal_extrinsics" default="false" />
   <xacro:property name="robot_model" value="$(arg robot_model)" />
   <xacro:property name="end_effector_right" value="$(arg end_effector_right)" />
@@ -27,4 +28,5 @@
   <xacro:property name="is_multiple" value="$(arg multiple)" />
   <xacro:property name="nsp" value="$(arg namespace)" />
+  <xacro:property name="use_nominal_extrinsics" value="$(arg use_nominal_extrinsics)"/>
   <xacro:if value="${robot_model not in ['v1', 'v2']}">
     <xacro:wrong_ari_robot_model/>
@@ -76,5 +78,5 @@
   <!-- Now we can start using the macros included above to define the actual robot -->
   <xacro:base name="base" robot_model="${robot_model}"/>
-  <xacro:torso_sensors name="torso" parent="base_link" robot_model="${robot_model}"/>
+  <xacro:torso_sensors name="torso" parent="base_link" robot_model="${robot_model}" use_nominal_extrinsics="${use_nominal_extrinsics}" />
   <xacro:head name="head" parent="base_link" robot_model="${robot_model}"/>
   <xacro:if value="${robot_model == 'v1'}">

File: ari_description/urdf/torso/torso_sensors.urdf.xacro (robot description, xacro)
@@ -19,5 +19,5 @@
   <xacro:property name="base_laser_y" value="0.0"/>
   <xacro:property name="base_laser_z" value="0.564"/>
-  <xacro:macro name="torso_sensors" params="name parent robot_model">
+  <xacro:macro name="torso_sensors" params="name parent robot_model use_nominal_extrinsics">
     <xacro:if value="${robot_model == 'v1'}">
       <!--Constant parameters-->
@@ -52,5 +52,5 @@
   <!-- Torso sensors -->
   <!-- Torso front camera -->
-  <sensor_d435 parent="${parent}" name="${name}_front_camera" topics_ns="${name}_front_camera">
+  <sensor_d435 parent="${parent}" name="${name}_front_camera" topics_ns="${name}_front_camera" use_nominal_extrinsics="${use_nominal_extrinsics}">
     <origin xyz="${torso_front_camera_position_x} ${torso_front_camera_position_y} ${torso_front_camera_position_z}"
             rpy="${torso_front_camera_orientation_r} ${torso_front_camera_orientation_p} ${torso_front_camera_orientation_y}"/>

Commit message: change parameter name

File: ari_description/robots/ari.urdf.xacro (robot description, xacro)
@@ -16,5 +16,5 @@
   <xacro:arg name="camera_model_head" default="raspi"/>
   <xacro:arg name="has_thermal" default="false"/>
-  <xacro:arg name="use_nominal_extrinsics" default="false" />
+  <xacro:arg name="simulation" default="false" />
   <xacro:property name="robot_model" value="$(arg robot_model)" />
   <xacro:property name="end_effector_right" value="$(arg end_effector_right)" />
@@ -28,5 +28,5 @@
   <xacro:property name="is_multiple" value="$(arg multiple)" />
   <xacro:property name="nsp" value="$(arg namespace)" />
-  <xacro:property name="use_nominal_extrinsics" value="$(arg use_nominal_extrinsics)"/>
+  <xacro:property name="use_nominal_extrinsics" value="$(arg simulation)"/>
   <xacro:if value="${robot_model not in ['v1', 'v2']}">
     <xacro:wrong_ari_robot_model/>

Commit message: added support to ydlidar

File: ari_description/robots/ari.urdf.xacro (robot description, xacro)
@@ -56,5 +56,5 @@
   <xacro:property name="has_front_fisheye_camera"           value="${front_fisheye_camera in ['Jetson', True, 'true', 'PC']}"/>
   <xacro:property name="has_back_fisheye_camera"           value="${back_fisheye_camera in ['Jetson', True, 'true', 'PC']}"/>
-  <xacro:if value="${laser_model not in ['No', 'false', False, 'sick-551', 'sick-561', 'sick-571', 'hokuyo']}">
+  <xacro:if value="${laser_model not in ['No', 'false', False, 'sick-551', 'sick-561', 'sick-571', 'hokuyo', 'ydlidar-tg30']}">
     <xacro:wrong_laser_model/>
   </xacro:if>

File: ari_description/urdf/torso/torso_sensors.urdf.xacro (robot description, xacro)
@@ -125,4 +125,11 @@
     </xacro:sick_tim571_laser>
   </xacro:if>
+  <xacro:if value="${laser_model == 'ydlidar-tg30'}">
+    <!-- Laser -->
+    <!-- Theoretic FOV = 220 -->
+    <xacro:sick_tim571_laser name="${name}_laser" parent="${parent}" ros_topic="scan_raw" update_rate="10" min_angle="${-180 * deg_to_rad}" max_angle="${180 * deg_to_rad}" >
+      <origin xyz="${base_laser_x} ${base_laser_y} ${base_laser_z}" rpy="0 0 ${ 180 * deg_to_rad }" />
+    </xacro:sick_tim571_laser>
+  </xacro:if>
  </xacro:macro>
 </robot>

Commit message: added support to ydlidar 15 and 30

File: ari_description/robots/ari.urdf.xacro (robot description, xacro)
@@ -56,5 +56,5 @@
   <xacro:property name="has_front_fisheye_camera"           value="${front_fisheye_camera in ['Jetson', True, 'true', 'PC']}"/>
   <xacro:property name="has_back_fisheye_camera"           value="${back_fisheye_camera in ['Jetson', True, 'true', 'PC']}"/>
-  <xacro:if value="${laser_model not in ['No', 'false', False, 'sick-551', 'sick-561', 'sick-571', 'hokuyo', 'ydlidar-tg30']}">
+  <xacro:if value="${laser_model not in ['No', 'false', False, 'sick-551', 'sick-561', 'sick-571', 'hokuyo', 'ydlidar-tg30', 'ydlidar-tg15']}">
     <xacro:wrong_laser_model/>
   </xacro:if>

File: ari_description/urdf/torso/torso_sensors.urdf.xacro (robot description, xacro)
@@ -15,4 +15,6 @@
   <xacro:include filename="$(find ari_description)/urdf/sensors/imx179_camera.gazebo.xacro"/>
   <xacro:include filename="$(find ari_description)/urdf/sensors/sick_tim571_laser.urdf.xacro"/>
+  <xacro:include filename="$(find ari_description)/urdf/sensors/ydlidar_tg30_laser.urdf.xacro"/>
+  <xacro:include filename="$(find ari_description)/urdf/sensors/ydlidar_tg15_laser.urdf.xacro"/>
   <!-- Laser characteristics -->
   <xacro:property name="base_laser_x" value="-0.34"/>
@@ -127,8 +129,15 @@
   <xacro:if value="${laser_model == 'ydlidar-tg30'}">
     <!-- Laser -->
-    <!-- Theoretic FOV = 220 -->
-    <xacro:sick_tim571_laser name="${name}_laser" parent="${parent}" ros_topic="scan_raw" update_rate="10" min_angle="${-180 * deg_to_rad}" max_angle="${180 * deg_to_rad}" >
+    <!-- Theoretic FOV = 360 -->
+    <xacro:ydlidar_tg30_laser name="${name}_laser" parent="${parent}" ros_topic="scan_raw" update_rate="10" min_angle="${-180 * deg_to_rad}" max_angle="${180 * deg_to_rad}" >
       <origin xyz="${base_laser_x} ${base_laser_y} ${base_laser_z}" rpy="0 0 ${ 180 * deg_to_rad }" />
-    </xacro:sick_tim571_laser>
+    </xacro:ydlidar_tg30_laser>
+  </xacro:if>
+  <xacro:if value="${laser_model == 'ydlidar-tg15'}">
+    <!-- Laser -->
+    <!-- Theoretic FOV = 360 -->
+    <xacro:ydlidar_tg15_laser name="${name}_laser" parent="${parent}" ros_topic="scan_raw" update_rate="10" min_angle="${-180 * deg_to_rad}" max_angle="${180 * deg_to_rad}" >
+      <origin xyz="${base_laser_x} ${base_laser_y} ${base_laser_z}" rpy="0 0 ${ 180 * deg_to_rad }" />
+    </xacro:ydlidar_tg15_laser>
   </xacro:if>
  </xacro:macro>
