Commit message: modified position ari v1 ydlidar

File: ari_description/robots/ari.urdf.xacro (robot description, xacro)
@@ -78,5 +78,5 @@
   <!-- Now we can start using the macros included above to define the actual robot -->
   <xacro:base name="base" robot_model="${robot_model}"/>
-  <xacro:torso_sensors name="torso" parent="base_link" robot_model="${robot_model}" use_nominal_extrinsics="${use_nominal_extrinsics}" />
+  <xacro:torso_sensors name="torso" parent="base_link" robot_model="${robot_model}" use_nominal_extrinsics="${use_nominal_extrinsics}" laser_model="${laser_model}" />
   <xacro:head name="head" parent="base_link" robot_model="${robot_model}"/>
   <xacro:if value="${robot_model == 'v1'}">

File: ari_description/urdf/torso/torso_sensors.urdf.xacro (robot description, xacro)
@@ -17,5 +17,5 @@
   <xacro:include filename="$(find ari_description)/urdf/sensors/ydlidar_tg30_laser.urdf.xacro"/>
   <xacro:include filename="$(find ari_description)/urdf/sensors/ydlidar_tg15_laser.urdf.xacro"/>
-  <xacro:macro name="torso_sensors" params="name parent robot_model use_nominal_extrinsics">
+  <xacro:macro name="torso_sensors" params="name parent robot_model use_nominal_extrinsics laser_model">
     <xacro:if value="${robot_model == 'v1'}">
       <!--Constant parameters-->
@@ -32,8 +32,13 @@
       <xacro:property name="torso_back_camera_orientation_p" value="${15 * deg_to_rad}" />
       <xacro:property name="torso_back_camera_orientation_y" value="${180 * deg_to_rad}" />
-        <!-- Laser characteristics -->
+      <!-- Laser characteristics -->
       <xacro:property name="base_laser_x" value="-0.34"/>
       <xacro:property name="base_laser_y" value="0.0"/>
       <xacro:property name="base_laser_z" value="0.564"/>
+      <xacro:if value="${laser_model in ['ydlidar-tg30', 'ydlidar-tg15']}">
+        <xacro:property name="base_laser_x" value="-0.39777"/>
+        <xacro:property name="base_laser_y" value="0.0"/>
+        <xacro:property name="base_laser_z" value="0.26848"/>
+      </xacro:if>
     </xacro:if>
     <xacro:if value="${robot_model == 'v2'}">

Commit message: merge end_effector_left and end_effector_right
As, on ARI, both hands are identifical

File: ari_description/robots/ari.urdf.xacro (robot description, xacro)
@@ -15,6 +15,5 @@
         name="ari" >
   <xacro:arg name="robot_model" default="v2"/>
-  <xacro:arg name="end_effector_right" default="no-hand"/>
-  <xacro:arg name="end_effector_left" default="no-hand"/>
+  <xacro:arg name="end_effector" default="no-hand"/>
   <xacro:arg name="front_fisheye_camera" default="false"/>
   <xacro:arg name="back_fisheye_camera" default="false"/>
@@ -28,6 +27,5 @@
   <xacro:arg name="use_sim" default="true"/>
   <xacro:property name="robot_model" value="$(arg robot_model)" />
-  <xacro:property name="end_effector_right" value="$(arg end_effector_right)" />
-  <xacro:property name="end_effector_left" value="$(arg end_effector_left)" />
+  <xacro:property name="end_effector" value="$(arg end_effector)" />
   <xacro:property name="front_fisheye_camera" value="$(arg front_fisheye_camera)" />
   <xacro:property name="back_fisheye_camera" value="$(arg back_fisheye_camera)" />
@@ -42,8 +40,5 @@
     <xacro:wrong_ari_robot_model/>
   </xacro:if>
-  <xacro:if value="${end_effector_right not in ['ari-hand', 'no-hand', 'false', False]}">
-    <xacro:wrong_end_effector/>
-  </xacro:if>
-  <xacro:if value="${end_effector_left not in ['ari-hand', 'no-hand', 'false', False]}">
+  <xacro:if value="${end_effector not in ['ari-hand', 'no-hand', 'false', False]}">
     <xacro:wrong_end_effector/>
   </xacro:if>
@@ -95,8 +90,8 @@
   <xacro:head name="head" parent="base_link" robot_model="${robot_model}"/>
   <xacro:if value="${robot_model == 'v1'}">
-    <xacro:ari_arm name="arm" parent="base_link" side="left" reflect="1" end_effector="${end_effector_left == 'ari-hand'}">
+    <xacro:ari_arm name="arm" parent="base_link" side="left" reflect="1" end_effector="${end_effector == 'ari-hand'}">
       <origin xyz="-0.219 0.097624 1.1111" rpy="${105.0 * deg_to_rad} ${0.0 * deg_to_rad} ${-180.0 * deg_to_rad}" />
     </xacro:ari_arm>
-    <xacro:ari_arm name="arm" parent="base_link" side="right" reflect="-1" end_effector="${end_effector_right == 'ari-hand'}">
+    <xacro:ari_arm name="arm" parent="base_link" side="right" reflect="-1" end_effector="${end_effector == 'ari-hand'}">
       <origin xyz="-0.219 -0.097624 1.1111" rpy="${-105.0 * deg_to_rad} ${0.0 * deg_to_rad} ${180.0 * deg_to_rad}" />
     </xacro:ari_arm>

Commit message: use_sim_time=False by default

File: ari_description/robots/ari.urdf.xacro (robot description, xacro)
@@ -25,5 +25,5 @@
   <xacro:arg name="multiple" default="false"/>
   <xacro:arg name="namespace" default=""/>
-  <xacro:arg name="use_sim" default="true"/>
+  <xacro:arg name="use_sim" default="false"/>
   <xacro:property name="robot_model" value="$(arg robot_model)" />
   <xacro:property name="end_effector" value="$(arg end_effector)" />

File: ari_description/ros2_control/ros2_control.urdf.xacro (robot description, xacro)
@@ -14,5 +14,5 @@
 <robot xmlns:xacro="http://ros.org/wiki/xacro"
        name="ari" >
-  <xacro:macro name="ari_ros2_control" params="use_sim:=^|true">
+  <xacro:macro name="ari_ros2_control" params="use_sim:=^|false">
     <xacro:arg name="robot_model" default="v2" />
     <xacro:arg name="description_calibration_dir" default="$(find ari_description)/urdf/calibration" />

Commit message: uniform namespace arg

File: ari_description/robots/ari.urdf.xacro (robot description, xacro)
@@ -35,5 +35,5 @@
   <xacro:property name="has_thermal" value="$(arg has_thermal)"/>
   <xacro:property name="is_multiple" value="$(arg multiple)" />
-  <xacro:property name="nsp" value="$(arg namespace)" />
+  <xacro:property name="namespace" value="$(arg namespace)" />
   <xacro:property name="use_nominal_extrinsics" value="$(arg use_sim)"/>
   <xacro:if value="${robot_model not in ['v1', 'v2']}">

Commit message: Adding change 2

File: ari_description/robots/ari.urdf.xacro (robot description, xacro)
@@ -19,5 +19,5 @@
   <xacro:arg name="back_fisheye_camera" default="false"/>
   <xacro:arg name="laser_model" default="ydlidar-tg15"/> <!-- false, hokuyo, sick-551, sick-561, sick-571, ydlidar-tg30, ydlidar-tg15 -->
-  <xacro:arg name="camera_model_head" default="raspi"/>
+  <xacro:arg name="head_camera_model" default="raspi"/>
   <xacro:arg name="rgbd_sensors" default="false"/> <!-- false, true-->
   <xacro:arg name="has_thermal" default="false"/>
@@ -31,5 +31,5 @@
   <xacro:property name="back_fisheye_camera" value="$(arg back_fisheye_camera)" />
   <xacro:property name="laser_model" value="$(arg laser_model)" />
-  <xacro:property name="camera_model_head" value="$(arg camera_model_head)"/>
+  <xacro:property name="head_camera_model" value="$(arg head_camera_model)"/>
   <xacro:property name="rgbd_sensors" value="$(arg rgbd_sensors)"/>
   <xacro:property name="has_thermal" value="$(arg has_thermal)"/>
@@ -54,5 +54,5 @@
     <xacro:wrong_laser_model/>
   </xacro:if>
-  <xacro:if value="${camera_model_head not in ['raspi', 'realsense-d435', 'realsense-d435i']}">
+  <xacro:if value="${head_camera_model not in ['raspi', 'realsense-d435', 'realsense-d435i']}">
     <xacro:wrong_camera_model/>
   </xacro:if>

File: ari_description/urdf/head/head.urdf.xacro (robot description, xacro)
@@ -262,8 +262,8 @@
     <xacro:head_1 name="${name}_1" parent="${parent}" robot_model="${robot_model}" />
     <xacro:head_2 name="${name}_2" parent="${name}_1_link" robot_model="${robot_model}"/>
-    <xacro:if value="${camera_model_head == 'raspi'}">
+    <xacro:if value="${head_camera_model == 'raspi'}">
       <xacro:head_front_camera name="${name}_front_camera" parent="${name}_2_link"/>
     </xacro:if>
-    <xacro:if value="${(camera_model_head == 'realsense-d435') or (camera_model_head == 'realsense-d435i')}">
+    <xacro:if value="${(head_camera_model == 'realsense-d435') or (head_camera_model == 'realsense-d435i')}">
       <xacro:head_rgbd name="${name}_rgbd" parent="${name}_2_link"/>
     </xacro:if>

Commit message: Fixing use_sim_time

File: ari_description/robots/ari.urdf.xacro (robot description, xacro)
@@ -25,5 +25,5 @@
   <xacro:arg name="multiple" default="false"/>
   <xacro:arg name="namespace" default=""/>
-  <xacro:arg name="use_sim" default="false"/>
+  <xacro:arg name="use_sim_time" default="false"/>
   <xacro:property name="robot_model" value="$(arg robot_model)" />
   <xacro:property name="end_effector" value="$(arg end_effector)" />
@@ -36,5 +36,5 @@
   <xacro:property name="is_multiple" value="$(arg multiple)" />
   <xacro:property name="namespace" value="$(arg namespace)" />
-  <xacro:property name="use_nominal_extrinsics" value="$(arg use_sim)"/>
+  <xacro:property name="use_nominal_extrinsics" value="$(arg use_sim_time)"/>
   <xacro:if value="${robot_model not in ['v1', 'v2']}">
     <xacro:wrong_ari_robot_model/>
@@ -82,5 +82,5 @@
   <xacro:include filename="$(find ari_description)/ros2_control/ros2_control.urdf.xacro" />
   <xacro:ari_ros2_control
-    use_sim="$(arg use_sim)" />
+    use_sim_time="$(arg use_sim_time)" />
   <!-- Materials for visualization -->
   <xacro:include filename="$(find ari_description)/urdf/materials.urdf.xacro" />

File: ari_description/ros2_control/ros2_control.urdf.xacro (robot description, xacro)
@@ -14,5 +14,5 @@
 <robot xmlns:xacro="http://ros.org/wiki/xacro"
        name="ari" >
-  <xacro:macro name="ari_ros2_control" params="use_sim:=^|false">
+  <xacro:macro name="ari_ros2_control" params="use_sim_time:=^|false">
     <xacro:arg name="robot_model" default="v2" />
     <xacro:arg name="description_calibration_dir" default="$(find ari_description)/urdf/calibration" />
@@ -21,9 +21,15 @@
     <xacro:include filename="$(arg description_calibration_dir)/calibration_constants.urdf.xacro" />
     <!-- Simulation -->
-    <xacro:if value="$(arg use_sim)">
+    <xacro:if value="$(arg use_sim_time)">
+      <!-- Init the ROS 2 control gazebo interface -->
+      <gazebo>
+        <plugin filename="libgazebo_ros2_control.so" name="gazebo_ros2_control">
+          <parameters>$(find ari_description)/ros2_control/gazebo_controller_manager_cfg.yaml</parameters>
+        </plugin>
+      </gazebo>
       <ros2_control name="ros2_control_gazebo_system" type="system">
-          <hardware>
-            <plugin>gazebo_ros2_control/GazeboSystem</plugin>
-          </hardware>
+        <hardware>
+          <plugin>gazebo_ros2_control/GazeboSystem</plugin>
+        </hardware>
         <!-- wheels -->
         <xacro:include filename="$(find ari_description)/urdf/wheels/wheel.ros2_control.xacro" />
@@ -41,5 +47,5 @@
     </xacro:if>
     <!-- Hardware -->
-    <xacro:unless value="$(arg use_sim)">
+    <xacro:unless value="$(arg use_sim_time)">
       <!-- Dynamixels system -->
       <ros2_control name="ros2_control_ari_system_dynamixel" type="system" rw_rate="200">

Commit message: Adding front&back camera

File: ari_description/robots/ari.urdf.xacro (robot description, xacro)
@@ -16,4 +16,6 @@
   <xacro:arg name="robot_model" default="v2"/>
   <xacro:arg name="end_effector" default="no-end-effector"/>
+  <xacro:arg name="torso_front_camera_model" default="realsense-d435"/>
+  <xacro:arg name="torso_back_camera_model" default="realsense-t265"/>
   <xacro:arg name="front_fisheye_camera" default="false"/>
   <xacro:arg name="back_fisheye_camera" default="false"/>
@@ -28,4 +30,6 @@
   <xacro:property name="robot_model" value="$(arg robot_model)" />
   <xacro:property name="end_effector" value="$(arg end_effector)" />
+  <xacro:property name="torso_front_camera_model" value="$(arg torso_front_camera_model)" />
+  <xacro:property name="torso_back_camera_model" value="$(arg torso_back_camera_model)" />
   <xacro:property name="front_fisheye_camera" value="$(arg front_fisheye_camera)" />
   <xacro:property name="back_fisheye_camera" value="$(arg back_fisheye_camera)" />
@@ -42,4 +46,10 @@
   <xacro:if value="${end_effector not in ['no-end-effector', 'ari-hand']}">
     <xacro:wrong_end_effector/>
+  </xacro:if>
+  <xacro:if value="${torso_front_camera_model not in ['no-camera', 'realsense-d435i', 'realsense-d435']}">
+    <xacro:wrong_torso_front_camera_model/>
+  </xacro:if>
+  <xacro:if value="${torso_back_camera_model not in ['no-camera', 'realsense-t265']}">
+    <xacro:wrong_torso_back_camera_model/>
   </xacro:if>
   <xacro:if value="${front_fisheye_camera not in ['true', True, 'false', False, 'Jetson', 'PC']}">

Commit message: Add gazebo_version xacro argument

File: ari_description/robots/ari.urdf.xacro (robot description, xacro)
@@ -28,4 +28,5 @@
   <xacro:arg name="namespace" default=""/>
   <xacro:arg name="use_sim_time" default="false"/>
+  <xacro:arg name="gazebo_version" default="classic"/>
   <xacro:property name="robot_model" value="$(arg robot_model)" />
   <xacro:property name="end_effector" value="$(arg end_effector)" />
@@ -41,4 +42,5 @@
   <xacro:property name="namespace" value="$(arg namespace)" />
   <xacro:property name="use_nominal_extrinsics" value="$(arg use_sim_time)"/>
+  <xacro:property name="gazebo_version" value="$(arg gazebo_version)"/>
   <xacro:if value="${robot_model not in ['v1', 'v2']}">
     <xacro:wrong_ari_robot_model/>
